Commit message: change the name to 'hydrus_ground_transportation' and add .gitignore

File: mbzirc2019/hydrus_ground_transportation/robots/aerial/additional_modules.urdf.xacro (robot description, xacro)
@@ -5,5 +5,5 @@
   <!-- downward camera -->
   <xacro:extra_module name = "downward_camera" parent = "link3" visible = "1"
-                      model_url = "package://aerial_robot_practice/urdf/mesh/modules/sensor/camera_200_note_type_holder.dae">
+                      model_url = "package://hydrus_ground_transportation/urdf/mesh/modules/sensor/camera_200_note_type_holder.dae">
     <origin xyz="0.09 0.0 -0.02175" rpy="0 ${pi/2} 0 "/>
     <inertial>
@@ -36,5 +36,5 @@
         <origin rpy="${-pi/2} 0 0" xyz="0 0 0"/>
         <geometry>
-          <mesh filename="package://aerial_robot_practice/urdf/mesh/modules/mechanical/roller_BCBE10.dae"/>
+          <mesh filename="package://hydrus_ground_transportation/urdf/mesh/modules/mechanical/roller_BCBE10.dae"/>
         </geometry>
       </visual>

File: mbzirc2019/hydrus_ground_transportation/robots/aerial/hydrus.gazebo.xacro (robot description, xacro)
@@ -5,5 +5,5 @@
   <xacro:include filename="$(find hydrus)/robots/quad/euclid201806.gazebo.xacro" />
   <!-- additional modules -->
-  <xacro:include filename="$(find aerial_robot_practice)/robots/ground/additional_modules.urdf.xacro" />
+  <xacro:include filename="$(find hydrus_ground_transportation)/robots/aerial/additional_modules.urdf.xacro" />
   <!-- sensor plugin for downward camera -->
   <gazebo reference="downward_camera">

File: mbzirc2019/hydrus_ground_transportation/robots/aerial/hydrus.urdf.xacro (robot description, xacro)
@@ -5,4 +5,4 @@
   <xacro:include filename="$(find hydrus)/robots/quad/euclid201806.urdf.xacro" />
   <!-- additional modules -->
-  <xacro:include filename="$(find aerial_robot_practice)/robots/aerial/additional_modules.urdf.xacro" />
+  <xacro:include filename="$(find hydrus_ground_transportation)/robots/aerial/additional_modules.urdf.xacro" />
 </robot>

File: mbzirc2019/hydrus_ground_transportation/robots/ground/additional_modules.urdf.xacro (robot description, xacro)
@@ -5,5 +5,5 @@
   <!-- downward camera -->
   <xacro:extra_module name = "downward_camera" parent = "link3" visible = "1"
-                      model_url = "package://aerial_robot_practice/urdf/mesh/modules/sensor/camera_200_note_type_holder.dae">
+                      model_url = "package://hydrus_ground_transportation/urdf/mesh/modules/sensor/camera_200_note_type_holder.dae">
     <origin xyz="0.09 0.0 -0.02175" rpy="0 ${pi/2} 0 "/>
     <inertial>
@@ -36,5 +36,5 @@
         <origin rpy="${-pi/2} 0 0" xyz="0 0 0"/>
         <geometry>
-          <mesh filename="package://aerial_robot_practice/urdf/mesh/modules/mechanical/roller_BCBE10.dae"/>
+          <mesh filename="package://hydrus_ground_transportation/urdf/mesh/modules/mechanical/roller_BCBE10.dae"/>
         </geometry>
       </visual>

File: mbzirc2019/hydrus_ground_transportation/robots/ground/hydrus.gazebo.xacro (robot description, xacro)
@@ -5,5 +5,5 @@
   <xacro:include filename="$(find hydrus)/robots/quad/euclid201806.gazebo.xacro" />
   <!-- additional modules -->
-  <xacro:include filename="$(find aerial_robot_practice)/robots/aerial/additional_modules.urdf.xacro" />
+  <xacro:include filename="$(find hydrus_ground_transportation)/robots/ground/additional_modules.urdf.xacro" />
   <!-- sensor plugin for downward camera -->
   <gazebo reference="downward_camera">

File: mbzirc2019/hydrus_ground_transportation/robots/ground/hydrus.urdf.xacro (robot description, xacro)
@@ -5,4 +5,4 @@
   <xacro:include filename="$(find hydrus)/robots/quad/euclid201806.urdf.xacro" />
   <!-- additional modules -->
-  <xacro:include filename="$(find aerial_robot_practice)/robots/ground/additional_modules.urdf.xacro" />
+  <xacro:include filename="$(find hydrus_ground_transportation)/robots/ground/additional_modules.urdf.xacro" />
 </robot>
