Commit message: Change the battery type and the arrangement

File: mbzirc2019/hydrus_ground_transportation/robots/hydrus.urdf.xacro (robot description, xacro)
@@ -5,8 +5,8 @@
   <xacro:include filename="$(find hydrus)/urdf/common.xacro" />
   <xacro:include filename="$(find hydrus)/urdf/link.urdf.xacro" />
-  <xacro:hydrusx_link self="1" child="2" rotor_direction="-1" />
-  <xacro:hydrusx_link self="2" child="3" rotor_direction="1"  with_leg= "0" />
-  <xacro:hydrusx_link self="3" child="4" rotor_direction="-1" with_leg= "0" />
-  <xacro:hydrusx_link self="4" child="4" rotor_direction="1" />
+  <xacro:hydrusx_link self="1" child="2" rotor_direction="-1" with_battery = "0" />
+  <xacro:hydrusx_link self="2" child="3" rotor_direction="1"  with_leg= "0" with_battery = "0" />
+  <xacro:hydrusx_link self="3" child="4" rotor_direction="-1" with_leg= "0" with_battery = "0" />
+  <xacro:hydrusx_link self="4" child="4" rotor_direction="1" with_battery = "0"/>
   <!-- oboard sensors and processors -->
   <xacro:include filename="$(find hydrus)/robots/onboards/tx2_zed_201810/onboards.urdf.xacro" />
@@ -126,23 +126,46 @@
     </collision>
   </link>
-    <transmission name="actuated_leg1_joint_tran">
-      <type>transmission_interface/SimpleTransmission</type>
-      <joint name="actuated_leg1_joint">
-        <hardwareInterface>hardware_interface/EffortJointInterface</hardwareInterface>
-      </joint>
-      <actuator name="actuated_leg1_joint">
-        <hardwareInterface>hardware_interface/EffortJointInterface</hardwareInterface>
-        <mechanicalReduction>1</mechanicalReduction>
-      </actuator>
-    </transmission>
-    <transmission name="actuated_leg2_joint_tran">
-      <type>transmission_interface/SimpleTransmission</type>
-      <joint name="actuated_leg2_joint">
-        <hardwareInterface>hardware_interface/EffortJointInterface</hardwareInterface>
-      </joint>
-      <actuator name="actuated_leg2_joint">
-        <hardwareInterface>hardware_interface/EffortJointInterface</hardwareInterface>
-        <mechanicalReduction>1</mechanicalReduction>
-      </actuator>
-    </transmission>
+  <!-- special battery arrangement -->
+  <xacro:extra_module name = "bat1" parent = "link1" visible = "1"
+                      model_url = "package://hydrus/urdf/mesh/modules/battery/Kypom-3000-6s.stl" scale="0.001">
+    <origin xyz="${link_length/2} 0.0 -0.048" rpy="${pi/2} 0 0"/>
+    <inertial>
+      <origin xyz="0 0 0" rpy="0 0 0"/>
+      <mass value="0.4108"/>
+      <inertia
+          ixx="0.0001" iyy="0.0006" izz="0.0006"
+          ixy="0.0" ixz="0.0"  iyz="0.0"/>
+    </inertial>
+  </xacro:extra_module>
+  <xacro:extra_module name = "bat2" parent = "link4" visible = "1"
+                      model_url = "package://hydrus/urdf/mesh/modules/battery/Kypom-3000-6s.stl" scale="0.001">
+    <origin xyz="${link_length/2} 0.0 -0.048" rpy="${pi/2} 0 0"/>
+    <inertial>
+      <origin xyz="0 0 0" rpy="0 0 0"/>
+      <mass value="0.4108"/>
+      <inertia
+          ixx="0.0001" iyy="0.0006" izz="0.0006"
+          ixy="0.0" ixz="0.0"  iyz="0.0"/>
+    </inertial>
+  </xacro:extra_module>
+  <transmission name="actuated_leg1_joint_tran">
+    <type>transmission_interface/SimpleTransmission</type>
+    <joint name="actuated_leg1_joint">
+      <hardwareInterface>hardware_interface/EffortJointInterface</hardwareInterface>
+    </joint>
+    <actuator name="actuated_leg1_joint">
+      <hardwareInterface>hardware_interface/EffortJointInterface</hardwareInterface>
+      <mechanicalReduction>1</mechanicalReduction>
+    </actuator>
+  </transmission>
+  <transmission name="actuated_leg2_joint_tran">
+    <type>transmission_interface/SimpleTransmission</type>
+    <joint name="actuated_leg2_joint">
+      <hardwareInterface>hardware_interface/EffortJointInterface</hardwareInterface>
+    </joint>
+    <actuator name="actuated_leg2_joint">
+      <hardwareInterface>hardware_interface/EffortJointInterface</hardwareInterface>
+      <mechanicalReduction>1</mechanicalReduction>
+    </actuator>
+  </transmission>
 </robot>

Commit message: Remove the wrong leg model in end link

File: mbzirc2019/hydrus_ground_transportation/robots/hydrus.urdf.xacro (robot description, xacro)
@@ -8,5 +8,5 @@
   <xacro:hydrusx_link self="2" child="3" rotor_direction="1"  with_leg= "0" with_battery = "0" />
   <xacro:hydrusx_link self="3" child="4" rotor_direction="-1" with_leg= "0" with_battery = "0" />
-  <xacro:hydrusx_link self="4" child="4" rotor_direction="1" with_battery = "0"/>
+  <xacro:hydrusx_link self="4" child="4" rotor_direction="1"  with_leg= "0" with_battery = "0"/>
   <!-- oboard sensors and processors -->
   <xacro:include filename="$(find hydrus)/robots/onboards/tx2_zed_201810/onboards.urdf.xacro" />
@@ -84,5 +84,5 @@
     </collision>
   </link>
-  <!-- actuated leg in end link -->
+  <!-- actuated leg in end links: one actuated leg and one standrad leg -->
   <xacro:extra_module name = "actuated_leg2_stationary_part" parent = "link4" visible = "1"
                       model_url = "package://hydrus_ground_transportation/urdf/mesh/modules/mechanical/actuated_leg_stationary_part.dae">
@@ -126,4 +126,7 @@
     </collision>
   </link>
+  <xacro:standard_leg parent = "link4" self= "3" >
+    <origin xyz="${end_leg_offset} 0.0 0" rpy="0 0 0"/>
+  </xacro:standard_leg>
   <!-- special battery arrangement -->
   <xacro:extra_module name = "bat1" parent = "link1" visible = "1"

Commit message: Change the position of actuated legs: - leg1: link1 -> link2 - leg2: link4 -> link3

File: mbzirc2019/hydrus_ground_transportation/robots/hydrus.urdf.xacro (robot description, xacro)
@@ -13,8 +13,8 @@
   <xacro:onboards link = "2" />
   <!-- additional legs -->
-  <!-- actuated leg in head link -->
-  <xacro:extra_module name = "actuated_leg1_stationary_part" parent = "link1" visible = "1"
+  <!-- actuated leg in the second link -->
+  <xacro:extra_module name = "actuated_leg1_stationary_part" parent = "link2" visible = "1"
                       model_url = "package://hydrus_ground_transportation/urdf/mesh/modules/mechanical/actuated_leg_stationary_part.dae">
-    <origin xyz="${link_length/2 + 0.2355} 0.0 0" rpy="0 0 ${pi}"/>
+    <origin xyz="${general_leg_offset} 0.0 0" rpy="0 0 0"/>
     <inertial>
       <mass value = "0.142" />
@@ -55,5 +55,5 @@
     </collision>
   </link>
-  <!-- small omniwheel in third link -->
+  <!-- small omniwheel in the third link -->
   <joint name="link3_to_leg2" type="fixed">
     <parent link="link3"/>
@@ -84,8 +84,8 @@
     </collision>
   </link>
-  <!-- actuated leg in end links: one actuated leg and one standrad leg -->
-  <xacro:extra_module name = "actuated_leg2_stationary_part" parent = "link4" visible = "1"
+  <!-- actuated leg in the thrid links: one actuated leg and one standrad leg -->
+  <xacro:extra_module name = "actuated_leg2_stationary_part" parent = "link3" visible = "1"
                       model_url = "package://hydrus_ground_transportation/urdf/mesh/modules/mechanical/actuated_leg_stationary_part.dae">
-    <origin xyz="${general_leg_offset} 0.0 0" rpy="0 0 0"/>
+    <origin xyz="${link_length/2 + 0.2355} 0.0 0" rpy="0 0 ${pi}"/>
     <inertial>
       <mass value = "0.142" />
