Commit message: Rename the task1 package.

File: mbzirc2020_task1/mbzirc2020_task1_common/urdf/hawk.urdf.xacro (robot description, xacro)
@@ -14,5 +14,5 @@
       <origin xyz="0 0 0" rpy="0 0 0" />
       <geometry>
-        <mesh filename="package://mbzirc_common/urdf/meshes/hawk.stl" scale=".0254 .0254 .0254"/> <!-- mm has bug, right now use inch from ST8 -->
+        <mesh filename="package://mbzirc2020_task1_common/urdf/meshes/hawk.stl" scale=".0254 .0254 .0254"/> <!-- mm has bug, right now use inch from ST8 -->
         <cylinder radius=".295" length=".23"/>
       </geometry>
@@ -24,5 +24,5 @@
       <origin xyz="0 0 0" rpy="0 0 0" />
       <geometry>
-        <mesh filename="package://mbzirc_common/urdf/meshes/hawk.stl" scale=".0254 .0254 .0254"/> <!-- mm has bug, right now use inch from ST8 -->
+        <mesh filename="package://mbzirc2020_task1_common/urdf/meshes/hawk.stl" scale=".0254 .0254 .0254"/> <!-- mm has bug, right now use inch from ST8 -->
       </geometry>
     </collision>
