Commit message: 1. add image trigger for the zed mini stereo camera, in order to let it pulish camera_info for the nodelet init function in "single_color_ground_object_detection.launch" 2. modify the hsv color filter paramters for real red object 3. modify the robot regarding to the sheet mass (0.41Kg) 4. set the oneshot search mode for the openning form search 5. seperate the model configuration regarding to the single red object between simulation and real machine

File: mbzirc2020_task3/mbzirc2020_task3_common/robots/hydrus.urdf.xacro (robot description, xacro)
@@ -8,5 +8,5 @@
   <xacro:onboards link = "2" />
   <!-- add sheet as a rigid point, meanings less inertia -->
-  <xacro:property name="sheet_mass" value=".5" />
+  <xacro:property name="sheet_mass" value=".41" />
   <xacro:extra_module name = "sheet_anchor1" parent = "leg1" visible = "0" >
     <origin xyz="0.0 0.0 0.0" rpy="0 0 0"/>
