Commit message: Refactor mbzirc2020_task3 package

File: mbzirc2020/mbzirc2020_task3/mbzirc2020_task3_common/robots/hydrus.gazebo.xacro (robot description, xacro)
@@ -5,4 +5,42 @@
   <xacro:include filename="$(find mbzirc2020_task3_common)/robots/hydrus.urdf.xacro" />
   <!-- gazebo plugin for sensors -->
-  <xacro:include filename="$(find hydrus)/robots/onboards/tx2_zed_201810/onboards.gazebo.xacro" />
+  <xacro:include filename="$(find mbzirc2020_common)/robots/default.gazebo.xacro" />
+  <!-- gazebo for FLIR -->
+  <!-- RGB camera instead of IR camera -->
+  <gazebo reference="flir_thermal_frame">
+    <sensor type="camera" name="flir_thermal_camera">
+      <update_rate>20.0</update_rate>
+      <camera name="thermal">
+        <horizontal_fov>1.57</horizontal_fov>
+        <image>
+          <width>1280</width>
+          <height>720</height>
+          <format>RGB</format>
+        </image>
+        <clip>
+          <near>0.02</near>
+          <far>300</far>
+        </clip>
+        <noise>
+          <type>gaussian</type>
+          <mean>0.0</mean>
+          <stddev>0.007</stddev>
+        </noise>
+      </camera>
+      <plugin name="camera_controller" filename="libgazebo_ros_camera.so">
+        <alwaysOn>true</alwaysOn>
+        <updateRate>0.0</updateRate>
+        <cameraName>flir</cameraName>
+        <imageTopicName>image_raw</imageTopicName>
+        <cameraInfoTopicName>camera_info</cameraInfoTopicName>
+        <frameName>flir_thermal_optical_frame</frameName>
+        <hackBaseline>0.07</hackBaseline>
+        <distortionK1>0.0</distortionK1>
+        <distortionK2>0.0</distortionK2>
+        <distortionK3>0.0</distortionK3>
+        <distortionT1>0.0</distortionT1>
+        <distortionT2>0.0</distortionT2>
+      </plugin>
+    </sensor>
+  </gazebo>
 </robot>

File: mbzirc2020/mbzirc2020_task3/mbzirc2020_task3_common/robots/hydrus.urdf.xacro (robot description, xacro)
@@ -3,9 +3,46 @@
     xmlns:xacro="http://www.ros.org/wiki/xacro" name="hydrusx" >
   <!-- base kinematics model -->
-  <xacro:include filename="$(find hydrus)/robots/quad/default.urdf.xacro" />
-  <!-- oboard sensors and processors -->
-  <xacro:include filename="$(find hydrus)/robots/onboards/tx2_zed_201810/onboards.urdf.xacro" />
-  <xacro:onboards link = "2" />
-  <!-- add sheet as a rigid point, meanings less inertia -->
+  <xacro:include filename="$(find mbzirc2020_common)/robots/default.urdf.xacro" />
+  <xacro:robot_model tilt_angle = "10" horizontal_vio = "0"  />
+  <!-- processor: intel upboard -->
+  <xacro:extra_module name = "pc" parent = "link2" visible = "1"
+                      model_url = "package://mbzirc2020_common/urdf/mesh/modules/processor/intel_upboard_fixed_joint_unit.dae" >
+    <origin xyz="${link_length / 2 + 0.2845} 0.011 0.016" rpy="0 0 ${pi}"/>
+    <inertial>
+      <mass value = "0.117" />
+      <origin xyz="${21 * 0.001} ${4 * 0.001} ${12 * 0.001}" rpy="0 0 0"/>
+      <inertia
+          ixx="0.00004" ixy="0.0" ixz="0.0"
+          iyy="0.00008" iyz="0.0"
+          izz="0.00011"/>
+    </inertial>
+  </xacro:extra_module>
+  <!-- end: intel upboard -->
+  <!-- sensor -->
+  <!-- 1. FLIR -->
+  <!-- TODO: accurate intertia parameters and position -->
+  <xacro:extra_module name = "flir_thermal_frame" parent = "link2" visible = "0"  >
+    <origin xyz="${link_length / 2 + 0.24455} 0.05545 -0.015" rpy="0 ${pi/2} ${3 * pi/4}"/>
+    <inertial>
+      <mass value = "0.02" />
+      <origin xyz="0 0 0" rpy="0 0 0"/>
+      <inertia
+          ixx="0.0" ixy="0.0" ixz="0.0"
+          iyy="0.0" iyz="0.0" izz="0.0"/>
+    </inertial>
+  </xacro:extra_module>
+  <xacro:extra_module name = "flir_thermal_optical_frame" parent = "flir_thermal_frame">
+    <origin xyz="0 0 0" rpy="${-pi / 2} 0 ${-pi / 2}"/>
+    <inertial>
+      <mass value = "0.0" />
+      <origin xyz="0 0 0" rpy="0 0 0"/>
+      <inertia
+          ixx="0.0" ixy="0.0" ixz="0.0"
+          iyy="0.0" iyz="0.0"
+          izz="0.0"/>
+    </inertial>
+  </xacro:extra_module>
+  <!-- sheet -->
+  <!--
   <xacro:property name="sheet_mass" value=".41" />
   <xacro:extra_module name = "sheet_anchor1" parent = "leg1" visible = "0" >
@@ -29,3 +66,4 @@
     </inertial>
   </xacro:extra_module>
+  -->
 </robot>
