Commit message: - Update the blanket weight - Rearrange the battery position and number - Rearrange the downward realsense sensor position

File: mbzirc2020/mbzirc2020_task3/mbzirc2020_task3_common/robots/hydrus.urdf.xacro (robot description, xacro)
@@ -5,5 +5,28 @@
   <xacro:arg name="horizontal_vio" default="0" />
   <xacro:include filename="$(find mbzirc2020_common)/robots/default.urdf.xacro" />
-  <xacro:robot_model tilt_angle = "10" horizontal_vio = "$(arg horizontal_vio)"  />
+  <xacro:robot_model tilt_angle = "10" downward_vio = "0" horizontal_vio = "$(arg horizontal_vio)" default_battery = "0"  />
+  <!-- special battery arrangement -->
+  <xacro:extra_module name = "bat1" parent = "link2" visible = "1"
+                      model_url = "package://hydrus/urdf/mesh/battery/Kypom-3000-6s.dae" scale="0.001">
+    <origin xyz="${link_length/2} 0.0 -0.048" rpy="0 0 0"/>
+    <inertial>
+      <origin xyz="0 0 0" rpy="0 0 0"/>
+      <mass value="0.4108"/>
+      <inertia
+          ixx="0.0001" iyy="0.0006" izz="0.0006"
+          ixy="0.0" ixz="0.0"  iyz="0.0"/>
+    </inertial>
+  </xacro:extra_module>
+  <xacro:extra_module name = "bat2" parent = "link3" visible = "1"
+                      model_url = "package://hydrus/urdf/mesh/battery/Kypom-3000-6s.dae" scale="0.001">
+    <origin xyz="${link_length/2} 0.0 -0.048" rpy="0 0 0"/>
+    <inertial>
+      <origin xyz="0 0 0" rpy="0 0 0"/>
+      <mass value="0.4108"/>
+      <inertia
+          ixx="0.0001" iyy="0.0006" izz="0.0006"
+          ixy="0.0" ixz="0.0"  iyz="0.0"/>
+    </inertial>
+  </xacro:extra_module>
   <!-- processor: intel upboard -->
   <xacro:extra_module name = "pc" parent = "link2" visible = "1"
@@ -11,5 +34,5 @@
     <origin xyz="${link_length / 2 + 0.2845} 0.011 0.016" rpy="0 0 ${pi}"/>
     <inertial>
-      <mass value = "0.117" />
+      <mass value = "0.120" />
       <origin xyz="${21 * 0.001} ${4 * 0.001} ${12 * 0.001}" rpy="0 0 0"/>
       <inertia
@@ -21,5 +44,19 @@
   <!-- end: intel upboard -->
   <!-- sensor -->
-  <!-- 1. FLIR -->
+  <!-- 1. downward rs-t265 (VIO) -->
+  <xacro:extra_module name = "realsense1_pose_frame" parent = "link3" visible = "1"
+                      model_url = "package://mbzirc2020_common/urdf/mesh/modules/sensor/downward_realsense_unit.STL">
+    <origin xyz="0.173 0.0 -0.022" rpy="${pi} ${pi/2} ${pi/2}"/>
+    <inertial>
+      <mass value = "0.065" /> <!-- sensor + usb-cable -->
+      <origin xyz="-0.009 -0.01 0" rpy="0 0 0"/>
+      <inertia
+          ixx="0.0" ixy="0.0" ixz="0.0"
+          iyy="0.0" iyz="0.0"
+          izz="0.0"/>
+    </inertial>
+  </xacro:extra_module>
+  <!-- end: rs-5265 -->
+  <!-- 2. FLIR -->
   <xacro:extra_module name = "lepton_camera" parent = "link2" visible = "0"  >
     <origin xyz="${link_length / 2 + 0.24455} 0.05545 -0.015" rpy="0 ${pi/2} ${3 * pi/4}"/>
@@ -44,5 +81,5 @@
   </xacro:extra_module>
   <!-- sheet -->
-  <xacro:property name="sheet_mass" value=".41" />
+  <xacro:property name="sheet_mass" value=".65" />
   <xacro:extra_module name = "sheet_anchor1" parent = "leg1" visible = "0" >
     <origin xyz="0.0 0.0 0.0" rpy="0 0 0"/>

Commit message: Update the sheet weight

File: mbzirc2020/mbzirc2020_task3/mbzirc2020_task3_common/robots/hydrus.urdf.xacro (robot description, xacro)
@@ -81,5 +81,5 @@
   </xacro:extra_module>
   <!-- sheet -->
-  <xacro:property name="sheet_mass" value=".65" />
+  <xacro:property name="sheet_mass" value=".68" />
   <xacro:extra_module name = "sheet_anchor1" parent = "leg1" visible = "0" >
     <origin xyz="0.0 0.0 0.0" rpy="0 0 0"/>

Commit message: modified realsense position in model for task3

File: mbzirc2020/mbzirc2020_task3/mbzirc2020_task3_common/robots/hydrus.urdf.xacro (robot description, xacro)
@@ -5,5 +5,5 @@
   <xacro:arg name="horizontal_vio" default="0" />
   <xacro:include filename="$(find mbzirc2020_common)/robots/default.urdf.xacro" />
-  <xacro:robot_model tilt_angle = "10" downward_vio = "0" horizontal_vio = "$(arg horizontal_vio)" default_battery = "0"  />
+  <xacro:robot_model tilt_angle = "10" downward_vio = "1" horizontal_vio = "$(arg horizontal_vio)" default_battery = "0"  />
   <!-- special battery arrangement -->
   <xacro:extra_module name = "bat1" parent = "link2" visible = "1"
@@ -45,16 +45,16 @@
   <!-- sensor -->
   <!-- 1. downward rs-t265 (VIO) -->
-  <xacro:extra_module name = "realsense1_pose_frame" parent = "link3" visible = "1"
-                      model_url = "package://mbzirc2020_common/urdf/mesh/modules/sensor/downward_realsense_unit.STL">
-    <origin xyz="0.173 0.0 -0.022" rpy="${pi} ${pi/2} ${pi/2}"/>
-    <inertial>
-      <mass value = "0.065" /> <!-- sensor + usb-cable -->
-      <origin xyz="-0.009 -0.01 0" rpy="0 0 0"/>
-      <inertia
-          ixx="0.0" ixy="0.0" ixz="0.0"
-          iyy="0.0" iyz="0.0"
-          izz="0.0"/>
-    </inertial>
-  </xacro:extra_module>
+  <!-- <xacro:extra_module name = "realsense1_pose_frame" parent = "link3" visible = "1" -->
+  <!--                     model_url = "package://mbzirc2020_common/urdf/mesh/modules/sensor/downward_realsense_unit.STL"> -->
+  <!--   <origin xyz="0.173 0.0 -0.022" rpy="${pi} ${pi/2} ${pi/2}"/> -->
+  <!--   <inertial> -->
+	<!--     <mass value = "0.065" /> -->
+  <!--     <origin xyz="-0.009 -0.01 0" rpy="0 0 0"/> -->
+  <!--     <inertia -->
+  <!--         ixx="0.0" ixy="0.0" ixz="0.0" -->
+  <!--         iyy="0.0" iyz="0.0" -->
+  <!--         izz="0.0"/> -->
+  <!--   </inertial> -->
+  <!-- </xacro:extra_module> -->
   <!-- end: rs-5265 -->
   <!-- 2. FLIR -->
