Commit message: - add fire inside the tower - set the camera view to be horizontal

File: mbzirc2020/mbzirc2020_task3/mbzirc2020_task3_common/robots/hydrus_hokuyo.urdf.xacro (robot description, xacro)
@@ -56,7 +56,12 @@
   <!-- </xacro:extra_module> -->
   <!-- end: rs-5265 -->
+  <!-- hokuyo ust201x laser -->
+  <xacro:include filename="$(find hector_sensors_description)/urdf/hokuyo_utm30lx.urdf.xacro" />
+  <xacro:hokuyo_utm30lx_model name="laser0" parent="link2">
+    <origin xyz="${link_length / 2 + 0.3} 0.0 0.1" rpy="0 0 ${-1 * pi/4}"/>
+  </xacro:hokuyo_utm30lx_model>
   <!-- 2. FLIR -->
-  <xacro:extra_module name = "lepton_camera" parent = "link2" visible = "0"  >
-    <origin xyz="${link_length / 2 + 0.24455} 0.05545 -0.015" rpy="0 ${pi/2} ${3 * pi/4}"/>
+  <xacro:extra_module name = "lepton_camera" parent = "laser0_frame" visible = "0"  >
+    <origin xyz="0.035 0 -0.04" rpy="0 0 0"/>
     <inertial>
       <mass value = "0.02" />
@@ -78,30 +83,3 @@
     </inertial>
   </xacro:extra_module>
-  <!-- sheet -->
-  <xacro:property name="sheet_mass" value=".68" />
-  <xacro:extra_module name = "sheet_anchor1" parent = "leg1" visible = "0" >
-    <origin xyz="0.0 0.0 0.0" rpy="0 0 0"/>
-    <inertial>
-      <origin xyz="0 0 0" rpy="0 0 0"/>
-      <mass value="${sheet_mass/2}"/>
-      <inertia
-          ixx="0.0001" iyy="0.0001" izz="0.0002"
-          ixy="0.0" ixz="0.0"  iyz="0.0"/>
-    </inertial>
-  </xacro:extra_module>
-  <xacro:extra_module name = "sheet_anchor2" parent = "leg5" visible = "0" >
-    <origin xyz="0.0 0.0 0.0" rpy="0 0 0"/>
-    <inertial>
-      <origin xyz="0 0 0" rpy="0 0 0"/>
-      <mass value="${sheet_mass/2}"/>
-      <inertia
-          ixx="0.0001" iyy="0.0001" izz="0.0002"
-          ixy="0.0" ixz="0.0"  iyz="0.0"/>
-    </inertial>
-  </xacro:extra_module>
-  <!-- hokuyo ust201x laser -->
-  <xacro:include filename="$(find hector_sensors_description)/urdf/hokuyo_utm30lx.urdf.xacro" />
-  <xacro:hokuyo_utm30lx_model name="laser0" parent="link2">
-    <origin xyz="${link_length / 2 + 0.3} 0.0 0.1" rpy="0 0 ${-1 * pi/4}"/>
-  </xacro:hokuyo_utm30lx_model>
 </robot>
