Commit message: Refactor mbzirc2020_task2 package

File: mbzirc2020/mbzirc2020_task2/mbzirc2020_task2_common/robots/hydrus.gazebo.xacro (robot description, xacro)
@@ -2,34 +2,15 @@
 <robot
     xmlns:xacro="http://www.ros.org/wiki/xacro" name="hydrusx" >
-  <!-- robot urdf and gazebo plugin for sensors-->
-  <xacro:include filename="$(find hydrus)/robots/default.gazebo.xacro" />
-    <!-- stereo camera: depth, color based on left camera -->
-  <xacro:extra_module name = "zed_left_camera_frame" parent = "zed_camera_center">
-    <origin xyz="0.002 0.03 0" rpy="0 0 0"/>
-    <inertial>
-      <mass value = "0.00001" />
-      <origin xyz="0 0 0" rpy="0 0 0"/>
-      <inertia
-          ixx="0.000001" ixy="0.0" ixz="0.0"
-          iyy="0.000001" iyz="0.0"
-          izz="0.000002"/>
-    </inertial>
-  </xacro:extra_module>
-  <xacro:extra_module name = "zed_left_camera_optical_frame" parent = "zed_left_camera_frame">
-    <origin xyz="0 0 0" rpy="${-pi / 2} 0 ${-pi / 2}"/>
-    <inertial>
-      <mass value = "0.00001" />
-      <origin xyz="0 0 0" rpy="0 0 0"/>
-      <inertia
-          ixx="0.000001" ixy="0.0" ixz="0.0"
-          iyy="0.000001" iyz="0.0"
-          izz="0.000002"/>
-    </inertial>
-  </xacro:extra_module>
-  <gazebo reference="zed_left_camera_frame">
-    <sensor type="depth" name="zed_depth_camera">
-      <update_rate>20.0</update_rate>
+  <!-- base robot model -->
+  <xacro:include filename="$(find mbzirc2020_task2_common)/robots/hydrus.urdf.xacro" />
+  <!-- gazebo plugin for sensors -->
+  <xacro:include filename="$(find mbzirc2020_common)/robots/default.gazebo.xacro" />
+  <!-- gazebo for Realsense D435 -->
+  <!-- TODO: precise topic name and optical frame position -->
+  <gazebo reference="rs_d435_camera_frame">
+    <sensor type="depth" name="rs_d435_camera">
+      <update_rate>30.0</update_rate>
       <camera name="head">
-        <horizontal_fov>1.57</horizontal_fov>
+        <horizontal_fov>1.59174027782</horizontal_fov>
         <image>
           <width>1280</width>
@@ -51,11 +32,11 @@
         <alwaysOn>true</alwaysOn>
         <updateRate>0.0</updateRate>
-        <cameraName>zed</cameraName>
-        <imageTopicName>rgb/image_rect_color</imageTopicName>
-        <cameraInfoTopicName>rgb/camera_info</cameraInfoTopicName>
+        <cameraName>rs_d435</cameraName>
+        <imageTopicName>rs_d435/image_rect_color</imageTopicName>
+        <cameraInfoTopicName>rs_d435/camera_info</cameraInfoTopicName>
         <depthImageTopicName>depth/depth_registered</depthImageTopicName>
         <depthImageInfoTopicName>depth/camera_info</depthImageInfoTopicName>
         <pointCloudTopicName>point_cloud/cloud_registered</pointCloudTopicName>
-        <frameName>zed_left_camera_optical_frame</frameName>
+        <frameName>rs_d435_camera_optical_frame</frameName>
         <pointCloudCutoff>0.05</pointCloudCutoff>
         <distortionK1>0</distortionK1>

Commit message: Add realsense D435 for task2: 1. add sensor urdf model 2. tune servo configuration for tilting sensor

File: mbzirc2020/mbzirc2020_task2/mbzirc2020_task2_common/robots/hydrus.gazebo.xacro (robot description, xacro)
@@ -7,47 +7,115 @@
   <xacro:include filename="$(find mbzirc2020_common)/robots/default.gazebo.xacro" />
   <!-- gazebo for Realsense D435 -->
-  <!-- TODO: precise topic name and optical frame position -->
-  <gazebo reference="rs_d435_camera_frame">
+  <!--  The following values model the aluminum peripherial case for the
+        D435 camera, with the camera joint represented by the actual
+        peripherial camera tripod mount -->
+  <xacro:property name="d435_cam_width" value="0.090"/>
+  <xacro:property name="d435_cam_height" value="0.025"/>
+  <xacro:property name="d435_cam_depth" value="0.02505"/>
+  <xacro:property name="d435_cam_mount_from_center_offset" value="0.0149"/>
+  <!--  The following offset is relative the the physical D435 camera peripherial
+        camera tripod mount -->
+  <xacro:property name="d435_cam_depth_px" value="${d435_cam_mount_from_center_offset}"/>
+  <xacro:property name="d435_cam_depth_py" value="0.0175"/>
+  <xacro:property name="d435_cam_depth_pz" value="${d435_cam_height/2}"/>
+  <material name="aluminum">
+    <color rgba="0.5 0.5 0.5 1"/>
+  </material>
+  <!-- camera depth joints and links -->
+  <joint name="rs_d435_depth_joint" type="fixed">
+    <origin xyz="0 0 0" rpy="0 0 0"/>
+    <parent link="rs_d435_link"/>
+    <child link="rs_d435_depth_frame" />
+  </joint>
+  <link name="rs_d435_depth_frame"/>
+  <joint name="rs_d435_depth_optical_joint" type="fixed">
+    <origin xyz="0 0 0" rpy="${-pi/2} 0 ${-pi/2}" />
+    <parent link="rs_d435_depth_frame" />
+    <child link="rs_d435_depth_optical_frame" />
+  </joint>
+  <link name="rs_d435_depth_optical_frame"/>
+  <!-- camera left IR joints and links -->
+  <joint name="rs_d435_left_ir_joint" type="fixed">
+    <origin xyz="0 ${d435_cam_depth_to_left_ir_offset} 0" rpy="0 0 0" />
+    <parent link="rs_d435_depth_frame" />
+    <child link="rs_d435_left_ir_frame" />
+  </joint>
+  <link name="rs_d435_left_ir_frame"/>
+  <joint name="rs_d435_left_ir_optical_joint" type="fixed">
+    <origin xyz="0 0 0" rpy="${-pi/2} 0 ${-pi/2}" />
+    <parent link="rs_d435_left_ir_frame" />
+    <child link="rs_d435_left_ir_optical_frame" />
+  </joint>
+  <link name="rs_d435_left_ir_optical_frame"/>
+  <!-- camera right IR joints and links -->
+  <joint name="rs_d435_right_ir_joint" type="fixed">
+    <origin xyz="0 ${d435_cam_depth_to_right_ir_offset} 0" rpy="0 0 0" />
+    <parent link="rs_d435_depth_frame" />
+    <child link="rs_d435_right_ir_frame" />
+  </joint>
+  <link name="rs_d435_right_ir_frame"/>
+  <joint name="rs_d435_right_ir_optical_joint" type="fixed">
+    <origin xyz="0 0 0" rpy="${-pi/2} 0 ${-pi/2}" />
+    <parent link="rs_d435_right_ir_frame" />
+    <child link="rs_d435_right_ir_optical_frame" />
+  </joint>
+  <link name="rs_d435_right_ir_optical_frame"/>
+  <!-- camera color joints and links -->
+  <joint name="rs_d435_color_joint" type="fixed">
+    <origin xyz="0 ${d435_cam_depth_to_color_offset} 0" rpy="0 0 0" />
+    <parent link="rs_d435_depth_frame" />
+    <child link="rs_d435_color_frame" />
+  </joint>
+  <link name="rs_d435_color_frame"/>
+  <joint name="rs_d435_color_optical_joint" type="fixed">
+    <origin xyz="0 0 0" rpy="${-pi/2} 0 ${-pi/2}" />
+    <parent link="rs_d435_color_frame" />
+    <child link="rs_d435_color_optical_frame" />
+  </joint>
+  <link name="rs_d435_color_optical_frame"/>
+  <!-- gazebo plugin -->
+  <gazebo reference="rs_d435_color_frame">
     <sensor type="depth" name="rs_d435_camera">
-      <update_rate>30.0</update_rate>
+      <update_rate>20.0</update_rate>
       <camera name="head">
-        <horizontal_fov>1.59174027782</horizontal_fov>
-        <image>
-          <width>1280</width>
-          <height>720</height>
-          <format>B8G8R8</format>
-        </image>
-        <clip>
-          <near>0.02</near>
-          <far>300</far>
-        </clip>
-        <noise>
-          <type>gaussian</type>
-          <mean>0.0</mean>
-          <stddev>0.007</stddev>
-        </noise>
+	<horizontal_fov>1.59174</horizontal_fov>
+	<vertical_fov>1.14319</vertical_fov>
+	<image>
+	  <width>1280</width>
+	  <height>720</height>
+	  <format>RGB</format>
+	</image>
+	<clip>
+	  <near>0.02</near>
+	  <far>300</far>
+	</clip>
+	<noise>
+	  <type>gaussian</type>
+	  <mean>0.0</mean>
+	  <stddev>0.007</stddev>
+	</noise>
       </camera>
       <plugin name="depth_camera" filename="libgazebo_ros_openni_kinect.so">
-        <baseline>0.06</baseline>
-        <alwaysOn>true</alwaysOn>
-        <updateRate>0.0</updateRate>
-        <cameraName>rs_d435</cameraName>
-        <imageTopicName>rs_d435/image_rect_color</imageTopicName>
-        <cameraInfoTopicName>rs_d435/camera_info</cameraInfoTopicName>
-        <depthImageTopicName>depth/depth_registered</depthImageTopicName>
-        <depthImageInfoTopicName>depth/camera_info</depthImageInfoTopicName>
-        <pointCloudTopicName>point_cloud/cloud_registered</pointCloudTopicName>
-        <frameName>rs_d435_camera_optical_frame</frameName>
-        <pointCloudCutoff>0.05</pointCloudCutoff>
-        <distortionK1>0</distortionK1>
-        <distortionK2>0</distortionK2>
-        <distortionK3>0</distortionK3>
-        <distortionT1>0</distortionT1>
-        <distortionT2>0</distortionT2>
-        <CxPrime>0</CxPrime>
-        <Cx>0</Cx>
-        <Cy>0</Cy>
-        <focalLength>0</focalLength>
-        <hackBaseline>0</hackBaseline>
+	<baseline>0.06</baseline>
+	<alwaysOn>true</alwaysOn>
+	<updateRate>0.0</updateRate>
+	<cameraName>rs_d435</cameraName>
+	<imageTopicName>color/image_rect_color</imageTopicName>
+	<cameraInfoTopicName>color/camera_info</cameraInfoTopicName>
+	<depthImageCameraInfoTopicName>aligned_depth_to_color/camera_info</depthImageCameraInfoTopicName>
+	<depthImageTopicName>aligned_depth_to_color/image_raw</depthImageTopicName>
+	<pointCloudTopicName>depth_registered/points</pointCloudTopicName>
+	<frameName>rs_d435_color_optical_frame</frameName>
+	<pointCloudCutoff>0.05</pointCloudCutoff>
+	<distortionK1>0</distortionK1>
+	<distortionK2>0</distortionK2>
+	<distortionK3>0</distortionK3>
+	<distortionT1>0</distortionT1>
+	<distortionT2>0</distortionT2>
+	<CxPrime>0</CxPrime>
+	<Cx>0</Cx>
+	<Cy>0</Cy>
+	<focalLength>0</focalLength>
+	<hackBaseline>0</hackBaseline>
       </plugin>
     </sensor>

File: mbzirc2020/mbzirc2020_task2/mbzirc2020_task2_common/robots/hydrus.urdf.xacro (robot description, xacro)
@@ -4,5 +4,5 @@
   <!-- base kinematics model -->
   <xacro:include filename="$(find mbzirc2020_common)/robots/default.urdf.xacro" />
-  <xacro:robot_model tilt_angle = "10" horizontal_vio = "0" default_battery = "0"  />
+  <xacro:robot_model tilt_angle = "10" downward_vio = "0" horizontal_vio = "0" default_battery = "0"  />
   <!-- special battery arrangement -->
   <xacro:extra_module name = "bat1" parent = "link1" visible = "1"
@@ -44,11 +44,25 @@
   <!-- end: intel upboard -->
   <!-- sensor -->
-  <!-- 1. Realsense D435 -->
-  <!-- TODO: accurate intertia parameters and position -->
+  <!-- 1. downward rs-t265 (VIO) -->
+  <xacro:extra_module name = "realsense1_pose_frame" parent = "link3" visible = "1"
+                      model_url = "package://mbzirc2020_common/urdf/mesh/modules/sensor/downward_realsense_unit.STL">
+    <origin xyz="${link_length/2 - 0.111} 0.0 -0.022" rpy="${pi} ${pi/2} ${pi/2}"/>
+    <inertial>
+      <mass value = "0.065" /> <!-- sensor + usb-cable -->
+      <origin xyz="-0.009 -0.01 0" rpy="0 0 0"/>
+      <inertia
+          ixx="0.0" ixy="0.0" ixz="0.0"
+          iyy="0.0" iyz="0.0"
+          izz="0.0"/>
+    </inertial>
+  </xacro:extra_module>
+  <!-- end: rs-5265 -->
+  <!-- 2. Realsense D435 -->
+    <!-- TODO: accurate intertia parameters and position -->
   <xacro:extra_module name = "rs_d435_mount" parent = "link2" visible = "1"
                       model_url = "package://mbzirc2020_common/urdf/mesh/modules/sensor/rs_d435_unit2.STL">
     <origin xyz="${link_length / 2} 0 0" rpy="0 0 0"/>
     <inertial>
-      <mass value = "0" />
+      <mass value = "0.0" />
       <origin xyz="0 0 0" rpy="0 0 0"/>
       <inertia
@@ -74,8 +88,8 @@
     </inertial>
   </link>
-  <xacro:extra_module name = "rs_d435_camera_frame" parent = "rs_d435_servo" visible = "1" model_url = "package://mbzirc2020_common/urdf/mesh/modules/sensor/rs_d435_unit1.STL">
+  <xacro:extra_module name = "rs_d435_unit" parent = "rs_d435_servo" visible = "1" model_url = "package://mbzirc2020_common/urdf/mesh/modules/sensor/rs_d435_unit1.STL">
     <origin xyz="0.05275 0.01005 0" rpy="0 0 ${pi / 2}"/>
     <inertial>
-      <mass value = "0.095" />
+      <mass value = "0.124" /> <!-- includes usb cable, servo, mounts -->
       <origin xyz="-0.01005 0 0" rpy="0 0 0"/>
       <inertia
@@ -84,13 +98,14 @@
     </inertial>
   </xacro:extra_module>
-  <xacro:extra_module name = "rs_d435_camera_optical_frame" parent = "rs_d435_camera_frame">
-    <origin xyz="0 0 0" rpy="${-pi / 2} 0 ${-pi / 2}"/>
+  <!-- rs_d435_link is the parrent of sensors' frame, identical to rs_d435_left_ir_frame  -->
+  <xacro:extra_module name = "rs_d435_link" parent = "rs_d435_unit" visible = "0" >
+    <origin xyz="-0.008 0.0175 0 " rpy="0 0 0"/>
     <inertial>
       <mass value = "0.0" />
       <origin xyz="0 0 0" rpy="0 0 0"/>
       <inertia
-          ixx="0.0" ixy="0.0" ixz="0.0"
-          iyy="0.0" iyz="0.0"
-          izz="0.0"/>
+	  ixx="0.0" ixy="0.0" ixz="0.0"
+	  iyy="0.0" iyz="0.0"
+	  izz="0.0"/>
     </inertial>
   </xacro:extra_module>

Commit message: Fix bug about missing paramters of realsense model in gazebo

File: mbzirc2020/mbzirc2020_task2/mbzirc2020_task2_common/robots/hydrus.gazebo.xacro (robot description, xacro)
@@ -10,4 +10,7 @@
         D435 camera, with the camera joint represented by the actual
         peripherial camera tripod mount -->
+  <xacro:property name="d435_cam_depth_to_left_ir_offset" value="0.0"/>
+  <xacro:property name="d435_cam_depth_to_right_ir_offset" value="-0.050"/>
+  <xacro:property name="d435_cam_depth_to_color_offset" value="0.015"/>
   <xacro:property name="d435_cam_width" value="0.090"/>
   <xacro:property name="d435_cam_height" value="0.025"/>
