Commit message: Improve the battery arrangement for passive gripper model

File: mbzirc2020/mbzirc2020_task2/mbzirc2020_task2_common/robots/hydrus_passive_gripper.urdf.xacro (robot description, xacro)
@@ -7,23 +7,45 @@
   <!-- special battery arrangement -->
   <xacro:extra_module name = "bat1" parent = "link1" visible = "1"
-                      model_url = "package://hydrus/urdf/mesh/battery/Kypom-3000-6s.dae" scale="0.001">
-    <origin xyz="${link_length/2} 0.0 -0.048" rpy="0 0 0"/>
-    <inertial>
-      <origin xyz="0 0 0" rpy="0 0 0"/>
-      <mass value="0.4108"/>
-      <inertia
-          ixx="0.0001" iyy="0.0006" izz="0.0006"
-          ixy="0.0" ixz="0.0"  iyz="0.0"/>
-    </inertial>
-  </xacro:extra_module>
-  <xacro:extra_module name = "bat2" parent = "link4" visible = "1"
-                      model_url = "package://hydrus/urdf/mesh/battery/Kypom-3000-6s.dae" scale="0.001">
-    <origin xyz="${link_length/2} 0.0 -0.048" rpy="0 0 0"/>
-    <inertial>
-      <origin xyz="0 0 0" rpy="0 0 0"/>
-      <mass value="0.4108"/>
-      <inertia
-          ixx="0.0001" iyy="0.0006" izz="0.0006"
-          ixy="0.0" ixz="0.0"  iyz="0.0"/>
+                      model_url = "package://hydrus/urdf/mesh/battery/VOLTON-PG-1300LP2-6s.stl" scale="0.001">
+    <origin xyz="${link_length/2} 0.0 -0.048" rpy="0 0 0"/>
+    <inertial>
+      <origin xyz="0 0 0" rpy="0 0 0"/>
+      <mass value="0.194"/>
+      <inertia
+          ixx="0.00005" iyy="0.00012" izz="0.00011"
+          ixy="0.0" ixz="0.0" iyz="0.0"/>
+    </inertial>
+  </xacro:extra_module>
+  <xacro:extra_module name = "bat2" parent = "link2" visible = "1"
+                      model_url = "package://hydrus/urdf/mesh/battery/VOLTON-PG-1300LP2-6s.stl" scale="0.001">
+    <origin xyz="${link_length/2} 0.0 -0.048" rpy="0 0 0"/>
+    <inertial>
+      <origin xyz="0 0 0" rpy="0 0 0"/>
+      <mass value="0.194"/>
+      <inertia
+          ixx="0.00005" iyy="0.00012" izz="0.00011"
+          ixy="0.0" ixz="0.0" iyz="0.0"/>
+    </inertial>
+  </xacro:extra_module>
+  <xacro:extra_module name = "bat3" parent = "link3" visible = "1"
+                      model_url = "package://hydrus/urdf/mesh/battery/VOLTON-PG-1300LP2-6s.stl" scale="0.001">
+    <origin xyz="${link_length/2} 0.0 -0.048" rpy="0 0 0"/>
+    <inertial>
+      <origin xyz="0 0 0" rpy="0 0 0"/>
+      <mass value="0.194"/>
+      <inertia
+          ixx="0.00005" iyy="0.00012" izz="0.00011"
+          ixy="0.0" ixz="0.0" iyz="0.0"/>
+    </inertial>
+  </xacro:extra_module>
+  <xacro:extra_module name = "bat4" parent = "link4" visible = "1"
+                      model_url = "package://hydrus/urdf/mesh/battery/VOLTON-PG-1300LP2-6s.stl" scale="0.001">
+    <origin xyz="${link_length/2} 0.0 -0.048" rpy="0 0 0"/>
+    <inertial>
+      <origin xyz="0 0 0" rpy="0 0 0"/>
+      <mass value="0.194"/>
+      <inertia
+          ixx="0.00005" iyy="0.00012" izz="0.00011"
+          ixy="0.0" ixz="0.0" iyz="0.0"/>
     </inertial>
   </xacro:extra_module>
