Commit message: update model with linear servo

File: mbzirc2020/mbzirc2020_task2/mbzirc2020_task2_common/robots/hydrus_ground_mode.gazebo.xacro (robot description, xacro)
@@ -6,5 +6,5 @@
   <!-- gazebo plugin for sensors -->
   <xacro:include filename="$(find mbzirc2020_common)/robots/default.gazebo.xacro" />
-  <gazebo reference="actuated_leg1_movable_part">
+  <gazebo reference="actuated_leg1_wheel">
     <mu1>0.11</mu1>
     <mu2>0.11</mu2>
@@ -13,5 +13,5 @@
     <selfCollide>false</selfCollide>
   </gazebo>
-  <gazebo reference="actuated_leg2_movable_part">
+  <gazebo reference="actuated_leg2_wheel">
     <mu1>0.11</mu1>
     <mu2>0.11</mu2>
@@ -20,5 +20,5 @@
     <selfCollide>false</selfCollide>
   </gazebo>
-  <gazebo reference="omni_leg1">
+  <gazebo reference="handmade_caster1_wheel">
     <mu1>0.11</mu1>
     <mu2>0.11</mu2>
@@ -27,5 +27,5 @@
     <selfCollide>false</selfCollide>
   </gazebo>
-  <gazebo reference="omni_leg2">
+  <gazebo reference="handmade_caster2_wheel">
     <mu1>0.11</mu1>
     <mu2>0.11</mu2>

File: mbzirc2020/mbzirc2020_task2/mbzirc2020_task2_common/robots/hydrus_ground_mode.urdf.xacro (robot description, xacro)
@@ -104,5 +104,5 @@
           iyy="0.0" iyz="0.0"
           izz="0.0"/>
-    </inertial>
+     </inertial>
   </xacro:extra_module>
   <!-- special battery arrangement -->
@@ -133,21 +133,21 @@
   <!-- in the second link -->
   <xacro:extra_module name = "actuated_leg1_stationary_part" parent = "link2" visible = "1"
-                      model_url = "package://mbzirc2020_task2_common/urdf/mesh/modules/mechanical/actuated_leg_servo.STL">
-    <origin xyz="${head_leg_offset+0.011} ${-0.028} -0.1024" rpy="${pi/2} 0 ${pi}"/>
-    <inertial>
-      <mass value = "0.142" />
-      <origin xyz="0 0 0" rpy="0 0 0"/>
-      <inertia
-          ixx="0.0001" ixy="0.0" ixz="0.0"
-          iyy="0.0001" iyz="0.0"
-          izz="0.0001"/>
+                      model_url = "package://mbzirc2020_task2_common/urdf/mesh/modules/mechanical/l16_100mm_in.STL">
+    <origin xyz="${head_leg_offset} -0.019 0.0186" rpy="${pi/2} 0 ${pi}"/>
+    <inertial>
+      <mass value = "0.0719" />
+      <origin xyz="0 0 0" rpy="0 0 0"/>
+      <inertia
+          ixx="0.000155" ixy="0.0" ixz="0.0"
+          iyy="0.000004" iyz="0.0"
+          izz="0.000154"/>
     </inertial>
   </xacro:extra_module>
   <joint name="actuated_leg1_joint" type="prismatic">
-    <limit effort="50" lower="0" upper="0.0927" velocity="1"/>
+    <limit effort="50" lower="0" upper="0.1" velocity="1"/>
     <parent link="actuated_leg1_stationary_part"/>
     <child link="actuated_leg1_movable_part"/>
-    <origin rpy="${-pi/2} 0 ${pi}" xyz="-0.0115 0 0"/> <!-- TODO: tune -y -->
-    <axis xyz="0 0 -1"/>
+    <origin rpy="0 0 0" xyz="0 -0.112 0"/>
+    <axis xyz="0 -1 0"/>
     <dynamics damping="0.1" friction="0.01"/>
   </joint>
@@ -164,20 +164,53 @@
   <link name="actuated_leg1_movable_part">
     <inertial>
-      <origin xyz="-0.002860 0.000000 -0.089840" rpy="0 0 0"/>
-      <mass value="0.107000"/>
-      <inertia
-          ixx="0.002466" iyy="0.003026" izz="0.000699"
-          ixy="0.000150" ixz="0.001147" iyz="0.000280"/>
-    </inertial>
-    <!-- <visual> -->
-    <!--   <origin xyz="0 0 0" rpy="${-pi/2} 0 0"/> -->
-    <!--   <geometry> -->
-    <!--     <mesh filename="package://mbzirc2020_task2_common/urdf/mesh/modules/mechanical/actuated_leg_movable_part.dae"/> -->
-    <!--   </geometry> -->
-    <!-- </visual> -->
-    <collision>
-      <origin rpy="0 0 0" xyz="0.0025 0 -0.128"/>
-      <geometry>
-        <sphere radius="${55 / 2 * 0.001}"/>
+      <origin xyz="0 0.000000 0" rpy="0 0 0"/>
+      <mass value="0.01871"/>
+      <inertia
+          ixx="0.0000320" iyy="0.0000308" izz="0.00000174"
+          ixy="0.000" ixz="0.000" iyz="0.000"/>
+    </inertial>
+    <visual>
+      <origin xyz="0 0 0" rpy="${-pi/2} ${pi*3/4} 0"/>
+      <geometry>
+        <mesh filename="package://mbzirc2020_task2_common/urdf/mesh/modules/mechanical/actuated_leg_pipe_mirror.STL"/>
+      </geometry>
+    </visual>
+    <collision>
+      <origin rpy="${pi/2} 0 0" xyz="0 ${0.1435/2-0.0435} 0"/>
+      <geometry>
+        <cylinder length="0.1435" radius="0.0045"/>
+      </geometry>
+    </collision>
+  </link>
+  <joint name="actuated_leg1_wheel_joint" type="fixed">
+    <parent link="actuated_leg1_movable_part"/>
+    <child link="actuated_leg1_wheel"/>
+    <axis xyz="0 1 0"/>
+    <origin xyz="${-0.00147/1.41421356237} -0.0375 ${-0.00147/1.41421356237}" rpy="${-pi/2} ${-pi/4} 0"/>
+  </joint>
+  <link name="actuated_leg1_wheel">
+    <inertial>
+      <origin xyz="0 0 0" rpy="0 0 0"/>
+      <mass value="0.05282"/>
+      <inertia
+          ixx="0.0000222" iyy="0.0000180" izz="0.0000222"
+          ixy="0.000000" ixz="0.000000" iyz="0.000000"/>
+    </inertial>
+    <visual>
+      <origin xyz="0 0 0" rpy="0 0 0"/>
+      <geometry>
+        <mesh filename="package://mbzirc2020_task2_common/urdf/mesh/modules/mechanical/actuated_leg_wheel.STL"/>
+      </geometry>
+    </visual>
+    <collision>
+      <origin rpy="${pi/2} 0 0" xyz="0 0.01435 0"/>
+      <geometry>
+        <cylinder length="0.008" radius="0.02816"/>
+      </geometry>
+    </collision>
+    <collision>
+      <origin rpy="${pi/2} 0 0" xyz="0 -0.01435 0"/>
+      <geometry>
+        <cylinder length="0.008" radius="0.02816"/>
       </geometry>
     </collision>
@@ -185,21 +218,21 @@
   <!-- in the thrid links -->
   <xacro:extra_module name = "actuated_leg2_stationary_part" parent = "link3" visible = "1"
-                      model_url = "package://mbzirc2020_task2_common/urdf/mesh/modules/mechanical/actuated_leg_stationary_part.dae">
-    <origin xyz="${end_leg_offset} 0.0 0" rpy="${-pi/2} 0 ${pi}"/>
-    <inertial>
-      <mass value = "0.142" />
-      <origin xyz="0 0 0" rpy="0 0 0"/>
-      <inertia
-          ixx="0.0001" ixy="0.0" ixz="0.0"
-          iyy="0.0001" iyz="0.0"
-          izz="0.0001"/>
+                      model_url = "package://mbzirc2020_task2_common/urdf/mesh/modules/mechanical/l16_100mm_in.STL">
+    <origin xyz="${end_leg_offset} -0.019 0.0186" rpy="${pi/2} 0 ${pi}"/>
+    <inertial>
+      <mass value = "0.0719" />
+      <origin xyz="0 0 0" rpy="0 0 0"/>
+      <inertia
+          ixx="0.000155" ixy="0.0" ixz="0.0"
+          iyy="0.000004" iyz="0.0"
+          izz="0.000154"/>
     </inertial>
   </xacro:extra_module>
   <joint name="actuated_leg2_joint" type="prismatic">
-    <limit effort="50" lower="0" upper="0.0927" velocity="1"/>
+    <limit effort="50" lower="0" upper="0.1" velocity="1"/>
     <parent link="actuated_leg2_stationary_part"/>
     <child link="actuated_leg2_movable_part"/>
-    <origin rpy="${-pi/2} 0 ${pi}" xyz="-0.0115 0 0"/> <!-- TODO: tune -y -->
-    <axis xyz="0 0 -1"/>
+    <origin rpy="0 0 0" xyz="0 -0.112 0"/>
+    <axis xyz="0 -1 0"/>
     <dynamics damping="0.1" friction="0.01"/>
   </joint>
@@ -216,20 +249,53 @@
   <link name="actuated_leg2_movable_part">
     <inertial>
-      <origin xyz="-0.002860 0.000000 -0.089840" rpy="0 0 0"/>
-      <mass value="0.107000"/>
-      <inertia
-          ixx="0.002466" iyy="0.003026" izz="0.000699"
-          ixy="0.000150" ixz="0.001147" iyz="0.000280"/>
-    </inertial>
-    <visual>
-      <origin xyz="0 0 0" rpy="${-pi/2} 0 0"/>
-      <geometry>
-        <mesh filename="package://mbzirc2020_task2_common/urdf/mesh/modules/mechanical/actuated_leg_movable_part.dae"/>
-      </geometry>
-    </visual>
-    <collision>
-      <origin rpy="0 0 0" xyz="0.0025 0 -0.128"/>
-      <geometry>
-        <sphere radius="${55 / 2 * 0.001}"/>
+      <origin xyz="0 0 0" rpy="0 0 0"/>
+      <mass value="0.01871"/>
+      <inertia
+          ixx="0.0000320" iyy="0.0000308" izz="0.00000174"
+          ixy="0.000" ixz="0.000" iyz="0.000"/>
+    </inertial>
+    <visual>
+      <origin xyz="0 0 0" rpy="${-pi/2} ${-pi*3/4} 0"/>
+      <geometry>
+        <mesh filename="package://mbzirc2020_task2_common/urdf/mesh/modules/mechanical/actuated_leg_pipe.STL"/>
+      </geometry>
+    </visual>
+    <collision>
+      <origin rpy="${pi/2} 0 0" xyz="0 ${0.1435/2-0.0435} 0"/>
+      <geometry>
+        <cylinder length="0.1435" radius="0.0045"/>
+      </geometry>
+    </collision>
+  </link>
+  <joint name="actuated_leg2_wheel_joint" type="fixed">
+    <parent link="actuated_leg2_movable_part"/>
+    <child link="actuated_leg2_wheel"/>
+    <axis xyz="0 1 0"/>
+    <origin xyz="${0.00147/1.41421356237} -0.0375 ${-0.00147/1.41421356237}" rpy="${-pi/2} ${-pi*3/4} 0"/>
+  </joint>
+  <link name="actuated_leg2_wheel">
+    <inertial>
+      <origin xyz="0 0 0" rpy="0 0 0"/>
+      <mass value="0.05282"/>
+      <inertia
+          ixx="0.0000222" iyy="0.0000180" izz="0.0000222"
+          ixy="0.000000" ixz="0.000000" iyz="0.000000"/>
+    </inertial>
+    <visual>
+      <origin xyz="0 0 0" rpy="0 0 0"/>
+      <geometry>
+        <mesh filename="package://mbzirc2020_task2_common/urdf/mesh/modules/mechanical/actuated_leg_wheel.STL"/>
+      </geometry>
+    </visual>
+    <collision>
+      <origin rpy="${pi/2} 0 0" xyz="0 0.01435 0"/>
+      <geometry>
+        <cylinder length="0.008" radius="0.02816"/>
+      </geometry>
+    </collision>
+    <collision>
+      <origin rpy="${pi/2} 0 0" xyz="0 -0.01435 0"/>
+      <geometry>
+        <cylinder length="0.008" radius="0.02816"/>
       </geometry>
     </collision>
@@ -244,5 +310,5 @@
   <link name="handmade_caster1_pipe">
     <inertial>
-      <origin xyz="0.000000 0.000000 -0.093340" rpy="0 0 0"/>
+      <origin xyz="0 0 0" rpy="0 0 0"/>
       <mass value="0.012000"/>
       <inertia
@@ -269,7 +335,17 @@
     <origin xyz="0.0 0.0 -0.131" rpy="0 0 0"/>
   </joint>
+  <transmission name="handmade_caster1_pipe_to_connector_joint_tran">
+    <type>transmission_interface/SimpleTransmission</type>
+    <joint name="handmade_caster1_pipe_to_connector_joint">
+      <hardwareInterface>hardware_interface/EffortJointInterface</hardwareInterface>
+    </joint>
+    <actuator name="handmade_caster1_pipe_to_connector_joint">
+      <hardwareInterface>hardware_interface/EffortJointInterface</hardwareInterface>
+      <mechanicalReduction>1</mechanicalReduction>
+    </actuator>
+  </transmission>
   <link name="handmade_caster1_connector">
     <inertial>
-      <origin xyz="0.000000 0.000000 -0.093340" rpy="0 0 0"/>
+      <origin xyz="0 0 0" rpy="0 0 0"/>
       <mass value="0.009"/>
       <inertia
@@ -284,5 +360,5 @@
     </visual>
   </link>
-    <joint name="handmade_caster1_connector_to_wheel_joint" type="continuous">
+  <joint name="handmade_caster1_connector_to_wheel_joint" type="fixed">
     <parent link="handmade_caster1_connector"/>
     <child link="handmade_caster1_wheel"/>
@@ -292,5 +368,5 @@
   <link name="handmade_caster1_wheel">
     <inertial>
-      <origin xyz="0.000000 0.000000 -0.093340" rpy="0 0 0"/>
+      <origin xyz="0.000000 0.000000 0.000000" rpy="0 0 0"/>
       <mass value="0.056"/>
       <inertia
@@ -344,4 +420,14 @@
     <origin xyz="0.0 0.0 -0.131" rpy="0 0 0"/>
   </joint>
+  <transmission name="handmade_caster2_pipe_to_connector_joint_tran">
+    <type>transmission_interface/SimpleTransmission</type>
+    <joint name="handmade_caster2_pipe_to_connector_joint">
+      <hardwareInterface>hardware_interface/EffortJointInterface</hardwareInterface>
+    </joint>
+    <actuator name="handmade_caster2_pipe_to_connector_joint">
+      <hardwareInterface>hardware_interface/EffortJointInterface</hardwareInterface>
+      <mechanicalReduction>1</mechanicalReduction>
+    </actuator>
+  </transmission>
   <link name="handmade_caster2_connector">
     <inertial>
@@ -359,5 +445,5 @@
     </visual>
   </link>
-    <joint name="handmade_caster2_connector_to_wheel_joint" type="continuous">
+  <joint name="handmade_caster2_connector_to_wheel_joint" type="fixed">
     <parent link="handmade_caster2_connector"/>
     <child link="handmade_caster2_wheel"/>

Commit message: add realsense to hydrus ground model

File: mbzirc2020/mbzirc2020_task2/mbzirc2020_task2_common/robots/hydrus_ground_mode.gazebo.xacro (robot description, xacro)
@@ -34,5 +34,122 @@
     <selfCollide>false</selfCollide>
   </gazebo>
-  <!-- TODO: gazebo for Realsense D435 -->
+    <!-- gazebo for Realsense D435 -->
+  <!--  The following values model the aluminum peripherial case for the
+        D435 camera, with the camera joint represented by the actual
+        peripherial camera tripod mount -->
+  <xacro:property name="d435_cam_depth_to_left_ir_offset" value="0.0"/>
+  <xacro:property name="d435_cam_depth_to_right_ir_offset" value="-0.050"/>
+  <xacro:property name="d435_cam_depth_to_color_offset" value="0.015"/>
+  <xacro:property name="d435_cam_width" value="0.090"/>
+  <xacro:property name="d435_cam_height" value="0.025"/>
+  <xacro:property name="d435_cam_depth" value="0.02505"/>
+  <xacro:property name="d435_cam_mount_from_center_offset" value="0.0149"/>
+  <!--  The following offset is relative the the physical D435 camera peripherial
+        camera tripod mount -->
+  <xacro:property name="d435_cam_depth_px" value="${d435_cam_mount_from_center_offset}"/>
+  <xacro:property name="d435_cam_depth_py" value="0.0175"/>
+  <xacro:property name="d435_cam_depth_pz" value="${d435_cam_height/2}"/>
+  <material name="aluminum">
+    <color rgba="0.5 0.5 0.5 1"/>
+  </material>
+  <!-- camera depth joints and links -->
+  <joint name="rs_d435_depth_joint" type="fixed">
+    <origin xyz="0 0 0" rpy="0 0 0"/>
+    <parent link="rs_d435_link"/>
+    <child link="rs_d435_depth_frame" />
+  </joint>
+  <link name="rs_d435_depth_frame"/>
+  <joint name="rs_d435_depth_optical_joint" type="fixed">
+    <origin xyz="0 0 0" rpy="${-pi/2} 0 ${-pi/2}" />
+    <parent link="rs_d435_depth_frame" />
+    <child link="rs_d435_depth_optical_frame" />
+  </joint>
+  <link name="rs_d435_depth_optical_frame"/>
+  <!-- camera left IR joints and links -->
+  <joint name="rs_d435_left_ir_joint" type="fixed">
+    <origin xyz="0 ${d435_cam_depth_to_left_ir_offset} 0" rpy="0 0 0" />
+    <parent link="rs_d435_depth_frame" />
+    <child link="rs_d435_left_ir_frame" />
+  </joint>
+  <link name="rs_d435_left_ir_frame"/>
+  <joint name="rs_d435_left_ir_optical_joint" type="fixed">
+    <origin xyz="0 0 0" rpy="${-pi/2} 0 ${-pi/2}" />
+    <parent link="rs_d435_left_ir_frame" />
+    <child link="rs_d435_left_ir_optical_frame" />
+  </joint>
+  <link name="rs_d435_left_ir_optical_frame"/>
+  <!-- camera right IR joints and links -->
+  <joint name="rs_d435_right_ir_joint" type="fixed">
+    <origin xyz="0 ${d435_cam_depth_to_right_ir_offset} 0" rpy="0 0 0" />
+    <parent link="rs_d435_depth_frame" />
+    <child link="rs_d435_right_ir_frame" />
+  </joint>
+  <link name="rs_d435_right_ir_frame"/>
+  <joint name="rs_d435_right_ir_optical_joint" type="fixed">
+    <origin xyz="0 0 0" rpy="${-pi/2} 0 ${-pi/2}" />
+    <parent link="rs_d435_right_ir_frame" />
+    <child link="rs_d435_right_ir_optical_frame" />
+  </joint>
+  <link name="rs_d435_right_ir_optical_frame"/>
+  <!-- camera color joints and links -->
+  <joint name="rs_d435_color_joint" type="fixed">
+    <origin xyz="0 ${d435_cam_depth_to_color_offset} 0" rpy="0 0 0" />
+    <parent link="rs_d435_depth_frame" />
+    <child link="rs_d435_color_frame" />
+  </joint>
+  <link name="rs_d435_color_frame"/>
+  <joint name="rs_d435_color_optical_joint" type="fixed">
+    <origin xyz="0 0 0" rpy="${-pi/2} 0 ${-pi/2}" />
+    <parent link="rs_d435_color_frame" />
+    <child link="rs_d435_color_optical_frame" />
+  </joint>
+  <link name="rs_d435_color_optical_frame"/>
+  <!-- gazebo plugin -->
+  <gazebo reference="rs_d435_color_frame">
+    <sensor type="depth" name="rs_d435_camera">
+      <update_rate>10.0</update_rate>
+      <camera name="head">
+	<horizontal_fov>1.59174</horizontal_fov>
+	<vertical_fov>1.14319</vertical_fov>
+	<image>
+	  <width>1280</width>
+	  <height>720</height>
+	  <format>RGB</format>
+	</image>
+	<clip>
+	  <near>0.02</near>
+	  <far>300</far>
+	</clip>
+	<noise>
+	  <type>gaussian</type>
+	  <mean>0.0</mean>
+	  <stddev>0.007</stddev>
+	</noise>
+      </camera>
+      <plugin name="depth_camera" filename="libgazebo_ros_openni_kinect.so">
+	<baseline>0.06</baseline>
+	<alwaysOn>true</alwaysOn>
+	<updateRate>0.0</updateRate>
+	<cameraName>rs_d435</cameraName>
+	<imageTopicName>color/image_rect_color</imageTopicName>
+	<cameraInfoTopicName>color/camera_info</cameraInfoTopicName>
+	<depthImageCameraInfoTopicName>aligned_depth_to_color/camera_info</depthImageCameraInfoTopicName>
+	<depthImageTopicName>aligned_depth_to_color/image_raw</depthImageTopicName>
+	<pointCloudTopicName>depth_registered/points</pointCloudTopicName>
+	<frameName>rs_d435_color_optical_frame</frameName>
+	<pointCloudCutoff>0.05</pointCloudCutoff>
+	<distortionK1>0</distortionK1>
+	<distortionK2>0</distortionK2>
+	<distortionK3>0</distortionK3>
+	<distortionT1>0</distortionT1>
+	<distortionT2>0</distortionT2>
+	<CxPrime>0</CxPrime>
+	<Cx>0</Cx>
+	<Cy>0</Cy>
+	<focalLength>0</focalLength>
+	<hackBaseline>0</hackBaseline>
+      </plugin>
+    </sensor>
+  </gazebo>
   <!-- gazebo grasp plugin -->
   <xacro:include filename="$(find mbzirc2020_task2_simulation)/urdf/gzplugin_grasp_fix.urdf.xacro" />

File: mbzirc2020/mbzirc2020_task2/mbzirc2020_task2_common/robots/hydrus_ground_mode.urdf.xacro (robot description, xacro)
@@ -106,4 +106,66 @@
      </inertial>
   </xacro:extra_module>
+  <!-- 2.4 Realsense D435 -->
+  <!-- TODO: accurate intertia parameters and position -->
+  <xacro:extra_module name = "rs_d435_mount" parent = "link2" visible = "1"
+                      model_url = "package://mbzirc2020_common/urdf/mesh/modules/sensor/rs_d435_unit2.STL">
+    <origin xyz="${link_length / 2} 0 0" rpy="0 0 0"/>
+    <inertial>
+      <mass value = "0.0" />
+      <origin xyz="0 0 0" rpy="0 0 0"/>
+      <inertia
+          ixx="0.0" ixy="0.0" ixz="0.0"
+          iyy="0.0" iyz="0.0" izz="0.0"/>
+    </inertial>
+  </xacro:extra_module>
+  <joint name="rs_d435_servo_joint" type="revolute">
+    <limit effort="0.2" lower="0" upper="1.8" velocity="0.1"/>
+    <parent link="link2"/>
+    <child link="rs_d435_servo"/>
+    <origin xyz="${link_length / 2 + 0.20395} 0.02495 -0.038" rpy="0 0 ${pi/4}"/>
+    <axis xyz="-1 0 0"/>
+    <dynamics damping="0.01" friction="0.0"/>
+  </joint>
+  <link name="rs_d435_servo">
+    <inertial>
+      <mass value = "0" />
+      <origin xyz="0 0 0" rpy="0 0 0"/>
+      <inertia
+          ixx="0.0" ixy="0.0" ixz="0.0"
+          iyy="0.0" iyz="0.0" izz="0.0"/>
+    </inertial>
+  </link>
+  <xacro:extra_module name = "rs_d435_unit" parent = "rs_d435_servo" visible = "1" model_url = "package://mbzirc2020_common/urdf/mesh/modules/sensor/rs_d435_unit1.STL">
+    <origin xyz="0.05275 0.01005 0" rpy="0 0 ${pi / 2}"/>
+    <inertial>
+      <mass value = "0.124" /> <!-- includes usb cable, servo, mounts -->
+      <origin xyz="-0.01005 0 0" rpy="0 0 0"/>
+      <inertia
+          ixx="0.0001" iyy="0.0001" izz="0.0002"
+          ixy="0" ixz="0" iyz="0"/>
+    </inertial>
+  </xacro:extra_module>
+  <!-- rs_d435_link is the parrent of sensors' frame, identical to rs_d435_left_ir_frame  -->
+  <xacro:extra_module name = "rs_d435_link" parent = "rs_d435_unit" visible = "0" >
+    <origin xyz="-0.008 0.0175 0 " rpy="0 0 0"/>
+    <inertial>
+      <mass value = "0.0" />
+      <origin xyz="0 0 0" rpy="0 0 0"/>
+      <inertia
+	  ixx="0.0" ixy="0.0" ixz="0.0"
+	  iyy="0.0" iyz="0.0"
+	  izz="0.0"/>
+    </inertial>
+  </xacro:extra_module>
+  <transmission name="rs_d435_servo_joint_tran">
+    <type>transmission_interface/SimpleTransmission</type>
+    <joint name="rs_d435_servo_joint">
+      <hardwareInterface>hardware_interface/EffortJointInterface</hardwareInterface>
+    </joint>
+    <actuator name="rs_d435_servo_joint">
+      <hardwareInterface>hardware_interface/EffortJointInterface</hardwareInterface>
+      <mechanicalReduction>1</mechanicalReduction>
+    </actuator>
+  </transmission>
   <!-- special battery arrangement -->
   <xacro:extra_module name = "bat1" parent = "link1" visible = "1"
