Commit message: [mbzirc2020_task2_common] change the length of leg in hydrus_ring_gripper model

File: mbzirc2020/mbzirc2020_task2/mbzirc2020_task2_common/robots/hydrus_ring_gripper.urdf.xacro (robot description, xacro)
@@ -4,5 +4,5 @@
   <!-- base kinematics model -->
   <xacro:include filename="$(find mbzirc2020_common)/robots/default.urdf.xacro" />
-  <xacro:robot_model tilt_angle = "10" downward_vio = "0" horizontal_vio = "0" default_battery = "0"  />
+  <xacro:robot_model tilt_angle = "10" downward_vio = "0" horizontal_vio = "0" default_battery = "0" with_leg="0"  />
   <!-- special battery arrangement -->
   <xacro:extra_module name = "bat1" parent = "link1" visible = "1"
@@ -163,4 +163,53 @@
     </collision>
   </link>
+  ##### leg #####
+  <xacro:standard_leg_end parent = "link1" self="1">
+    <origin xyz="${head_leg_offset} 0.0 0" rpy="0 0 0"/>
+  </xacro:standard_leg_end>
+  <xacro:standard_leg_joint parent = "link1" self="2">
+    <origin xyz="0.6 0.0 0" rpy="0 0 0"/>
+  </xacro:standard_leg_joint>
+  <xacro:standard_leg_joint parent = "link4" self="3">
+    <origin xyz="0.0 0.0 0" rpy="0 0 0"/>
+  </xacro:standard_leg_joint>
+  <xacro:standard_leg_end parent = "link4" self="4">
+    <origin xyz="${end_leg_offset} 0.0 0" rpy="0 0 0"/>
+  </xacro:standard_leg_end>
+  <xacro:macro name="leg_collision_model" params="name parent *origin">
+    <joint name="${parent}2${name}" type="fixed">
+      <parent link="${parent}"/>
+      <child link="${name}"/>
+      <xacro:insert_block name="origin" />
+    </joint>
+    <link name="${name}">
+      <inertial>
+        <mass value = "0.00001" />
+        <origin xyz="0.0 0.0 0.0" rpy="0 0 0"/>
+        <inertia
+            ixx="0.000001" ixy="0.000000" ixz="0.0000000"
+            iyy="0.000001" iyz="0.000000" izz="0.000001"/>
+      </inertial>
+      <collision>
+        <geometry>
+          <box size="0.05 0.05 0.09"/>
+        </geometry>
+      </collision>
+    </link>
+  </xacro:macro>
+  <xacro:leg_collision_model name = "leg_collision_model1" parent = "leg1">
+    <origin xyz="0 0 -0.05" rpy="0 0 0"/>
+  </xacro:leg_collision_model>
+  <xacro:leg_collision_model name = "leg_collision_model2" parent = "leg2">
+    <origin xyz="0 0 -0.05" rpy="0 0 0"/>
+  </xacro:leg_collision_model>
+  <xacro:leg_collision_model name = "leg_collision_model3" parent = "leg3">
+    <origin xyz="0 0 -0.05" rpy="0 0 0"/>
+  </xacro:leg_collision_model>
+  <xacro:leg_collision_model name = "leg_collision_model4" parent = "leg4">
+    <origin xyz="0 0 -0.05" rpy="0 0 0"/>
+  </xacro:leg_collision_model>
+  <xacro:leg_collision_model name = "leg_collision_model5" parent = "link3">
+    <origin xyz="0 0 -0.05" rpy="0 0 0"/>
+  </xacro:leg_collision_model>
   <transmission name="rs_d435_servo_joint_tran">
     <type>transmission_interface/SimpleTransmission</type>

Commit message: [mbzirc2020_task2_common] update ring gripper model

File: mbzirc2020/mbzirc2020_task2/mbzirc2020_task2_common/robots/hydrus_ring_gripper.urdf.xacro (robot description, xacro)
@@ -118,9 +118,9 @@
   <link name="ring_gripper_left">
     <inertial>
-      <mass value = "0.0733147" />
-      <origin xyz="0.0000000 0.1954388 0.0039469" rpy="0 0 0"/>
-      <inertia
-          ixx="0.0000290" ixy="0.0000000" ixz="0.0000000"
-          iyy="0.0002193" iyz="0.0000001" izz="0.0002130"/>
+      <mass value = "0.086507" />
+      <origin xyz="0.0000000 0.196326 -0.020803" rpy="0 0 0"/>
+      <inertia
+          ixx="0.000072" ixy="0.0000000" ixz="0.0000000"
+          iyy="0.000274" iyz="-0.000013" izz="0.000226"/>
     </inertial>
     <visual>
@@ -144,9 +144,9 @@
   <link name="ring_gripper_right">
     <inertial>
-      <mass value = "0.0733147" />
-      <origin xyz="0.0000000 0.1954388 0.0039469" rpy="0 0 0"/>
-      <inertia
-          ixx="0.0000290" ixy="0.0000000" ixz="0.0000000"
-          iyy="0.0002193" iyz="0.0000001" izz="0.0002130"/>
+      <mass value = "0.086507" />
+      <origin xyz="0.0000000 0.196326 -0.020803" rpy="0 0 0"/>
+      <inertia
+          ixx="0.000072" ixy="0.0000000" ixz="0.0000000"
+          iyy="0.000274" iyz="-0.000013" izz="0.000226"/>
     </inertial>
     <visual>

Commit message: [mbzirc2020_task2_common] update ring gripper model

File: mbzirc2020/mbzirc2020_task2/mbzirc2020_task2_common/robots/hydrus_ring_gripper.urdf.xacro (robot description, xacro)
@@ -4,5 +4,6 @@
   <!-- base kinematics model -->
   <xacro:include filename="$(find mbzirc2020_common)/robots/default.urdf.xacro" />
-  <xacro:robot_model tilt_angle = "10" downward_vio = "0" horizontal_vio = "0" default_battery = "0" with_leg="0"  />
+  <xacro:property name="modified_leg_collision_model_height" value="0.1715"/>
+  <xacro:robot_model tilt_angle = "10" downward_vio = "0" horizontal_vio = "0" default_battery = "0" with_leg="0" />
   <!-- special battery arrangement -->
   <xacro:extra_module name = "bat1" parent = "link2" visible = "1"
@@ -118,5 +119,5 @@
   <link name="ring_gripper_left">
     <inertial>
-      <mass value = "0.086507" />
+      <mass value = "0.106" />
       <origin xyz="0.0000000 0.196326 -0.020803" rpy="0 0 0"/>
       <inertia
@@ -148,5 +149,5 @@
   <link name="ring_gripper_right">
     <inertial>
-      <mass value = "0.086507" />
+      <mass value = "0.106" />
       <origin xyz="0.0000000 0.196326 -0.020803" rpy="0 0 0"/>
       <inertia
@@ -200,5 +201,5 @@
       <collision>
         <geometry>
-          <box size="0.05 0.05 ${leg_collision_model_height}"/>
+          <box size="0.05 0.05 ${modified_leg_collision_model_height}"/>
         </geometry>
       </collision>
@@ -206,17 +207,17 @@
   </xacro:macro>
   <xacro:leg_collision_model name = "leg_collision_model1" parent = "leg1">
-    <origin xyz="0 0 ${-leg_collision_model_height / 2}" rpy="0 0 0"/>
+    <origin xyz="0 0 ${-modified_leg_collision_model_height / 2}" rpy="0 0 0"/>
   </xacro:leg_collision_model>
   <xacro:leg_collision_model name = "leg_collision_model2" parent = "leg2">
-    <origin xyz="0 0 ${-leg_collision_model_height / 2}" rpy="0 0 0"/>
+    <origin xyz="0 0 ${-modified_leg_collision_model_height / 2}" rpy="0 0 0"/>
   </xacro:leg_collision_model>
   <xacro:leg_collision_model name = "leg_collision_model3" parent = "leg3">
-    <origin xyz="0 0 ${-leg_collision_model_height / 2}" rpy="0 0 0"/>
+    <origin xyz="0 0 ${-modified_leg_collision_model_height / 2}" rpy="0 0 0"/>
   </xacro:leg_collision_model>
   <xacro:leg_collision_model name = "leg_collision_model4" parent = "leg4">
-    <origin xyz="0 0 ${-leg_collision_model_height / 2}" rpy="0 0 0"/>
+    <origin xyz="0 0 ${-modified_leg_collision_model_height / 2}" rpy="0 0 0"/>
   </xacro:leg_collision_model>
   <xacro:leg_collision_model name = "leg_collision_model5" parent = "link3">
-    <origin xyz="0 0 ${-leg_collision_model_height / 2}" rpy="0 0 0"/>
+    <origin xyz="0 0 ${-modified_leg_collision_model_height / 2}" rpy="0 0 0"/>
   </xacro:leg_collision_model>
   <transmission name="rs_d435_servo_joint_tran">

Commit message: [mbzirc2020_task2_common] add battery arrangement argument in ring gripper model

File: mbzirc2020/mbzirc2020_task2/mbzirc2020_task2_common/robots/hydrus_ring_gripper.urdf.xacro (robot description, xacro)
@@ -4,29 +4,32 @@
   <!-- base kinematics model -->
   <xacro:include filename="$(find mbzirc2020_common)/robots/default.urdf.xacro" />
+  <xacro:arg name="default_battery" default="1"/>
   <xacro:property name="modified_leg_collision_model_height" value="0.1715"/>
-  <xacro:robot_model tilt_angle = "10" downward_vio = "0" horizontal_vio = "0" default_battery = "0" with_leg="0" />
+  <xacro:robot_model tilt_angle = "10" downward_vio = "0" horizontal_vio = "0" default_battery = "$(arg default_battery)" with_leg="0" />
   <!-- special battery arrangement -->
-  <xacro:extra_module name = "bat1" parent = "link2" visible = "1"
-                      model_url = "package://hydrus/urdf/mesh/battery/Kypom-3000-6s.dae" scale="0.001">
-    <origin xyz="${link_length/2} 0.0 -0.048" rpy="0 0 0"/>
-    <inertial>
-      <origin xyz="0 0 0" rpy="0 0 0"/>
-      <mass value="0.4108"/>
-      <inertia
-          ixx="0.0001" iyy="0.0006" izz="0.0006"
-          ixy="0.0" ixz="0.0"  iyz="0.0"/>
-    </inertial>
-  </xacro:extra_module>
-  <xacro:extra_module name = "bat2" parent = "link3" visible = "1"
-                      model_url = "package://hydrus/urdf/mesh/battery/Kypom-3000-6s.dae" scale="0.001">
-    <origin xyz="${link_length/2} 0.0 -0.048" rpy="0 0 0"/>
-    <inertial>
-      <origin xyz="0 0 0" rpy="0 0 0"/>
-      <mass value="0.4108"/>
-      <inertia
-          ixx="0.0001" iyy="0.0006" izz="0.0006"
-          ixy="0.0" ixz="0.0"  iyz="0.0"/>
-    </inertial>
-  </xacro:extra_module>
+  <xacro:if value="${$(arg default_battery) == 0}">
+    <xacro:extra_module name = "bat1" parent = "link2" visible = "1"
+                        model_url = "package://hydrus/urdf/mesh/battery/Kypom-3000-6s.dae" scale="0.001">
+      <origin xyz="${link_length/2} 0.0 -0.048" rpy="0 0 0"/>
+      <inertial>
+        <origin xyz="0 0 0" rpy="0 0 0"/>
+        <mass value="0.4108"/>
+        <inertia
+            ixx="0.0001" iyy="0.0006" izz="0.0006"
+            ixy="0.0" ixz="0.0"  iyz="0.0"/>
+      </inertial>
+    </xacro:extra_module>
+    <xacro:extra_module name = "bat2" parent = "link3" visible = "1"
+                        model_url = "package://hydrus/urdf/mesh/battery/Kypom-3000-6s.dae" scale="0.001">
+      <origin xyz="${link_length/2} 0.0 -0.048" rpy="0 0 0"/>
+      <inertial>
+        <origin xyz="0 0 0" rpy="0 0 0"/>
+        <mass value="0.4108"/>
+        <inertia
+            ixx="0.0001" iyy="0.0006" izz="0.0006"
+            ixy="0.0" ixz="0.0"  iyz="0.0"/>
+      </inertial>
+    </xacro:extra_module>
+  </xacro:if>
   <!-- processor: intel upboard -->
   <!-- TODO: change to brix -->
