Commit message: Fix the model and configuration about sensor servo in task2

File: mbzirc2020/mbzirc2020_task2/mbzirc2020_task2_common/robots/hydrus.urdf.xacro (robot description, xacro)
@@ -72,10 +72,10 @@
   </xacro:extra_module>
   <joint name="rs_d435_servo_joint" type="revolute">
-    <limit effort="0.2" lower="0" upper="1.6" velocity="0.5"/>
+    <limit effort="0.2" lower="0" upper="1.8" velocity="0.1"/>
     <parent link="link2"/>
     <child link="rs_d435_servo"/>
     <origin xyz="${link_length / 2 + 0.20395} 0.02495 -0.038" rpy="0 0 ${pi/4}"/>
     <axis xyz="-1 0 0"/>
-    <dynamics damping="0.2" friction="0.0"/>
+    <dynamics damping="0.01" friction="0.0"/>
   </joint>
   <link name="rs_d435_servo">
@@ -94,6 +94,6 @@
       <origin xyz="-0.01005 0 0" rpy="0 0 0"/>
       <inertia
-          ixx="0.00006" ixy="0.0" ixz="0.00006"
-          iyy="0.0" iyz="0.0" izz="0.0"/>
+          ixx="0.0001" iyy="0.0001" izz="0.0002"
+          ixy="0" ixz="0" iyz="0"/>
     </inertial>
   </xacro:extra_module>

Commit message: Change the weight of the upboard becuase of the new wifi

File: mbzirc2020/mbzirc2020_task2/mbzirc2020_task2_common/robots/hydrus.urdf.xacro (robot description, xacro)
@@ -35,5 +35,5 @@
     <origin xyz="${link_length / 2 + 0.2845} 0.011 0.016" rpy="0 0 ${pi}"/>
     <inertial>
-      <mass value = "0.117" />
+      <mass value = "0.122" />
       <origin xyz="${21 * 0.001} ${4 * 0.001} ${12 * 0.001}" rpy="0 0 0"/>
       <inertia

File: mbzirc2020/mbzirc2020_task2/mbzirc2020_task2_common/robots/hydrus_ground_mode.urdf.xacro (robot description, xacro)
@@ -46,5 +46,5 @@
     <origin xyz="${link_length / 2 + 0.2845} 0.011 0.016" rpy="0 0 ${pi}"/>
     <inertial>
-      <mass value = "0.117" />
+      <mass value = "0.122" />
       <origin xyz="${21 * 0.001} ${4 * 0.001} ${12 * 0.001}" rpy="0 0 0"/>
       <inertia

File: mbzirc2020/mbzirc2020_task3/mbzirc2020_task3_common/robots/hydrus.urdf.xacro (robot description, xacro)
@@ -34,5 +34,5 @@
     <origin xyz="${link_length / 2 + 0.2845} 0.011 0.016" rpy="0 0 ${pi}"/>
     <inertial>
-      <mass value = "0.120" />
+      <mass value = "0.122" />
       <origin xyz="${21 * 0.001} ${4 * 0.001} ${12 * 0.001}" rpy="0 0 0"/>
       <inertia
