Commit message: [mbzirc2020_task2_common] add joint friction and dumping in hydrus_ball_joint_gripper.urdf.xacro

File: mbzirc2020/mbzirc2020_task2/mbzirc2020_task2_common/robots/hydrus_ball_joint_gripper.urdf.xacro (robot description, xacro)
@@ -231,4 +231,5 @@
     <axis xyz="1 0 0"/>
     <limit lower="0" upper="0" effort="0" velocity="0"/>
+    <dynamics damping="0.2" friction="0.02"/>
   </joint>
   <link name="ball_joint12_left">
@@ -253,4 +254,5 @@
     <axis xyz="1 0 0"/>
     <limit lower="-0.4363" upper="0.4363" effort="100" velocity="100"/>
+    <dynamics damping="0.2" friction="0.02"/>
   </joint>
   <link name="dummy_left">
@@ -268,4 +270,5 @@
     <axis xyz="0 0 1"/>
     <limit lower="-0.4363" upper="0.4363" effort="100" velocity="100"/>
+    <dynamics damping="0.2" friction="0.02"/>
   </joint>
   <link name="dummy2_left">
@@ -283,4 +286,5 @@
     <axis xyz="0 1 0"/>
     <limit effort="100" velocity="100"/>
+    <dynamics damping="0.2" friction="0.02"/>
   </joint>
   <link name="ball_joint2_left">
@@ -303,4 +307,5 @@
     <child link="circle_gripper_left"/>
     <origin xyz="-0.068 0.04 -0.068" rpy="0 0 0"/>
+    <dynamics damping="0.2" friction="0.02"/>
   </joint>
   <link name="circle_gripper_left">
@@ -334,4 +339,5 @@
     <axis xyz="1 0 0"/>
     <limit lower="0" upper="0" effort="0" velocity="0"/>
+    <dynamics damping="0.2" friction="0.02"/>
   </joint>
   <link name="dummy_gripper_left">
@@ -385,4 +391,5 @@
     <axis xyz="1 0 0"/>
     <limit lower="0" upper="0" effort="0" velocity="0"/>
+    <dynamics damping="0.2" friction="0.02"/>
   </joint>
   <link name="ball_joint12_right">
@@ -407,4 +414,5 @@
     <axis xyz="1 0 0"/>
     <limit lower="-0.4363" upper="0.4363" effort="100" velocity="100"/>
+    <dynamics damping="0.2" friction="0.02"/>
   </joint>
   <link name="dummy_right">
@@ -422,4 +430,5 @@
     <axis xyz="0 0 1"/>
     <limit lower="-0.4363" upper="0.4363" effort="100" velocity="100"/>
+    <dynamics damping="0.2" friction="0.02"/>
   </joint>
   <link name="dummy2_right">
@@ -437,4 +446,5 @@
     <axis xyz="0 1 0"/>
     <limit effort="100" velocity="100"/>
+    <dynamics damping="0.2" friction="0.02"/>
   </joint>
   <link name="ball_joint2_right">
@@ -485,4 +495,5 @@
     <axis xyz="1 0 0"/>
     <limit lower="0" upper="0" effort="0" velocity="0"/>
+    <dynamics damping="0.2" friction="0.02"/>
   </joint>
   <link name="dummy_gripper_right">
