Commit message: MBZIRC2020 Task1: 1. update the battery arragement (four bat -> two bat) 2. fix the wrong camera image format in gazebo
MBZIRC2020 Task3:
1. fix the wrong camera image format in gazebo
2. fix the CMakeLists.txt

File: mbzirc2020/mbzirc2020_task1/mbzirc2020_task1_common/robots/hydrus.gazebo.xacro (robot description, xacro)
@@ -16,5 +16,5 @@
           <width>1280</width>
           <height>720</height>
-          <format>RGB</format>
+          <format>B8G8R8</format>
         </image>
         <clip>

File: mbzirc2020/mbzirc2020_task1/mbzirc2020_task1_common/robots/hydrus.urdf.xacro (robot description, xacro)
@@ -4,5 +4,28 @@
   <!-- base kinematics model -->
   <xacro:include filename="$(find mbzirc2020_common)/robots/default.urdf.xacro" />
-  <xacro:robot_model tilt_angle = "10" horizontal_vio = "0"  />
+  <xacro:robot_model tilt_angle = "10" horizontal_vio = "0"  default_battery = "0"/>
+  <!-- special battery arrangement -->
+  <xacro:extra_module name = "bat1" parent = "link1" visible = "1"
+                      model_url = "package://hydrus/urdf/mesh/battery/Kypom-3000-6s.dae">
+    <origin xyz="${link_length/2} 0.0 -0.048" rpy="0 0 0"/>
+    <inertial>
+      <origin xyz="0 0 0" rpy="0 0 0"/>
+      <mass value="0.4108"/>
+      <inertia
+          ixx="0.0001" iyy="0.0006" izz="0.0006"
+          ixy="0.0" ixz="0.0"  iyz="0.0"/>
+    </inertial>
+  </xacro:extra_module>
+  <xacro:extra_module name = "bat2" parent = "link4" visible = "1"
+                      model_url = "package://hydrus/urdf/mesh/battery/Kypom-3000-6s.dae">
+    <origin xyz="${link_length/2} 0.0 -0.048" rpy="0 0 0"/>
+    <inertial>
+      <origin xyz="0 0 0" rpy="0 0 0"/>
+      <mass value="0.4108"/>
+      <inertia
+          ixx="0.0001" iyy="0.0006" izz="0.0006"
+          ixy="0.0" ixz="0.0"  iyz="0.0"/>
+    </inertial>
+  </xacro:extra_module>
   <!-- processor: intel upboard -->
   <xacro:extra_module name = "pc" parent = "link2" visible = "1"

File: mbzirc2020/mbzirc2020_task3/mbzirc2020_task3_common/robots/hydrus.gazebo.xacro (robot description, xacro)
@@ -16,5 +16,5 @@
           <width>1280</width>
           <height>720</height>
-          <format>RGB</format>
+          <format>B8G8R8</format>
         </image>
         <clip>

Commit message: Update the robot model for task1:     - Add brix i7 model     - Add realsense D435 sensor module for drone detection.     - Update the battery configuration for hydrus

File: mbzirc2020/mbzirc2020_task1/mbzirc2020_task1_common/robots/hydrus.gazebo.xacro (robot description, xacro)
@@ -6,39 +6,119 @@
   <!-- gazebo plugin for sensors -->
   <xacro:include filename="$(find mbzirc2020_common)/robots/default.gazebo.xacro" />
-  <!-- gazebo for FLIR -->
-  <!-- RGB camera instead of IR camera -->
-  <gazebo reference="rgb_camera_frame">
-    <sensor type="camera" name="rgb_camera_frame">
-      <update_rate>30.0</update_rate>
-      <camera name="thermal">
-        <horizontal_fov>1.57</horizontal_fov>
-        <image>
-          <width>1280</width>
-          <height>720</height>
-          <format>B8G8R8</format>
-        </image>
-        <clip>
-          <near>0.02</near>
-          <far>300</far>
-        </clip>
-        <noise>
-          <type>gaussian</type>
-          <mean>0.0</mean>
-          <stddev>0.007</stddev>
-        </noise>
+  <!-- gazebo for Realsense D435 -->
+  <!--  The following values model the aluminum peripherial case for the
+        D435 camera, with the camera joint represented by the actual
+        peripherial camera tripod mount -->
+  <xacro:property name="d435_cam_depth_to_left_ir_offset" value="0.0"/>
+  <xacro:property name="d435_cam_depth_to_right_ir_offset" value="-0.050"/>
+  <xacro:property name="d435_cam_depth_to_color_offset" value="0.015"/>
+  <xacro:property name="d435_cam_width" value="0.090"/>
+  <xacro:property name="d435_cam_height" value="0.025"/>
+  <xacro:property name="d435_cam_depth" value="0.02505"/>
+  <xacro:property name="d435_cam_mount_from_center_offset" value="0.0149"/>
+  <!--  The following offset is relative the the physical D435 camera peripherial
+        camera tripod mount -->
+  <xacro:property name="d435_cam_depth_px" value="${d435_cam_mount_from_center_offset}"/>
+  <xacro:property name="d435_cam_depth_py" value="0.0175"/>
+  <xacro:property name="d435_cam_depth_pz" value="${d435_cam_height/2}"/>
+  <material name="aluminum">
+    <color rgba="0.5 0.5 0.5 1"/>
+  </material>
+  <!-- camera depth joints and links -->
+  <joint name="rs_d435_depth_joint" type="fixed">
+    <origin xyz="0 0 0" rpy="0 0 0"/>
+    <parent link="rs_d435_link"/>
+    <child link="rs_d435_depth_frame" />
+  </joint>
+  <link name="rs_d435_depth_frame"/>
+  <joint name="rs_d435_depth_optical_joint" type="fixed">
+    <origin xyz="0 0 0" rpy="${-pi/2} 0 ${-pi/2}" />
+    <parent link="rs_d435_depth_frame" />
+    <child link="rs_d435_depth_optical_frame" />
+  </joint>
+  <link name="rs_d435_depth_optical_frame"/>
+  <!-- camera left IR joints and links -->
+  <joint name="rs_d435_left_ir_joint" type="fixed">
+    <origin xyz="0 ${d435_cam_depth_to_left_ir_offset} 0" rpy="0 0 0" />
+    <parent link="rs_d435_depth_frame" />
+    <child link="rs_d435_left_ir_frame" />
+  </joint>
+  <link name="rs_d435_left_ir_frame"/>
+  <joint name="rs_d435_left_ir_optical_joint" type="fixed">
+    <origin xyz="0 0 0" rpy="${-pi/2} 0 ${-pi/2}" />
+    <parent link="rs_d435_left_ir_frame" />
+    <child link="rs_d435_left_ir_optical_frame" />
+  </joint>
+  <link name="rs_d435_left_ir_optical_frame"/>
+  <!-- camera right IR joints and links -->
+  <joint name="rs_d435_right_ir_joint" type="fixed">
+    <origin xyz="0 ${d435_cam_depth_to_right_ir_offset} 0" rpy="0 0 0" />
+    <parent link="rs_d435_depth_frame" />
+    <child link="rs_d435_right_ir_frame" />
+  </joint>
+  <link name="rs_d435_right_ir_frame"/>
+  <joint name="rs_d435_right_ir_optical_joint" type="fixed">
+    <origin xyz="0 0 0" rpy="${-pi/2} 0 ${-pi/2}" />
+    <parent link="rs_d435_right_ir_frame" />
+    <child link="rs_d435_right_ir_optical_frame" />
+  </joint>
+  <link name="rs_d435_right_ir_optical_frame"/>
+  <!-- camera color joints and links -->
+  <joint name="rs_d435_color_joint" type="fixed">
+    <origin xyz="0 ${d435_cam_depth_to_color_offset} 0" rpy="0 0 0" />
+    <parent link="rs_d435_depth_frame" />
+    <child link="rs_d435_color_frame" />
+  </joint>
+  <link name="rs_d435_color_frame"/>
+  <joint name="rs_d435_color_optical_joint" type="fixed">
+    <origin xyz="0 0 0" rpy="${-pi/2} 0 ${-pi/2}" />
+    <parent link="rs_d435_color_frame" />
+    <child link="rs_d435_color_optical_frame" />
+  </joint>
+  <link name="rs_d435_color_optical_frame"/>
+  <!-- gazebo plugin -->
+  <gazebo reference="rs_d435_color_frame">
+    <sensor type="depth" name="rs_d435_camera">
+      <update_rate>20.0</update_rate>
+      <camera name="head">
+	<horizontal_fov>1.59174</horizontal_fov>
+	<vertical_fov>1.14319</vertical_fov>
+	<image>
+	  <width>1280</width>
+	  <height>720</height>
+	  <format>RGB</format>
+	</image>
+	<clip>
+	  <near>0.02</near>
+	  <far>300</far>
+	</clip>
+	<noise>
+	  <type>gaussian</type>
+	  <mean>0.0</mean>
+	  <stddev>0.007</stddev>
+	</noise>
       </camera>
-      <plugin name="camera_controller" filename="libgazebo_ros_camera.so">
-        <alwaysOn>true</alwaysOn>
-        <updateRate>0.0</updateRate>
-        <cameraName>rgb_camera</cameraName>
-        <imageTopicName>image_raw</imageTopicName>
-        <cameraInfoTopicName>camera_info</cameraInfoTopicName>
-        <frameName>rgb_camera_optical_frame</frameName>
-        <hackBaseline>0.07</hackBaseline>
-        <distortionK1>0.0</distortionK1>
-        <distortionK2>0.0</distortionK2>
-        <distortionK3>0.0</distortionK3>
-        <distortionT1>0.0</distortionT1>
-        <distortionT2>0.0</distortionT2>
+      <plugin name="depth_camera" filename="libgazebo_ros_openni_kinect.so">
+	<baseline>0.06</baseline>
+	<alwaysOn>true</alwaysOn>
+	<updateRate>0.0</updateRate>
+	<cameraName>rs_d435</cameraName>
+	<imageTopicName>color/image_rect_color</imageTopicName>
+	<cameraInfoTopicName>color/camera_info</cameraInfoTopicName>
+	<depthImageCameraInfoTopicName>aligned_depth_to_color/camera_info</depthImageCameraInfoTopicName>
+	<depthImageTopicName>aligned_depth_to_color/image_raw</depthImageTopicName>
+	<pointCloudTopicName>depth_registered/points</pointCloudTopicName>
+	<frameName>rs_d435_color_optical_frame</frameName>
+	<pointCloudCutoff>0.05</pointCloudCutoff>
+	<distortionK1>0</distortionK1>
+	<distortionK2>0</distortionK2>
+	<distortionK3>0</distortionK3>
+	<distortionT1>0</distortionT1>
+	<distortionT2>0</distortionT2>
+	<CxPrime>0</CxPrime>
+	<Cx>0</Cx>
+	<Cy>0</Cy>
+	<focalLength>0</focalLength>
+	<hackBaseline>0</hackBaseline>
       </plugin>
     </sensor>

File: mbzirc2020/mbzirc2020_task1/mbzirc2020_task1_common/robots/hydrus.urdf.xacro (robot description, xacro)
@@ -13,4 +13,5 @@
       <origin xyz="0 0 0" rpy="0 0 0"/>
       <mass value="0.4108"/>
+      <!-- <mass value="0.4238"/> -->
       <inertia
           ixx="0.0001" iyy="0.0006" izz="0.0006"
@@ -24,4 +25,5 @@
       <origin xyz="0 0 0" rpy="0 0 0"/>
       <mass value="0.4108"/>
+      <!-- <mass value="0.4238"/> -->
       <inertia
           ixx="0.0001" iyy="0.0006" izz="0.0006"
@@ -29,33 +31,43 @@
     </inertial>
   </xacro:extra_module>
-  <!-- processor: intel upboard -->
+  <!-- 1.3 processor: gygabyte brix i7 -->
   <xacro:extra_module name = "pc" parent = "link2" visible = "1"
-                      model_url = "package://mbzirc2020_common/urdf/mesh/modules/processor/intel_upboard_fixed_joint_unit.dae" >
-    <origin xyz="${link_length / 2 + 0.2845} 0.011 0.016" rpy="0 0 ${pi}"/>
+                      model_url = "package://mbzirc2020_common/urdf/mesh/modules/processor/gygabyte_brix_fixed_joint_unit.STL" >
+    <origin xyz="${link_length / 2 + 0.27486} 0.02569 0.04" rpy="0 0 0"/>
     <inertial>
-      <mass value = "0.117" />
-      <origin xyz="${21 * 0.001} ${4 * 0.001} ${12 * 0.001}" rpy="0 0 0"/>
+      <mass value = "0.323" /> <!-- plus cable for leddar one-->
+      <origin xyz="${1.5 * 0.001} ${-3.5 * 0.001} ${8.9 * 0.001}" rpy="0 0 0"/>
       <inertia
-          ixx="0.00004" ixy="0.0" ixz="0.0"
-          iyy="0.00008" iyz="0.0"
-          izz="0.00011"/>
+          ixx="0.000351" ixy="0.0" ixz="0.0"
+          iyy="0.000272" iyz="0.0"
+          izz="0.000570"/>
     </inertial>
   </xacro:extra_module>
-  <!-- end: intel upboard -->
+  <!-- end: gygabyte brix i7 -->
   <!-- sensor -->
-  <!-- 1. RGB camera -->
-  <!-- TODO: accurate intertia parameters and position -->
-  <xacro:extra_module name = "rgb_camera_frame" parent = "link2" visible = "0"  >
-    <origin xyz="${link_length / 2 + 0.140} 0.162 0.063" rpy="0 0 ${3 * pi/4}"/>
+  <xacro:extra_module name = "rs_d435_unit" parent = "link2" visible = "1" model_url = "package://mbzirc2020_task1_common/urdf/meshes/sensor/rs_d435_unit3_center_bar.dae">
+    <origin xyz="${link_length / 2 + 0.0605} 0.2395 0.0502" rpy="0 0 ${pi * 3/4}"/>
     <inertial>
-      <mass value = "0.001" /> <!-- temporary -->
+      <mass value = "0.07669" /> <!-- includes sensor and mount -->
+      <origin xyz="0.014374 0 0.01599" rpy="0 0 0"/>
+      <inertia
+          ixx="0.000088" iyy="0.000012" izz="0.000089"
+          ixy="0" ixz="0" iyz="0"/>
+    </inertial>
+  </xacro:extra_module>
+  <xacro:extra_module name = "rs_d435_usb_cable" parent = "rs_d435_unit" visible = "0" >
+    <origin xyz="-0.13 0 0 " rpy="0 0 0"/>
+    <inertial>
+      <mass value = "0.033" />
       <origin xyz="0 0 0" rpy="0 0 0"/>
       <inertia
           ixx="0.0" ixy="0.0" ixz="0.0"
-          iyy="0.0" iyz="0.0" izz="0.0"/>
+          iyy="0.0" iyz="0.0"
+          izz="0.0"/>
     </inertial>
   </xacro:extra_module>
-  <xacro:extra_module name = "rgb_camera_optical_frame" parent = "rgb_camera_frame">
-    <origin xyz="0 0 0" rpy="${-pi / 2} 0 ${-pi / 2}"/>
+  <!-- rs_d435_link is the parrent of sensors' frame, identical to rs_d435_left_ir_frame -->
+  <xacro:extra_module name = "rs_d435_link" parent = "rs_d435_unit" visible = "0" >
+    <origin xyz="0.03 0.0175 0.019 " rpy="0 0 0"/>
     <inertial>
       <mass value = "0.0" />
