Commit message: [Temp] update robot model - add mocular camera

File: mbzirc2020/mbzirc2020_task1/mbzirc2020_task1_common/robots/hydrus.gazebo.xacro (robot description, xacro)
@@ -3,124 +3,127 @@
     xmlns:xacro="http://www.ros.org/wiki/xacro" name="hydrusx" >
   <!-- base robot model -->
+  <xacro:arg name="monocular_camera" default="true" />
   <xacro:include filename="$(find mbzirc2020_task1_common)/robots/hydrus.urdf.xacro" />
   <!-- gazebo plugin for sensors -->
   <xacro:include filename="$(find mbzirc2020_common)/robots/default.gazebo.xacro" />
   <!-- gazebo for Realsense D435 -->
-  <!--  The following values model the aluminum peripherial case for the
-        D435 camera, with the camera joint represented by the actual
-        peripherial camera tripod mount -->
-  <xacro:property name="d435_cam_depth_to_left_ir_offset" value="0.0"/>
-  <xacro:property name="d435_cam_depth_to_right_ir_offset" value="-0.050"/>
-  <xacro:property name="d435_cam_depth_to_color_offset" value="0.015"/>
-  <xacro:property name="d435_cam_width" value="0.090"/>
-  <xacro:property name="d435_cam_height" value="0.025"/>
-  <xacro:property name="d435_cam_depth" value="0.02505"/>
-  <xacro:property name="d435_cam_mount_from_center_offset" value="0.0149"/>
-  <!--  The following offset is relative the the physical D435 camera peripherial
-        camera tripod mount -->
-  <xacro:property name="d435_cam_depth_px" value="${d435_cam_mount_from_center_offset}"/>
-  <xacro:property name="d435_cam_depth_py" value="0.0175"/>
-  <xacro:property name="d435_cam_depth_pz" value="${d435_cam_height/2}"/>
-  <material name="aluminum">
-    <color rgba="0.5 0.5 0.5 1"/>
-  </material>
-  <!-- camera depth joints and links -->
-  <joint name="rs_d435_depth_joint" type="fixed">
-    <origin xyz="0 0 0" rpy="0 0 0"/>
-    <parent link="rs_d435_link"/>
-    <child link="rs_d435_depth_frame" />
-  </joint>
-  <link name="rs_d435_depth_frame"/>
-  <joint name="rs_d435_depth_optical_joint" type="fixed">
-    <origin xyz="0 0 0" rpy="${-pi/2} 0 ${-pi/2}" />
-    <parent link="rs_d435_depth_frame" />
-    <child link="rs_d435_depth_optical_frame" />
-  </joint>
-  <link name="rs_d435_depth_optical_frame"/>
-  <!-- camera left IR joints and links -->
-  <joint name="rs_d435_left_ir_joint" type="fixed">
-    <origin xyz="0 ${d435_cam_depth_to_left_ir_offset} 0" rpy="0 0 0" />
-    <parent link="rs_d435_depth_frame" />
-    <child link="rs_d435_left_ir_frame" />
-  </joint>
-  <link name="rs_d435_left_ir_frame"/>
-  <joint name="rs_d435_left_ir_optical_joint" type="fixed">
-    <origin xyz="0 0 0" rpy="${-pi/2} 0 ${-pi/2}" />
-    <parent link="rs_d435_left_ir_frame" />
-    <child link="rs_d435_left_ir_optical_frame" />
-  </joint>
-  <link name="rs_d435_left_ir_optical_frame"/>
-  <!-- camera right IR joints and links -->
-  <joint name="rs_d435_right_ir_joint" type="fixed">
-    <origin xyz="0 ${d435_cam_depth_to_right_ir_offset} 0" rpy="0 0 0" />
-    <parent link="rs_d435_depth_frame" />
-    <child link="rs_d435_right_ir_frame" />
-  </joint>
-  <link name="rs_d435_right_ir_frame"/>
-  <joint name="rs_d435_right_ir_optical_joint" type="fixed">
-    <origin xyz="0 0 0" rpy="${-pi/2} 0 ${-pi/2}" />
-    <parent link="rs_d435_right_ir_frame" />
-    <child link="rs_d435_right_ir_optical_frame" />
-  </joint>
-  <link name="rs_d435_right_ir_optical_frame"/>
-  <!-- camera color joints and links -->
-  <joint name="rs_d435_color_joint" type="fixed">
-    <origin xyz="0 ${d435_cam_depth_to_color_offset} 0" rpy="0 0 0" />
-    <parent link="rs_d435_depth_frame" />
-    <child link="rs_d435_color_frame" />
-  </joint>
-  <link name="rs_d435_color_frame"/>
-  <joint name="rs_d435_color_optical_joint" type="fixed">
-    <origin xyz="0 0 0" rpy="${-pi/2} 0 ${-pi/2}" />
-    <parent link="rs_d435_color_frame" />
-    <child link="rs_d435_color_optical_frame" />
-  </joint>
-  <link name="rs_d435_color_optical_frame"/>
-  <!-- gazebo plugin -->
-  <gazebo reference="rs_d435_color_frame">
-    <sensor type="depth" name="rs_d435_camera">
-      <update_rate>20.0</update_rate>
-      <camera name="head">
-	<horizontal_fov>1.59174</horizontal_fov>
-	<vertical_fov>1.14319</vertical_fov>
-	<image>
-	  <width>1280</width>
-	  <height>720</height>
-	  <format>RGB</format>
-	</image>
-	<clip>
-	  <near>0.02</near>
-	  <far>300</far>
-	</clip>
-	<noise>
-	  <type>gaussian</type>
-	  <mean>0.0</mean>
-	  <stddev>0.007</stddev>
-	</noise>
-      </camera>
-      <plugin name="depth_camera" filename="libgazebo_ros_openni_kinect.so">
-	<baseline>0.06</baseline>
-	<alwaysOn>true</alwaysOn>
-	<updateRate>0.0</updateRate>
-	<cameraName>rs_d435</cameraName>
-	<imageTopicName>color/image_rect_color</imageTopicName>
-	<cameraInfoTopicName>color/camera_info</cameraInfoTopicName>
-	<depthImageCameraInfoTopicName>aligned_depth_to_color/camera_info</depthImageCameraInfoTopicName>
-	<depthImageTopicName>aligned_depth_to_color/image_raw</depthImageTopicName>
-	<pointCloudTopicName>depth_registered/points</pointCloudTopicName>
-	<frameName>rs_d435_color_optical_frame</frameName>
-	<pointCloudCutoff>0.05</pointCloudCutoff>
-	<distortionK1>0</distortionK1>
-	<distortionK2>0</distortionK2>
-	<distortionK3>0</distortionK3>
-	<distortionT1>0</distortionT1>
-	<distortionT2>0</distortionT2>
-	<CxPrime>0</CxPrime>
-	<Cx>0</Cx>
-	<Cy>0</Cy>
-	<focalLength>0</focalLength>
-	<hackBaseline>0</hackBaseline>
-      </plugin>
-    </sensor>
-  </gazebo>
+  <xacro:unless value="$(arg monocular_camera)">
+    <!--  The following values model the aluminum peripherial case for the
+         D435 camera, with the camera joint represented by the actual
+         peripherial camera tripod mount -->
+    <xacro:property name="d435_cam_depth_to_left_ir_offset" value="0.0"/>
+    <xacro:property name="d435_cam_depth_to_right_ir_offset" value="-0.050"/>
+    <xacro:property name="d435_cam_depth_to_color_offset" value="0.015"/>
+    <xacro:property name="d435_cam_width" value="0.090"/>
+    <xacro:property name="d435_cam_height" value="0.025"/>
+    <xacro:property name="d435_cam_depth" value="0.02505"/>
+    <xacro:property name="d435_cam_mount_from_center_offset" value="0.0149"/>
+    <!--  The following offset is relative the the physical D435 camera peripherial
+         camera tripod mount -->
+    <xacro:property name="d435_cam_depth_px" value="${d435_cam_mount_from_center_offset}"/>
+    <xacro:property name="d435_cam_depth_py" value="0.0175"/>
+    <xacro:property name="d435_cam_depth_pz" value="${d435_cam_height/2}"/>
+    <material name="aluminum">
+      <color rgba="0.5 0.5 0.5 1"/>
+    </material>
+    <!-- camera depth joints and links -->
+    <joint name="rs_d435_depth_joint" type="fixed">
+      <origin xyz="0 0 0" rpy="0 0 0"/>
+      <parent link="rs_d435_link"/>
+      <child link="rs_d435_depth_frame" />
+    </joint>
+    <link name="rs_d435_depth_frame"/>
+    <joint name="rs_d435_depth_optical_joint" type="fixed">
+      <origin xyz="0 0 0" rpy="${-pi/2} 0 ${-pi/2}" />
+      <parent link="rs_d435_depth_frame" />
+      <child link="rs_d435_depth_optical_frame" />
+    </joint>
+    <link name="rs_d435_depth_optical_frame"/>
+    <!-- camera left IR joints and links -->
+    <joint name="rs_d435_left_ir_joint" type="fixed">
+      <origin xyz="0 ${d435_cam_depth_to_left_ir_offset} 0" rpy="0 0 0" />
+      <parent link="rs_d435_depth_frame" />
+      <child link="rs_d435_left_ir_frame" />
+    </joint>
+    <link name="rs_d435_left_ir_frame"/>
+    <joint name="rs_d435_left_ir_optical_joint" type="fixed">
+      <origin xyz="0 0 0" rpy="${-pi/2} 0 ${-pi/2}" />
+      <parent link="rs_d435_left_ir_frame" />
+      <child link="rs_d435_left_ir_optical_frame" />
+    </joint>
+    <link name="rs_d435_left_ir_optical_frame"/>
+    <!-- camera right IR joints and links -->
+    <joint name="rs_d435_right_ir_joint" type="fixed">
+      <origin xyz="0 ${d435_cam_depth_to_right_ir_offset} 0" rpy="0 0 0" />
+      <parent link="rs_d435_depth_frame" />
+      <child link="rs_d435_right_ir_frame" />
+    </joint>
+    <link name="rs_d435_right_ir_frame"/>
+    <joint name="rs_d435_right_ir_optical_joint" type="fixed">
+      <origin xyz="0 0 0" rpy="${-pi/2} 0 ${-pi/2}" />
+      <parent link="rs_d435_right_ir_frame" />
+      <child link="rs_d435_right_ir_optical_frame" />
+    </joint>
+    <link name="rs_d435_right_ir_optical_frame"/>
+    <!-- camera color joints and links -->
+    <joint name="rs_d435_color_joint" type="fixed">
+      <origin xyz="0 ${d435_cam_depth_to_color_offset} 0" rpy="0 0 0" />
+      <parent link="rs_d435_depth_frame" />
+      <child link="rs_d435_color_frame" />
+    </joint>
+    <link name="rs_d435_color_frame"/>
+    <joint name="rs_d435_color_optical_joint" type="fixed">
+      <origin xyz="0 0 0" rpy="${-pi/2} 0 ${-pi/2}" />
+      <parent link="rs_d435_color_frame" />
+      <child link="rs_d435_color_optical_frame" />
+    </joint>
+    <link name="rs_d435_color_optical_frame"/>
+    <!-- gazebo plugin -->
+    <gazebo reference="rs_d435_color_frame">
+      <sensor type="depth" name="rs_d435_camera">
+        <update_rate>20.0</update_rate>
+        <camera name="head">
+	  <horizontal_fov>1.59174</horizontal_fov>
+	  <vertical_fov>1.14319</vertical_fov>
+	  <image>
+	    <width>1280</width>
+	    <height>720</height>
+	    <format>RGB</format>
+	  </image>
+	  <clip>
+	    <near>0.02</near>
+	    <far>300</far>
+	  </clip>
+	  <noise>
+	    <type>gaussian</type>
+	    <mean>0.0</mean>
+	    <stddev>0.007</stddev>
+	  </noise>
+        </camera>
+        <plugin name="depth_camera" filename="libgazebo_ros_openni_kinect.so">
+	  <baseline>0.06</baseline>
+	  <alwaysOn>true</alwaysOn>
+	  <updateRate>0.0</updateRate>
+	  <cameraName>rs_d435</cameraName>
+	  <imageTopicName>color/image_rect_color</imageTopicName>
+	  <cameraInfoTopicName>color/camera_info</cameraInfoTopicName>
+	  <depthImageCameraInfoTopicName>aligned_depth_to_color/camera_info</depthImageCameraInfoTopicName>
+	  <depthImageTopicName>aligned_depth_to_color/image_raw</depthImageTopicName>
+	  <pointCloudTopicName>depth_registered/points</pointCloudTopicName>
+	  <frameName>rs_d435_color_optical_frame</frameName>
+	  <pointCloudCutoff>0.05</pointCloudCutoff>
+	  <distortionK1>0</distortionK1>
+	  <distortionK2>0</distortionK2>
+	  <distortionK3>0</distortionK3>
+	  <distortionT1>0</distortionT1>
+	  <distortionT2>0</distortionT2>
+	  <CxPrime>0</CxPrime>
+	  <Cx>0</Cx>
+	  <Cy>0</Cy>
+	  <focalLength>0</focalLength>
+	  <hackBaseline>0</hackBaseline>
+        </plugin>
+      </sensor>
+    </gazebo>
+  </xacro:unless>
 </robot>

File: mbzirc2020/mbzirc2020_task1/mbzirc2020_task1_common/robots/hydrus.urdf.xacro (robot description, xacro)
@@ -3,4 +3,6 @@
     xmlns:xacro="http://www.ros.org/wiki/xacro" name="hydrusx" >
   <!-- base kinematics model -->
+  <xacro:arg name="monocular_camera" default="true" />
+  <xacro:arg name="camera_height" default="0" />
   <xacro:arg name="horizontal_vio" default="false" />
   <xacro:include filename="$(find mbzirc2020_common)/robots/default.urdf.xacro" />
@@ -12,6 +14,5 @@
     <inertial>
       <origin xyz="0 0 0" rpy="0 0 0"/>
-      <mass value="0.4108"/>
-      <!-- <mass value="0.4238"/> -->
+      <mass value="0.411"/>
       <inertia
           ixx="0.0001" iyy="0.0006" izz="0.0006"
@@ -24,6 +25,5 @@
     <inertial>
       <origin xyz="0 0 0" rpy="0 0 0"/>
-      <mass value="0.4108"/>
-      <!-- <mass value="0.4238"/> -->
+      <mass value="0.411"/>
       <inertia
           ixx="0.0001" iyy="0.0006" izz="0.0006"
@@ -46,38 +46,155 @@
   <!-- end: gygabyte brix i7 -->
   <!-- sensor -->
-  <xacro:extra_module name = "rs_d435_unit" parent = "link2" visible = "1" model_url = "package://mbzirc2020_task1_common/urdf/meshes/sensor/rs_d435_unit3_center_bar.dae">
-    <origin xyz="${link_length / 2 + 0.0605} 0.2395 0.0502" rpy="0 0 ${pi * 3/4}"/>
-    <inertial>
-      <mass value = "0.07669" /> <!-- includes sensor and mount -->
-      <origin xyz="0.014374 0 0.01599" rpy="0 0 0"/>
-      <inertia
-          ixx="0.000088" iyy="0.000012" izz="0.000089"
-          ixy="0" ixz="0" iyz="0"/>
-    </inertial>
-  </xacro:extra_module>
-  <xacro:extra_module name = "rs_d435_usb_cable" parent = "rs_d435_unit" visible = "0" >
-    <origin xyz="-0.13 0 0 " rpy="0 0 0"/>
-    <inertial>
-      <mass value = "0.033" />
-      <origin xyz="0 0 0" rpy="0 0 0"/>
-      <inertia
-          ixx="0.0" ixy="0.0" ixz="0.0"
-          iyy="0.0" iyz="0.0"
-          izz="0.0"/>
-    </inertial>
-  </xacro:extra_module>
-  <!-- rs_d435_link is the parrent of sensors' frame, identical to rs_d435_left_ir_frame -->
-  <xacro:extra_module name = "rs_d435_link" parent = "rs_d435_unit" visible = "0" >
-    <origin xyz="0.03 0.0175 0.019 " rpy="0 0 0"/>
-    <inertial>
-      <mass value = "0.0" />
-      <origin xyz="0 0 0" rpy="0 0 0"/>
-      <inertia
-          ixx="0.0" ixy="0.0" ixz="0.0"
-          iyy="0.0" iyz="0.0"
-          izz="0.0"/>
-    </inertial>
-  </xacro:extra_module>
+  <!-- Monocular camera -->
+  <xacro:if value="$(arg monocular_camera)">
+    <!-- direct mount type -->
+    <xacro:unless value="$(arg camera_height)">
+      <xacro:extra_module name = "monocular_camera_unit" parent = "link2" visible = "1" model_url = "package://mbzirc2020_task1_common/urdf/meshes/sensor/ELP_SUSB1080P_direct_unit.dae">
+        <origin xyz="${link_length / 2 + 0.0605} 0.2395 0.0502" rpy="0 0 ${pi * 3/4}"/>
+        <inertial>
+          <mass value = "0.0435" />
+          <origin xyz="0.011 0 0.005" rpy="0 0 0"/>
+          <inertia
+              ixx="0.0" iyy="0.0" izz="0.0"
+              ixy="0.0" ixz="0.0" iyz="0.0"/>
+        </inertial>
+      </xacro:extra_module>
+      <xacro:extra_module name = "color_camera_frame" parent = "monocular_camera_unit" visible = "0" >
+        <origin xyz="0.014 0.0 0.005 " rpy="0 0 0"/>
+        <inertial>
+          <mass value = "0.0" />
+          <origin xyz="0 0 0" rpy="0 0 0"/>
+          <inertia
+              ixx="0.0" ixy="0.0" ixz="0.0"
+              iyy="0.0" iyz="0.0"
+              izz="0.0"/>
+        </inertial>
+      </xacro:extra_module>
+      <xacro:extra_module name = "camera_usb_cable" parent = "monocular_camera_unit" visible = "0" >
+        <origin xyz="-0.13 0 0 " rpy="0 0 0"/>
+        <inertial>
+          <mass value = "0.0474" />
+          <origin xyz="0 0 0" rpy="0 0 0"/>
+          <inertia
+              ixx="0.0" ixy="0.0" ixz="0.0"
+              iyy="0.0" iyz="0.0"
+              izz="0.0"/>
+        </inertial>
+      </xacro:extra_module>
+    </xacro:unless>
+    <!-- carbon pipe mount type -->
+    <xacro:if value="$(arg camera_height)">
+      <xacro:extra_module name = "center_bar" parent = "link2" visible = "1" model_url = "package://mbzirc2020_task1_common/urdf/meshes/sensor/single_camera_center_bar.dae">
+        <origin xyz="${link_length / 2 + 0.0605} 0.2395 0.0502" rpy="0 0 ${pi * 3/4}"/>
+        <inertial>
+          <mass value = "0.0233" />
+          <origin xyz="-0.003 0 -0.01" rpy="0 0 0"/>
+          <inertia
+              ixx="0.0" iyy="0.0" izz="0.0"
+              ixy="0.0" ixz="0.0" iyz="0.0"/>
+        </inertial>
+      </xacro:extra_module>
+      <xacro:extra_module name = "monocular_camera_unit" parent = "center_bar" visible = "1" model_url = "package://mbzirc2020_task1_common/urdf/meshes/sensor/ELP_SUSB1080P_unit.dae">
+        <origin xyz="0.001 0 $(arg camera_height)" rpy="0 0 0"/>
+        <inertial>
+          <mass value = "0.036" />
+          <origin xyz="-0.003 0 -0.01" rpy="0 0 0"/>
+          <inertia
+              ixx="0.0" iyy="0.0" izz="0.0"
+              ixy="0.0" ixz="0.0" iyz="0.0"/>
+        </inertial>
+      </xacro:extra_module>
+      <xacro:extra_module name = "camera_usb_cable" parent = "center_bar" visible = "0" >
+        <origin xyz="-0.11 0 0 " rpy="0 0 0"/>
+        <inertial>
+          <mass value = "0.0474" />
+          <origin xyz="0 0 0" rpy="0 0 0"/>
+          <inertia
+              ixx="0.0" ixy="0.0" ixz="0.0"
+              iyy="0.0" iyz="0.0"
+              izz="0.0"/>
+        </inertial>
+      </xacro:extra_module>
+      <xacro:extra_module name = "color_camera_frame" parent = "monocular_camera_unit" visible = "0" >
+        <origin xyz="0.0 0.0 0.0 " rpy="${pi} 0 0"/>
+        <inertial>
+          <mass value = "0.0" />
+          <origin xyz="0 0 0" rpy="0 0 0"/>
+          <inertia
+              ixx="0.0" ixy="0.0" ixz="0.0"
+              iyy="0.0" iyz="0.0"
+              izz="0.0"/>
+        </inertial>
+      </xacro:extra_module>
+    </xacro:if>
+    <xacro:extra_module name = "color_camera_optical_frame" parent = "color_camera_frame" visible = "0" >
+      <origin xyz="0.0 0.0 0.0 " rpy="${-pi/2} 0 ${-pi/2}"/>
+      <inertial>
+        <mass value = "0.0" />
+        <origin xyz="0 0 0" rpy="0 0 0"/>
+        <inertia
+            ixx="0.0" ixy="0.0" ixz="0.0"
+            iyy="0.0" iyz="0.0"
+            izz="0.0"/>
+      </inertial>
+    </xacro:extra_module>
+  </xacro:if>
+  <!-- Realsense D435 -->
+  <xacro:unless value="$(arg monocular_camera)">
+    <xacro:extra_module name = "rs_d435_unit" parent = "link2" visible = "1" model_url = "package://mbzirc2020_task1_common/urdf/meshes/sensor/rs_d435_unit3_center_bar.dae">
+      <origin xyz="${link_length / 2 + 0.0605} 0.2395 0.0502" rpy="0 0 ${pi * 3/4}"/>
+      <inertial>
+        <mass value = "0.07669" /> <!-- includes sensor and mount -->
+        <origin xyz="0.014374 0 0.01599" rpy="0 0 0"/>
+        <inertia
+            ixx="0.000088" iyy="0.000012" izz="0.000089"
+            ixy="0" ixz="0" iyz="0"/>
+      </inertial>
+    </xacro:extra_module>
+    <xacro:extra_module name = "rs_d435_usb_cable" parent = "rs_d435_unit" visible = "0" >
+      <origin xyz="-0.13 0 0 " rpy="0 0 0"/>
+      <inertial>
+        <mass value = "0.033" />
+        <origin xyz="0 0 0" rpy="0 0 0"/>
+        <inertia
+            ixx="0.0" ixy="0.0" ixz="0.0"
+            iyy="0.0" iyz="0.0"
+            izz="0.0"/>
+      </inertial>
+    </xacro:extra_module>
+    <!-- rs_d435_link is the parrent of sensors' frame, identical to rs_d435_left_ir_frame -->
+    <xacro:extra_module name = "rs_d435_link" parent = "rs_d435_unit" visible = "0" >
+      <origin xyz="0.03 0.0175 0.019 " rpy="0 0 0"/>
+      <inertial>
+        <mass value = "0.0" />
+        <origin xyz="0 0 0" rpy="0 0 0"/>
+        <inertia
+            ixx="0.0" ixy="0.0" ixz="0.0"
+            iyy="0.0" iyz="0.0"
+            izz="0.0"/>
+      </inertial>
+    </xacro:extra_module>
+  </xacro:unless>
   <!-- net -->
-  <!-- TODO: add net at the ends -->
+  <xacro:property name="net_mass" value=".035" />
+  <xacro:extra_module name = "net_anchor1" parent = "leg1" visible = "0" >
+    <origin xyz="0.0 0.0 0.0" rpy="0 0 0"/>
+    <inertial>
+      <origin xyz="0 0 0" rpy="0 0 0"/>
+      <mass value="${net_mass/2}"/>
+      <inertia
+          ixx="0.0" iyy="0.0" izz="0.0"
+          ixy="0.0" ixz="0.0"  iyz="0.0"/>
+    </inertial>
+  </xacro:extra_module>
+  <xacro:extra_module name = "net_anchor2" parent = "leg5" visible = "0" >
+    <origin xyz="0.0 0.0 0.0" rpy="0 0 0"/>
+    <inertial>
+      <origin xyz="0 0 0" rpy="0 0 0"/>
+      <mass value="${net_mass/2}"/>
+      <inertia
+          ixx="0.0" iyy="0.0" izz="0.0"
+          ixy="0.0" ixz="0.0"  iyz="0.0"/>
+    </inertial>
+  </xacro:extra_module>
 </robot>
