Commit message: Add gygabyte brix i7 model for task1 and task2

File: mbzirc2020/mbzirc2020_task1/mbzirc2020_task1_common/robots/hydrus.urdf.xacro (robot description, xacro)
@@ -28,18 +28,18 @@
     </inertial>
   </xacro:extra_module>
-  <!-- processor: intel upboard -->
+  <!-- 1.3 processor: gygabyte brix i7 -->
   <xacro:extra_module name = "pc" parent = "link2" visible = "1"
-                      model_url = "package://mbzirc2020_common/urdf/mesh/modules/processor/intel_upboard_fixed_joint_unit.dae" >
-    <origin xyz="${link_length / 2 + 0.2845} 0.011 0.016" rpy="0 0 ${pi}"/>
+                      model_url = "package://mbzirc2020_common/urdf/mesh/modules/processor/gygabyte_brix_fixed_joint_unit.STL" >
+    <origin xyz="${link_length / 2 + 0.27486} 0.02569 0.04" rpy="0 0 0"/>
     <inertial>
-      <mass value = "0.117" />
-      <origin xyz="${21 * 0.001} ${4 * 0.001} ${12 * 0.001}" rpy="0 0 0"/>
+      <mass value = "0.323" /> <!-- plus cable for leddar one-->
+      <origin xyz="${1.5 * 0.001} ${-3.5 * 0.001} ${8.9 * 0.001}" rpy="0 0 0"/>
       <inertia
-          ixx="0.00004" ixy="0.0" ixz="0.0"
-          iyy="0.00008" iyz="0.0"
-          izz="0.00011"/>
+          ixx="0.000351" ixy="0.0" ixz="0.0"
+          iyy="0.000272" iyz="0.0"
+          izz="0.000570"/>
     </inertial>
   </xacro:extra_module>
-  <!-- end: intel upboard -->
+  <!-- end: gygabyte brix i7 -->
   <!-- sensor -->
   <!-- 1. RGB camera -->

File: mbzirc2020/mbzirc2020_task2/mbzirc2020_task2_common/robots/hydrus.urdf.xacro (robot description, xacro)
@@ -28,19 +28,18 @@
     </inertial>
   </xacro:extra_module>
-  <!-- processor: intel upboard -->
-  <!-- TODO: change to brix -->
+  <!-- 1.3 processor: gygabyte brix i7 -->
   <xacro:extra_module name = "pc" parent = "link2" visible = "1"
-                      model_url = "package://mbzirc2020_common/urdf/mesh/modules/processor/intel_upboard_fixed_joint_unit.dae" >
-    <origin xyz="${link_length / 2 + 0.2845} 0.011 0.016" rpy="0 0 ${pi}"/>
+                      model_url = "package://mbzirc2020_common/urdf/mesh/modules/processor/gygabyte_brix_fixed_joint_unit.STL" >
+    <origin xyz="${link_length / 2 + 0.27486} 0.02569 0.04" rpy="0 0 0"/>
     <inertial>
-      <mass value = "0.117" />
-      <origin xyz="${21 * 0.001} ${4 * 0.001} ${12 * 0.001}" rpy="0 0 0"/>
+      <mass value = "0.323" /> <!-- plus cable for leddar one-->
+      <origin xyz="${1.5 * 0.001} ${-3.5 * 0.001} ${8.9 * 0.001}" rpy="0 0 0"/>
       <inertia
-          ixx="0.00004" ixy="0.0" ixz="0.0"
-          iyy="0.00008" iyz="0.0"
-          izz="0.00011"/>
+          ixx="0.000351" ixy="0.0" ixz="0.0"
+          iyy="0.000272" iyz="0.0"
+          izz="0.000570"/>
     </inertial>
   </xacro:extra_module>
-  <!-- end: intel upboard -->
+  <!-- end: gygabyte brix i7 -->
   <!-- sensor -->
   <!-- 1. downward rs-t265 (VIO) -->

File: mbzirc2020/mbzirc2020_task2/mbzirc2020_task2_common/robots/hydrus_ground_mode.urdf.xacro (robot description, xacro)
@@ -40,19 +40,18 @@
   </xacro:extra_module>
   <!-- end: processor: neuron -->
-  <!-- 1.3 processor: intel upboard -->
-  <!-- TODO: change to brix -->
+  <!-- 1.3 processor: gygabyte brix i7 -->
   <xacro:extra_module name = "pc" parent = "link2" visible = "1"
-                      model_url = "package://mbzirc2020_common/urdf/mesh/modules/processor/intel_upboard_fixed_joint_unit.dae" >
-    <origin xyz="${link_length / 2 + 0.2845} 0.011 0.016" rpy="0 0 ${pi}"/>
-    <inertial>
-      <mass value = "0.117" />
-      <origin xyz="${21 * 0.001} ${4 * 0.001} ${12 * 0.001}" rpy="0 0 0"/>
-      <inertia
-          ixx="0.00004" ixy="0.0" ixz="0.0"
-          iyy="0.00008" iyz="0.0"
-          izz="0.00011"/>
-    </inertial>
-  </xacro:extra_module>
-  <!-- end: intel upboard -->
+                      model_url = "package://mbzirc2020_common/urdf/mesh/modules/processor/gygabyte_brix_fixed_joint_unit.STL" >
+    <origin xyz="${link_length / 2 + 0.27486} 0.02569 0.04" rpy="0 0 0"/>
+    <inertial>
+      <mass value = "0.323" /> <!-- plus cable for leddar one-->
+      <origin xyz="${1.5 * 0.001} ${-3.5 * 0.001} ${8.9 * 0.001}" rpy="0 0 0"/>
+      <inertia
+          ixx="0.000351" ixy="0.0" ixz="0.0"
+          iyy="0.000272" iyz="0.0"
+          izz="0.000570"/>
+    </inertial>
+  </xacro:extra_module>
+  <!-- end: gygabyte brix i7 -->
   <!-- 2.  sensor -->
   <!-- 2.1 leddar one -->

Commit message: update robot model - add monocular camera

File: mbzirc2020/mbzirc2020_task1/mbzirc2020_task1_common/robots/hydrus.urdf.xacro (robot description, xacro)
@@ -3,4 +3,6 @@
     xmlns:xacro="http://www.ros.org/wiki/xacro" name="hydrusx" >
   <!-- base kinematics model -->
+  <xacro:arg name="monocular_camera" default="true" />
+  <xacro:arg name="camera_height" default="0" />
   <xacro:arg name="horizontal_vio" default="false" />
   <xacro:include filename="$(find mbzirc2020_common)/robots/default.urdf.xacro" />
@@ -12,6 +14,5 @@
     <inertial>
       <origin xyz="0 0 0" rpy="0 0 0"/>
-      <mass value="0.4108"/>
-      <!-- <mass value="0.4238"/> -->
+      <mass value="0.411"/>
       <inertia
           ixx="0.0001" iyy="0.0006" izz="0.0006"
@@ -24,6 +25,5 @@
     <inertial>
       <origin xyz="0 0 0" rpy="0 0 0"/>
-      <mass value="0.4108"/>
-      <!-- <mass value="0.4238"/> -->
+      <mass value="0.411"/>
       <inertia
           ixx="0.0001" iyy="0.0006" izz="0.0006"
@@ -46,38 +46,155 @@
   <!-- end: gygabyte brix i7 -->
   <!-- sensor -->
-  <xacro:extra_module name = "rs_d435_unit" parent = "link2" visible = "1" model_url = "package://mbzirc2020_task1_common/urdf/meshes/sensor/rs_d435_unit3_center_bar.dae">
-    <origin xyz="${link_length / 2 + 0.0605} 0.2395 0.0502" rpy="0 0 ${pi * 3/4}"/>
-    <inertial>
-      <mass value = "0.07669" /> <!-- includes sensor and mount -->
-      <origin xyz="0.014374 0 0.01599" rpy="0 0 0"/>
-      <inertia
-          ixx="0.000088" iyy="0.000012" izz="0.000089"
-          ixy="0" ixz="0" iyz="0"/>
-    </inertial>
-  </xacro:extra_module>
-  <xacro:extra_module name = "rs_d435_usb_cable" parent = "rs_d435_unit" visible = "0" >
-    <origin xyz="-0.13 0 0 " rpy="0 0 0"/>
-    <inertial>
-      <mass value = "0.033" />
-      <origin xyz="0 0 0" rpy="0 0 0"/>
-      <inertia
-          ixx="0.0" ixy="0.0" ixz="0.0"
-          iyy="0.0" iyz="0.0"
-          izz="0.0"/>
-    </inertial>
-  </xacro:extra_module>
-  <!-- rs_d435_link is the parrent of sensors' frame, identical to rs_d435_left_ir_frame -->
-  <xacro:extra_module name = "rs_d435_link" parent = "rs_d435_unit" visible = "0" >
-    <origin xyz="0.03 0.0175 0.019 " rpy="0 0 0"/>
-    <inertial>
-      <mass value = "0.0" />
-      <origin xyz="0 0 0" rpy="0 0 0"/>
-      <inertia
-          ixx="0.0" ixy="0.0" ixz="0.0"
-          iyy="0.0" iyz="0.0"
-          izz="0.0"/>
-    </inertial>
-  </xacro:extra_module>
+  <!-- Monocular camera -->
+  <xacro:if value="$(arg monocular_camera)">
+    <!-- direct mount type -->
+    <xacro:unless value="$(arg camera_height)">
+      <xacro:extra_module name = "monocular_camera_unit" parent = "link2" visible = "1" model_url = "package://mbzirc2020_task1_common/urdf/meshes/sensor/ELP_SUSB1080P_direct_unit.dae">
+        <origin xyz="${link_length / 2 + 0.0605} 0.2395 0.0402" rpy="0 ${0.05} ${pi * 3/4 + 0.05}"/> <!-- calibrate by rviz camera plugin -->w
+        <inertial>
+          <mass value = "0.0435" />
+          <origin xyz="0.011 0 0.005" rpy="0 0 0"/>
+          <inertia
+              ixx="0.0" iyy="0.0" izz="0.0"
+              ixy="0.0" ixz="0.0" iyz="0.0"/>
+        </inertial>
+      </xacro:extra_module>
+      <xacro:extra_module name = "color_camera_frame" parent = "monocular_camera_unit" visible = "0" >
+        <origin xyz="0.016 0.0 0.005 " rpy="0 0 0"/>
+        <inertial>
+          <mass value = "0.0" />
+          <origin xyz="0 0 0" rpy="0 0 0"/>
+          <inertia
+              ixx="0.0" ixy="0.0" ixz="0.0"
+              iyy="0.0" iyz="0.0"
+              izz="0.0"/>
+        </inertial>
+      </xacro:extra_module>
+      <xacro:extra_module name = "camera_usb_cable" parent = "monocular_camera_unit" visible = "0" >
+        <origin xyz="-0.13 0 0 " rpy="0 0 0"/>
+        <inertial>
+          <mass value = "0.0474" />
+          <origin xyz="0 0 0" rpy="0 0 0"/>
+          <inertia
+              ixx="0.0" ixy="0.0" ixz="0.0"
+              iyy="0.0" iyz="0.0"
+              izz="0.0"/>
+        </inertial>
+      </xacro:extra_module>
+    </xacro:unless>
+    <!-- carbon pipe mount type -->
+    <xacro:if value="$(arg camera_height)">
+      <xacro:extra_module name = "center_bar" parent = "link2" visible = "1" model_url = "package://mbzirc2020_task1_common/urdf/meshes/sensor/single_camera_center_bar.dae">
+        <origin xyz="${link_length / 2 + 0.0605} 0.2395 0.0402" rpy="0 ${0.05} ${pi * 3/4 + 0.05}"/> <!-- copy the diret mount type, TODO: calibrate by rviz camera plugin -->
+        <inertial>
+          <mass value = "0.0233" />
+          <origin xyz="-0.003 0 -0.01" rpy="0 0 0"/>
+          <inertia
+              ixx="0.0" iyy="0.0" izz="0.0"
+              ixy="0.0" ixz="0.0" iyz="0.0"/>
+        </inertial>
+      </xacro:extra_module>
+      <xacro:extra_module name = "monocular_camera_unit" parent = "center_bar" visible = "1" model_url = "package://mbzirc2020_task1_common/urdf/meshes/sensor/ELP_SUSB1080P_unit.dae">
+        <origin xyz="0.001 0 $(arg camera_height)" rpy="0 0 0"/>
+        <inertial>
+          <mass value = "0.036" />
+          <origin xyz="-0.003 0 -0.01" rpy="0 0 0"/>
+          <inertia
+              ixx="0.0" iyy="0.0" izz="0.0"
+              ixy="0.0" ixz="0.0" iyz="0.0"/>
+        </inertial>
+      </xacro:extra_module>
+      <xacro:extra_module name = "camera_usb_cable" parent = "center_bar" visible = "0" >
+        <origin xyz="-0.11 0 0 " rpy="0 0 0"/>
+        <inertial>
+          <mass value = "0.0474" />
+          <origin xyz="0 0 0" rpy="0 0 0"/>
+          <inertia
+              ixx="0.0" ixy="0.0" ixz="0.0"
+              iyy="0.0" iyz="0.0"
+              izz="0.0"/>
+        </inertial>
+      </xacro:extra_module>
+      <xacro:extra_module name = "color_camera_frame" parent = "monocular_camera_unit" visible = "0" >
+        <origin xyz="0.0 0.0 0.0 " rpy="${pi} 0 0"/>
+        <inertial>
+          <mass value = "0.0" />
+          <origin xyz="0 0 0" rpy="0 0 0"/>
+          <inertia
+              ixx="0.0" ixy="0.0" ixz="0.0"
+              iyy="0.0" iyz="0.0"
+              izz="0.0"/>
+        </inertial>
+      </xacro:extra_module>
+    </xacro:if>
+    <xacro:extra_module name = "color_camera_optical_frame" parent = "color_camera_frame" visible = "0" >
+      <origin xyz="0.0 0.0 0.0 " rpy="${-pi/2} 0 ${-pi/2}"/>
+      <inertial>
+        <mass value = "0.0" />
+        <origin xyz="0 0 0" rpy="0 0 0"/>
+        <inertia
+            ixx="0.0" ixy="0.0" ixz="0.0"
+            iyy="0.0" iyz="0.0"
+            izz="0.0"/>
+      </inertial>
+    </xacro:extra_module>
+  </xacro:if>
+  <!-- Realsense D435 -->
+  <xacro:unless value="$(arg monocular_camera)">
+    <xacro:extra_module name = "rs_d435_unit" parent = "link2" visible = "1" model_url = "package://mbzirc2020_task1_common/urdf/meshes/sensor/rs_d435_unit3_center_bar.dae">
+      <origin xyz="${link_length / 2 + 0.0605} 0.2395 0.0502" rpy="0 0 ${pi * 3/4}"/>
+      <inertial>
+        <mass value = "0.07669" /> <!-- includes sensor and mount -->
+        <origin xyz="0.014374 0 0.01599" rpy="0 0 0"/>
+        <inertia
+            ixx="0.000088" iyy="0.000012" izz="0.000089"
+            ixy="0" ixz="0" iyz="0"/>
+      </inertial>
+    </xacro:extra_module>
+    <xacro:extra_module name = "rs_d435_usb_cable" parent = "rs_d435_unit" visible = "0" >
+      <origin xyz="-0.13 0 0 " rpy="0 0 0"/>
+      <inertial>
+        <mass value = "0.033" />
+        <origin xyz="0 0 0" rpy="0 0 0"/>
+        <inertia
+            ixx="0.0" ixy="0.0" ixz="0.0"
+            iyy="0.0" iyz="0.0"
+            izz="0.0"/>
+      </inertial>
+    </xacro:extra_module>
+    <!-- rs_d435_link is the parrent of sensors' frame, identical to rs_d435_left_ir_frame -->
+    <xacro:extra_module name = "rs_d435_link" parent = "rs_d435_unit" visible = "0" >
+      <origin xyz="0.03 0.0175 0.019 " rpy="0 0 0"/>
+      <inertial>
+        <mass value = "0.0" />
+        <origin xyz="0 0 0" rpy="0 0 0"/>
+        <inertia
+            ixx="0.0" ixy="0.0" ixz="0.0"
+            iyy="0.0" iyz="0.0"
+            izz="0.0"/>
+      </inertial>
+    </xacro:extra_module>
+  </xacro:unless>
   <!-- net -->
-  <!-- TODO: add net at the ends -->
+  <xacro:property name="net_mass" value=".035" />
+  <xacro:extra_module name = "net_anchor1" parent = "leg1" visible = "0" >
+    <origin xyz="0.0 0.0 0.0" rpy="0 0 0"/>
+    <inertial>
+      <origin xyz="0 0 0" rpy="0 0 0"/>
+      <mass value="${net_mass/2}"/>
+      <inertia
+          ixx="0.0" iyy="0.0" izz="0.0"
+          ixy="0.0" ixz="0.0"  iyz="0.0"/>
+    </inertial>
+  </xacro:extra_module>
+  <xacro:extra_module name = "net_anchor2" parent = "leg5" visible = "0" >
+    <origin xyz="0.0 0.0 0.0" rpy="0 0 0"/>
+    <inertial>
+      <origin xyz="0 0 0" rpy="0 0 0"/>
+      <mass value="${net_mass/2}"/>
+      <inertia
+          ixx="0.0" iyy="0.0" izz="0.0"
+          ixy="0.0" ixz="0.0"  iyz="0.0"/>
+    </inertial>
+  </xacro:extra_module>
 </robot>

Commit message: [Temp] tuning the camera optical frame using rviz camera plugin with the robot model

File: mbzirc2020/mbzirc2020_task1/mbzirc2020_task1_common/robots/hydrus.urdf.xacro (robot description, xacro)
@@ -51,5 +51,5 @@
     <xacro:unless value="$(arg camera_height)">
       <xacro:extra_module name = "monocular_camera_unit" parent = "link2" visible = "1" model_url = "package://mbzirc2020_task1_common/urdf/meshes/sensor/ELP_SUSB1080P_direct_unit.dae">
-        <origin xyz="${link_length / 2 + 0.0605} 0.2395 0.0502" rpy="0 0 ${pi * 3/4}"/>
+        <origin xyz="${link_length / 2 + 0.0605} 0.2395 0.0402" rpy="0 ${0.05} ${pi * 3/4 + 0.05}"/> <!-- calibrate by rviz camera plugin -->w
         <inertial>
           <mass value = "0.0435" />
@@ -61,5 +61,5 @@
       </xacro:extra_module>
       <xacro:extra_module name = "color_camera_frame" parent = "monocular_camera_unit" visible = "0" >
-        <origin xyz="0.014 0.0 0.005 " rpy="0 0 0"/>
+        <origin xyz="0.016 0.0 0.005 " rpy="0 0 0"/>
         <inertial>
           <mass value = "0.0" />
@@ -86,5 +86,5 @@
     <xacro:if value="$(arg camera_height)">
       <xacro:extra_module name = "center_bar" parent = "link2" visible = "1" model_url = "package://mbzirc2020_task1_common/urdf/meshes/sensor/single_camera_center_bar.dae">
-        <origin xyz="${link_length / 2 + 0.0605} 0.2395 0.0502" rpy="0 0 ${pi * 3/4}"/>
+        <origin xyz="${link_length / 2 + 0.0605} 0.2395 0.0402" rpy="0 ${0.05} ${pi * 3/4 + 0.05}"/> <!-- copy the diret mount type, TODO: calibrate by rviz camera plugin -->
         <inertial>
           <mass value = "0.0233" />

Commit message: Mass value could not be 0 in urdf file.

File: mbzirc2020/mbzirc2020_task1/mbzirc2020_task1_common/robots/hydrus.urdf.xacro (robot description, xacro)
@@ -63,5 +63,5 @@
         <origin xyz="0.016 0.0 0.005 " rpy="0 0 0"/>
         <inertial>
-          <mass value = "0.0" />
+          <mass value = "0.00001" />
           <origin xyz="0 0 0" rpy="0 0 0"/>
           <inertia

Commit message: Update the robot model:     - the urdf files regarding the sensor modules     - camera calibration files     - the delay launch for realsense d435 because of the conflict with realsense t265

File: mbzirc2020/mbzirc2020_task1/mbzirc2020_task1_common/robots/hydrus.urdf.xacro (robot description, xacro)
@@ -31,5 +31,5 @@
     </inertial>
   </xacro:extra_module>
-  <!-- 1.3 processor: gygabyte brix i7 -->
+  <!-- processor: gygabyte brix i7 -->
   <xacro:extra_module name = "pc" parent = "link2" visible = "1"
                       model_url = "package://mbzirc2020_common/urdf/mesh/modules/processor/gygabyte_brix_fixed_joint_unit.STL" >
@@ -45,4 +45,16 @@
   </xacro:extra_module>
   <!-- end: gygabyte brix i7 -->
+  <!-- edge TPU coral -->
+  <xacro:extra_module name = "edgetpu" parent = "link2" visible = "0" >
+    <origin xyz="${link_length / 2 + 0.22} 0.01 0.02" rpy="0 0 0"/>
+    <inertial>
+      <mass value = "0.0348" /> <!-- plus usb cable -->
+      <origin xyz="0 0 0" rpy="0 0 0"/>
+      <inertia
+          ixx="0.0" ixy="0.0" ixz="0.0"
+          iyy="0.0" iyz="0.0" izz="0.0"/>
+    </inertial>
+  </xacro:extra_module>
+  <!-- end: edge TPU coral -->
   <!-- sensor -->
   <!-- Monocular camera -->
@@ -51,24 +63,19 @@
     <xacro:unless value="$(arg camera_height)">
       <xacro:extra_module name = "monocular_camera_unit" parent = "link2" visible = "1" model_url = "package://mbzirc2020_task1_common/urdf/meshes/sensor/ELP_SUSB1080P_direct_unit.dae">
-        <origin xyz="${link_length / 2 + 0.0605} 0.2395 0.0402" rpy="0 ${0.05} ${pi * 3/4 + 0.05}"/> <!-- calibrate by rviz camera plugin -->w
+        <origin xyz="${link_length / 2 + 0.0605} 0.2395 0.0502" rpy="0 0.05 ${pi * 3/4}"/>
         <inertial>
-          <mass value = "0.0435" />
-          <origin xyz="0.011 0 0.005" rpy="0 0 0"/>
+          <mass value = "0.0457" />
+          <origin xyz="0.027 0 0.005" rpy="0 0 0"/>
           <inertia
-              ixx="0.0" iyy="0.0" izz="0.0"
+              ixx="0.000062" iyy="0.000009" izz="0.000066"
               ixy="0.0" ixz="0.0" iyz="0.0"/>
         </inertial>
       </xacro:extra_module>
-      <xacro:extra_module name = "color_camera_frame" parent = "monocular_camera_unit" visible = "0" >
+      <joint name="monocular_camera_unit2color_camera_frame" type="fixed">
         <origin xyz="0.016 0.0 0.005 " rpy="0 0 0"/>
-        <inertial>
-          <mass value = "0.00001" />
-          <origin xyz="0 0 0" rpy="0 0 0"/>
-          <inertia
-              ixx="0.0" ixy="0.0" ixz="0.0"
-              iyy="0.0" iyz="0.0"
-              izz="0.0"/>
-        </inertial>
-      </xacro:extra_module>
+        <parent link="monocular_camera_unit" />
+        <child link="color_camera_frame" />
+      </joint>
+      <link name="color_camera_frame"/>
       <xacro:extra_module name = "camera_usb_cable" parent = "monocular_camera_unit" visible = "0" >
         <origin xyz="-0.13 0 0 " rpy="0 0 0"/>
@@ -86,15 +93,15 @@
     <xacro:if value="$(arg camera_height)">
       <xacro:extra_module name = "center_bar" parent = "link2" visible = "1" model_url = "package://mbzirc2020_task1_common/urdf/meshes/sensor/single_camera_center_bar.dae">
-        <origin xyz="${link_length / 2 + 0.0605} 0.2395 0.0402" rpy="0 ${0.05} ${pi * 3/4 + 0.05}"/> <!-- copy the diret mount type, TODO: calibrate by rviz camera plugin -->
+        <origin xyz="${link_length / 2 + 0.0605} 0.2395 0.0502" rpy="0 0.05 ${pi * 3/4}"/>
         <inertial>
-          <mass value = "0.0233" />
-          <origin xyz="-0.003 0 -0.01" rpy="0 0 0"/>
+          <mass value = "0.0255" />
+          <origin xyz="0.014307 0 0.005" rpy="0 0 0"/>
           <inertia
-              ixx="0.0" iyy="0.0" izz="0.0"
+              ixx="0.000058" iyy="0.0" izz="0.000059"
               ixy="0.0" ixz="0.0" iyz="0.0"/>
         </inertial>
       </xacro:extra_module>
       <xacro:extra_module name = "monocular_camera_unit" parent = "center_bar" visible = "1" model_url = "package://mbzirc2020_task1_common/urdf/meshes/sensor/ELP_SUSB1080P_unit.dae">
-        <origin xyz="0.001 0 $(arg camera_height)" rpy="0 0 0"/>
+        <origin xyz="0.02014 0 $(arg camera_height)" rpy="0 0 0"/>
         <inertial>
           <mass value = "0.036" />
@@ -116,38 +123,28 @@
         </inertial>
       </xacro:extra_module>
-      <xacro:extra_module name = "color_camera_frame" parent = "monocular_camera_unit" visible = "0" >
+      <joint name="monocular_camera_unit2color_camera_frame" type="fixed">
         <origin xyz="0.0 0.0 0.0 " rpy="${pi} 0 0"/>
-        <inertial>
-          <mass value = "0.0" />
-          <origin xyz="0 0 0" rpy="0 0 0"/>
-          <inertia
-              ixx="0.0" ixy="0.0" ixz="0.0"
-              iyy="0.0" iyz="0.0"
-              izz="0.0"/>
-        </inertial>
-      </xacro:extra_module>
+        <parent link="monocular_camera_unit" />
+        <child link="color_camera_frame" />
+      </joint>
+      <link name="color_camera_frame"/>
     </xacro:if>
-    <xacro:extra_module name = "color_camera_optical_frame" parent = "color_camera_frame" visible = "0" >
+    <joint name="color_camera_frame2color_camera_optical_frame" type="fixed">
       <origin xyz="0.0 0.0 0.0 " rpy="${-pi/2} 0 ${-pi/2}"/>
-      <inertial>
-        <mass value = "0.0" />
-        <origin xyz="0 0 0" rpy="0 0 0"/>
-        <inertia
-            ixx="0.0" ixy="0.0" ixz="0.0"
-            iyy="0.0" iyz="0.0"
-            izz="0.0"/>
-      </inertial>
-    </xacro:extra_module>
+      <parent link="color_camera_frame" />
+      <child link="color_camera_optical_frame" />
+    </joint>
+    <link name="color_camera_optical_frame"/>
   </xacro:if>
   <!-- Realsense D435 -->
   <xacro:unless value="$(arg monocular_camera)">
-    <xacro:extra_module name = "rs_d435_unit" parent = "link2" visible = "1" model_url = "package://mbzirc2020_task1_common/urdf/meshes/sensor/rs_d435_unit3_center_bar.dae">
+    <xacro:extra_module name = "rs_d435_unit" parent = "link2" visible = "1" model_url = "package://mbzirc2020_task1_common/urdf/meshes/sensor/rs_d435_unit3_front_center_bar.dae">
       <origin xyz="${link_length / 2 + 0.0605} 0.2395 0.0502" rpy="0 0 ${pi * 3/4}"/>
       <inertial>
-        <mass value = "0.07669" /> <!-- includes sensor and mount -->
-        <origin xyz="0.014374 0 0.01599" rpy="0 0 0"/>
+        <mass value = "0.0789" /> <!-- includes sensor and mount -->
+        <origin xyz="0.0315 -0.0247 0.01568" rpy="0 0 0"/>
         <inertia
-            ixx="0.000088" iyy="0.000012" izz="0.000089"
-            ixy="0" ixz="0" iyz="0"/>
+            ixx="0.000111" iyy="0.000016" izz="0.000116"
+            ixy="-0.000008" ixz="0.000004" iyz="-0.00005"/>
       </inertial>
     </xacro:extra_module>
@@ -165,5 +162,5 @@
     <!-- rs_d435_link is the parrent of sensors' frame, identical to rs_d435_left_ir_frame -->
     <xacro:extra_module name = "rs_d435_link" parent = "rs_d435_unit" visible = "0" >
-      <origin xyz="0.03 0.0175 0.019 " rpy="0 0 0"/>
+      <origin xyz="0.03 -0.015 0.019 " rpy="0 0 0"/>
       <inertial>
         <mass value = "0.0" />

Commit message: - Refine the rosbag record script - Modify the teleop parameter - Slightly change the net configuration in urdf

File: mbzirc2020/mbzirc2020_task1/mbzirc2020_task1_common/robots/hydrus.urdf.xacro (robot description, xacro)
@@ -174,5 +174,5 @@
   </xacro:unless>
   <!-- net -->
-  <xacro:property name="net_mass" value=".035" />
+  <xacro:property name="net_mass" value=".03" />
   <xacro:extra_module name = "net_anchor1" parent = "leg1" visible = "0" >
     <origin xyz="0.0 0.0 0.0" rpy="0 0 0"/>
