Commit message: - Change the weight of the net. - Fix the bug about the wrong pitch angle of the monocular camera, and this camera as a parameter which can be set from bringup.launch

File: mbzirc2020/mbzirc2020_task1/mbzirc2020_task1_common/robots/hydrus.urdf.xacro (robot description, xacro)
@@ -5,4 +5,5 @@
   <xacro:arg name="monocular_camera" default="true" />
   <xacro:arg name="camera_height" default="0" />
+  <xacro:arg name="camera_pitch_angle" default="0" />
   <xacro:arg name="horizontal_vio" default="false" />
   <xacro:include filename="$(find mbzirc2020_common)/robots/default.urdf.xacro" />
@@ -63,5 +64,5 @@
     <xacro:unless value="$(arg camera_height)">
       <xacro:extra_module name = "monocular_camera_unit" parent = "link2" visible = "1" model_url = "package://mbzirc2020_task1_common/urdf/meshes/sensor/ELP_SUSB1080P_direct_unit.dae">
-        <origin xyz="${link_length / 2 + 0.0605} 0.2395 0.0502" rpy="0 0.05 ${pi * 3/4}"/>
+        <origin xyz="${link_length / 2 + 0.0605} 0.2395 0.0502" rpy="0 $(arg camera_pitch_angle) ${pi * 3/4}"/>
         <inertial>
           <mass value = "0.0457" />
@@ -93,5 +94,5 @@
     <xacro:if value="$(arg camera_height)">
       <xacro:extra_module name = "center_bar" parent = "link2" visible = "1" model_url = "package://mbzirc2020_task1_common/urdf/meshes/sensor/single_camera_center_bar.dae">
-        <origin xyz="${link_length / 2 + 0.0605} 0.2395 0.0502" rpy="0 0.05 ${pi * 3/4}"/>
+        <origin xyz="${link_length / 2 + 0.0605} 0.2395 0.0502" rpy="0 $(arg camera_pitch_angle) ${pi * 3/4}"/>
         <inertial>
           <mass value = "0.0255" />
@@ -174,5 +175,5 @@
   </xacro:unless>
   <!-- net -->
-  <xacro:property name="net_mass" value=".03" />
+  <xacro:property name="net_mass" value=".06" />
   <xacro:extra_module name = "net_anchor1" parent = "leg1" visible = "0" >
     <origin xyz="0.0 0.0 0.0" rpy="0 0 0"/>

Commit message: temp.

File: mbzirc2020/mbzirc2020_task1/mbzirc2020_task1_common/robots/hydrus.urdf.xacro (robot description, xacro)
@@ -174,6 +174,27 @@
     </xacro:extra_module>
   </xacro:unless>
+  <!-- upward carbon pipe to avoid upside down crash on the ground -->
+  <xacro:extra_module name = "upward_pipe1" parent = "link2" visible = "0" >
+    <origin xyz="0.04 0.0 0.04" rpy="0 0 0"/>
+    <inertial>
+      <origin xyz="0 0 0" rpy="0 0 0"/>
+      <mass value="0.01"/>
+      <inertia
+          ixx="0.0" iyy="0.0" izz="0.0"
+          ixy="0.0" ixz="0.0"  iyz="0.0"/>
+    </inertial>
+  </xacro:extra_module>
+  <xacro:extra_module name = "upward_pipe2" parent = "link3" visible = "0" >
+    <origin xyz="0.56 0.0 0.04" rpy="0 0 0"/>
+    <inertial>
+      <origin xyz="0 0 0" rpy="0 0 0"/>
+      <mass value="0.01"/>
+      <inertia
+          ixx="0.0" iyy="0.0" izz="0.0"
+          ixy="0.0" ixz="0.0"  iyz="0.0"/>
+    </inertial>
+  </xacro:extra_module>
   <!-- net -->
-  <xacro:property name="net_mass" value=".06" />
+  <xacro:property name="net_mass" value=".075" />
   <xacro:extra_module name = "net_anchor1" parent = "leg1" visible = "0" >
     <origin xyz="0.0 0.0 0.0" rpy="0 0 0"/>
