Commit message: add ground model

File: mbzirc2020/mbzirc2020_common/robots/default.urdf.xacro (robot description, xacro)
@@ -6,10 +6,10 @@
   <xacro:include filename="$(find hydrus)/urdf/link.urdf.xacro" />
   <xacro:include filename="$(find mbzirc2020_common)/urdf/fixed_link.urdf.xacro" />
-  <xacro:macro name="robot_model" params="tilt_angle:=0 horizontal_vio:=0 default_battery:=1">
+  <xacro:macro name="robot_model" params="tilt_angle:=0 horizontal_vio:=0 default_battery:=1 ground_mode:=0">
     <xacro:if value="${tilt_angle == 0}"> <!--no tilt angle-->
-      <xacro:hydrusx_link links="4" self="1" rotor_direction="-1" with_battery = "${default_battery}" tilt_mode="0" />
-      <xacro:hydrusx_fixed_link self="2" rotor_direction="1"  with_battery = "${default_battery}" tilt_angle = "0" />
+      <xacro:hydrusx_link links="4" self="1" rotor_direction="-1" with_battery = "${default_battery}" tilt_mode="0" with_leg = "${1- ground_mode}" />
+      <xacro:hydrusx_fixed_link self="2" rotor_direction="1"  with_battery = "${default_battery}" tilt_angle = "0" with_leg = "${1- ground_mode}" />
       <xacro:hydrusx_fixed_link self="3" rotor_direction="-1" with_battery = "${default_battery}" tilt_angle = "0" />
-      <xacro:hydrusx_link links="4" self="4" rotor_direction="1"  with_battery = "${default_battery}" tilt_mode="0" />
+      <xacro:hydrusx_link links="4" self="4" rotor_direction="1"  with_battery = "${default_battery}" tilt_mode="0" with_leg = "${1- ground_mode}" />
     </xacro:if>
     <xacro:unless value="${tilt_angle == 0}">

File: mbzirc2020/mbzirc2020_common/urdf/fixed_link.urdf.xacro (robot description, xacro)
@@ -2,5 +2,5 @@
 <robot
     xmlns:xacro="http://www.ros.org/wiki/xacro" name="hydrusx_fixed_link" >
-  <xacro:macro name="hydrusx_fixed_link" params="self rotor_direction with_battery:=1 tilt_angle:=0">
+  <xacro:macro name="hydrusx_fixed_link" params="self rotor_direction with_battery:=1 tilt_angle:=0 with_leg:=1">
     <!-- link -->
     <link name="link${self}">
@@ -110,7 +110,9 @@
     <xacro:if value="${self == 2}">
       <!-- leg -->
-      <xacro:standard_leg_joint parent = "link${self}" >
-        <origin xyz="0.0 0.0 0" rpy="0 0 0"/>
-      </xacro:standard_leg_joint>
+      <xacro:if value="${with_leg == 1}">
+	<xacro:standard_leg_joint parent = "link${self}" >
+          <origin xyz="0.0 0.0 0" rpy="0 0 0"/>
+	</xacro:standard_leg_joint>
+      </xacro:if>
       <!-- fixed joint  -->
       <joint name="joint${self}" type="fixed">

File: mbzirc2020/mbzirc2020_task2/mbzirc2020_task2_common/robots/hydrus.urdf.xacro (robot description, xacro)
@@ -2,7 +2,10 @@
 <robot
     xmlns:xacro="http://www.ros.org/wiki/xacro" name="hydrusx" >
+  <!-- ground_mode flag -->
+  <xacro:property name="ground_mode" value="0" />
+  <xacro:property name="fixed_leg" value="0" />
   <!-- base kinematics model -->
   <xacro:include filename="$(find mbzirc2020_common)/robots/default.urdf.xacro" />
-  <xacro:robot_model tilt_angle = "10" horizontal_vio = "0" default_battery = "1"  />
+  <xacro:robot_model tilt_angle = "0" horizontal_vio = "0" default_battery = "1" ground_mode = "${ground_mode}" />
   <!-- processor: intel upboard -->
   <!-- TODO: change to brix -->
@@ -84,3 +87,218 @@
   <!-- gripper -->
   <!-- TODO: add gripper at the ends -->
+  <!-- actuated and omni leg when ground_mode -->
+  <xacro:if value = "${ground_mode}">
+    <!-- actuated legs -->
+    <!-- in the second link -->
+    <xacro:extra_module name = "actuated_leg1_stationary_part" parent = "link2" visible = "1"
+  			model_url = "package://mbzirc2020_task2_common/urdf/mesh/modules/mechanical/actuated_leg_stationary_part.dae">
+      <origin xyz="${head_leg_offset} 0 0" rpy="${-pi/2} 0 0"/>
+      <inertial>
+  	<mass value = "0.142" />
+  	<origin xyz="0 0 0" rpy="0 0 0"/>
+  	<inertia
+            ixx="0.0001" ixy="0.0" ixz="0.0"
+            iyy="0.0001" iyz="0.0"
+            izz="0.0001"/>
+      </inertial>
+    </xacro:extra_module>
+    <xacro:if value="${fixed_leg}">
+      <joint name="actuated_leg1_joint" type="fixed">
+  	<parent link="actuated_leg1_stationary_part"/>
+  	<child link="actuated_leg1_movable_part"/>
+  	<origin rpy="${-pi/2} 0 ${pi}" xyz="-0.0115 0.1042 0"/>
+  	<axis xyz="0 0 -1"/>
+      </joint>
+    </xacro:if>
+    <xacro:unless value="${fixed_leg == 1}">
+      <joint name="actuated_leg1_joint" type="prismatic">
+    	<limit effort="50" lower="0" upper="0.0927" velocity="1"/>
+    	<parent link="actuated_leg1_stationary_part"/>
+    	<child link="actuated_leg1_movable_part"/>
+    	<origin rpy="${-pi/2} 0 ${pi}" xyz="-0.0115 0 0"/> <!-- TODO: tune -y -->
+    	<axis xyz="0 0 -1"/>
+    	<dynamics damping="0.1" friction="0.01"/>
+      </joint>
+      <transmission name="actuated_leg1_joint_tran">
+    	<type>transmission_interface/SimpleTransmission</type>
+    	<joint name="actuated_leg1_joint">
+    	  <hardwareInterface>hardware_interface/EffortJointInterface</hardwareInterface>
+    	</joint>
+    	<actuator name="actuated_leg1_joint">
+    	  <hardwareInterface>hardware_interface/EffortJointInterface</hardwareInterface>
+    	  <mechanicalReduction>1</mechanicalReduction>
+    	</actuator>
+      </transmission>
+    </xacro:unless>
+    <link name="actuated_leg1_movable_part">
+      <inertial>
+  	<origin xyz="-0.002860 0.000000 -0.089840" rpy="0 0 0"/>
+  	<mass value="0.107000"/>
+  	<inertia
+            ixx="0.002466" iyy="0.003026" izz="0.000699"
+            ixy="0.000150" ixz="0.001147" iyz="0.000280"/>
+      </inertial>
+      <visual>
+  	<origin xyz="0 0 0" rpy="${-pi/2} 0 0"/>
+  	<geometry>
+          <mesh filename="package://mbzirc2020_task2_common/urdf/mesh/modules/mechanical/actuated_leg_movable_part.dae"/>
+  	</geometry>
+      </visual>
+      <collision>
+  	<origin rpy="0 0 0" xyz="0.0025 0 -0.128"/>
+  	<geometry>
+          <sphere radius="${55 / 2 * 0.001}"/>
+  	</geometry>
+      </collision>
+    </link>
+    <!-- in the thrid links -->
+    <xacro:extra_module name = "actuated_leg2_stationary_part" parent = "link3" visible = "1"
+  			model_url = "package://mbzirc2020_task2_common/urdf/mesh/modules/mechanical/actuated_leg_stationary_part.dae">
+      <origin xyz="${end_leg_offset} 0.0 0" rpy="${-pi/2} 0 ${pi}"/>
+      <inertial>
+  	<mass value = "0.142" />
+  	<origin xyz="0 0 0" rpy="0 0 0"/>
+  	<inertia
+            ixx="0.0001" ixy="0.0" ixz="0.0"
+            iyy="0.0001" iyz="0.0"
+            izz="0.0001"/>
+      </inertial>
+    </xacro:extra_module>
+    <xacro:if value="${fixed_leg}">
+      <joint name="actuated_leg2_joint" type="fixed">
+  	<parent link="actuated_leg2_stationary_part"/>
+  	<child link="actuated_leg2_movable_part"/>
+  	<origin rpy="${-pi/2} 0 ${pi}" xyz="-0.0115 0.1042 0"/>
+  	<axis xyz="0 0 -1"/>
+      </joint>
+    </xacro:if>
+    <xacro:unless value="${fixed_leg == 1}">
+      <joint name="actuated_leg2_joint" type="prismatic">
+    	<limit effort="50" lower="0" upper="0.0927" velocity="1"/>
+    	<parent link="actuated_leg2_stationary_part"/>
+    	<child link="actuated_leg2_movable_part"/>
+    	<origin rpy="${-pi/2} 0 ${pi}" xyz="-0.0115 0 0"/> <!-- TODO: tune -y -->
+    	<axis xyz="0 0 -1"/>
+    	<dynamics damping="0.1" friction="0.01"/>
+      </joint>
+      <transmission name="actuated_leg2_joint_tran">
+    	<type>transmission_interface/SimpleTransmission</type>
+    	<joint name="actuated_leg2_joint">
+    	  <hardwareInterface>hardware_interface/EffortJointInterface</hardwareInterface>
+    	</joint>
+    	<actuator name="actuated_leg2_joint">
+    	  <hardwareInterface>hardware_interface/EffortJointInterface</hardwareInterface>
+    	  <mechanicalReduction>1</mechanicalReduction>
+    	</actuator>
+      </transmission>
+    </xacro:unless>
+    <link name="actuated_leg2_movable_part">
+      <inertial>
+  	<origin xyz="-0.002860 0.000000 -0.089840" rpy="0 0 0"/>
+  	<mass value="0.107000"/>
+  	<inertia
+            ixx="0.002466" iyy="0.003026" izz="0.000699"
+            ixy="0.000150" ixz="0.001147" iyz="0.000280"/>
+      </inertial>
+      <visual>
+  	<origin xyz="0 0 0" rpy="${-pi/2} 0 0"/>
+  	<geometry>
+          <mesh filename="package://mbzirc2020_task2_common/urdf/mesh/modules/mechanical/actuated_leg_movable_part.dae"/>
+  	</geometry>
+      </visual>
+      <collision>
+  	<origin rpy="0 0 0" xyz="0.0025 0 -0.128"/>
+  	<geometry>
+          <sphere radius="${55 / 2 * 0.001}"/>
+  	</geometry>
+      </collision>
+    </link>
+    <!-- omniwheel normal legs -->
+    <!-- in the first link -->
+    <joint name="link1_to_leg1" type="fixed">
+      <parent link="link1"/>
+      <child link="omni_leg1"/>
+      <origin xyz="${head_leg_offset} 0.0 0" rpy="0 0 0"/>
+      <origin rpy="0 0 0" xyz="-0.0115 0 -0.0115"/>
+      <axis xyz="0 0 0"/>
+    </joint>
+    <link name="omni_leg1">
+      <inertial>
+  	<origin xyz="0.000000 0.000000 -0.093340" rpy="0 0 0"/>
+  	<mass value="0.072000"/>
+  	<inertia
+            ixx="-0.000617" iyy="-0.000627" izz="0.0000"
+            ixy="0.000000" ixz="0.000000" iyz="0.000000"/>
+      </inertial>
+      <visual>
+  	<origin xyz="0 0 0" rpy="${-pi/2} 0 0"/>
+  	<geometry>
+          <mesh filename="package://mbzirc2020_task2_common/urdf/mesh/modules/mechanical/passive_stationary_part.dae"/>
+  	</geometry>
+      </visual>
+      <collision>
+        <origin rpy="0 0 0" xyz="0 -0.002 -0.14"/>
+        <geometry>
+          <sphere radius="${55 / 2 * 0.001}"/>
+        </geometry>
+      </collision>
+    </link>
+    <!-- in the forth link -->
+    <joint name="link4_to_leg3" type="fixed">
+      <parent link="link4"/>
+      <child link="omni_leg2"/>
+      <origin xyz="${end_leg_offset} 0.0 0" rpy="0 0 0"/>
+      <origin rpy="0 0 0" xyz="-0.0115 0 -0.0115"/>
+      <axis xyz="0 0 0"/>
+    </joint>
+    <link name="omni_leg2">
+      <inertial>
+  	<origin xyz="0.000000 0.000000 -0.093340" rpy="0 0 0"/>
+  	<mass value="0.072000"/>
+  	<inertia
+            ixx="-0.000617" iyy="-0.000627" izz="0.0000"
+            ixy="0.000000" ixz="0.000000" iyz="0.000000"/>
+      </inertial>
+      <visual>
+  	<origin xyz="0 0 0" rpy="${-pi/2} 0 0"/>
+  	<geometry>
+          <mesh filename="package://mbzirc2020_task2_common/urdf/mesh/modules/mechanical/passive_stationary_part.dae"/>
+  	</geometry>
+      </visual>
+      <collision>
+        <origin rpy="0 0 0" xyz="0 -0.002 -0.14"/>
+        <geometry>
+          <sphere radius="${55 / 2 * 0.001}"/>
+        </geometry>
+      </collision>
+    </link>
+    <gazebo reference="actuated_leg1_movable_part">
+      <mu1>0.11</mu1>
+      <mu2>0.11</mu2>
+      <fdir1>1 1 0</fdir1>
+      <minDepth>0.00</minDepth>
+      <selfCollide>false</selfCollide>
+    </gazebo>
+    <gazebo reference="actuated_leg2_movable_part">
+      <mu1>0.11</mu1>
+      <mu2>0.11</mu2>
+      <fdir1>1 1 0</fdir1>
+      <minDepth>0.00</minDepth>
+      <selfCollide>false</selfCollide>
+    </gazebo>
+    <gazebo reference="omni_leg1">
+      <mu1>0.11</mu1>
+      <mu2>0.11</mu2>
+      <fdir1>1 1 0</fdir1>
+      <minDepth>0.00</minDepth>
+      <selfCollide>false</selfCollide>
+    </gazebo>
+    <gazebo reference="omni_leg2">
+      <mu1>0.11</mu1>
+      <mu2>0.11</mu2>
+      <fdir1>1 1 0</fdir1>
+      <minDepth>0.00</minDepth>
+      <selfCollide>false</selfCollide>
+    </gazebo>
+  </xacro:if>
 </robot>

Commit message: MBZIRC2020_common:  1. add arg `model_suffix` to support derived model in each task (e.g., ground model in task2)
MBZIRC2020_task2:
 1. add ground model. Please follow mbzirc2020_task2/README.md

File: mbzirc2020/mbzirc2020_common/robots/default.urdf.xacro (robot description, xacro)
@@ -6,16 +6,16 @@
   <xacro:include filename="$(find hydrus)/urdf/link.urdf.xacro" />
   <xacro:include filename="$(find mbzirc2020_common)/urdf/fixed_link.urdf.xacro" />
-  <xacro:macro name="robot_model" params="tilt_angle:=0 horizontal_vio:=0 default_battery:=1">
+  <xacro:macro name="robot_model" params="tilt_angle:=0 horizontal_vio:=0 default_battery:=1 with_leg:=1">
     <xacro:if value="${tilt_angle == 0}"> <!--no tilt angle-->
-      <xacro:hydrusx_link links="4" self="1" rotor_direction="-1" with_battery = "${default_battery}" tilt_mode="0" />
-      <xacro:hydrusx_fixed_link self="2" rotor_direction="1"  with_battery = "${default_battery}" tilt_angle = "0" />
-      <xacro:hydrusx_fixed_link self="3" rotor_direction="-1" with_battery = "${default_battery}" tilt_angle = "0" />
-      <xacro:hydrusx_link links="4" self="4" rotor_direction="1"  with_battery = "${default_battery}" tilt_mode="0" />
+      <xacro:hydrusx_link links="4" self="1" rotor_direction="-1" with_battery = "${default_battery}" with_leg = "${with_leg}" tilt_mode="0" />
+      <xacro:hydrusx_fixed_link self="2" rotor_direction="1"  with_battery = "${default_battery}" with_leg = "${with_leg}" tilt_angle = "0" />
+      <xacro:hydrusx_fixed_link self="3" rotor_direction="-1" with_battery = "${default_battery}" with_leg = "${with_leg}" tilt_angle = "0" />
+      <xacro:hydrusx_link links="4" self="4" rotor_direction="1"  with_battery = "${default_battery}" with_leg = "${with_leg}" tilt_mode="0" />
     </xacro:if>
     <xacro:unless value="${tilt_angle == 0}">
-      <xacro:hydrusx_link links="4" self="1" rotor_direction="-1" with_battery = "${default_battery}" tilt_mode="1" tilt_angle="${tilt_angle}" />
-      <xacro:hydrusx_fixed_link self="2" rotor_direction="1"  with_battery = "${default_battery}" tilt_angle = "${tilt_angle}" />
-      <xacro:hydrusx_fixed_link self="3" rotor_direction="-1" with_battery = "${default_battery}" tilt_angle = "${tilt_angle}" />
-      <xacro:hydrusx_link links="4" self="4" rotor_direction="1"  with_battery = "${default_battery}" tilt_mode="1" tilt_angle="${tilt_angle}"/>
+      <xacro:hydrusx_link links="4" self="1" rotor_direction="-1" with_battery = "${default_battery}" with_leg = "${with_leg}" tilt_mode="1" tilt_angle="${tilt_angle}" />
+      <xacro:hydrusx_fixed_link self="2" rotor_direction="1"  with_battery = "${default_battery}" with_leg = "${with_leg}" tilt_angle = "${tilt_angle}" />
+      <xacro:hydrusx_fixed_link self="3" rotor_direction="-1" with_battery = "${default_battery}" with_leg = "${with_leg}" tilt_angle = "${tilt_angle}" />
+      <xacro:hydrusx_link links="4" self="4" rotor_direction="1"  with_battery = "${default_battery}" with_leg = "${with_leg}" tilt_mode="1" tilt_angle="${tilt_angle}"/>
     </xacro:unless>
     <!-- onboard -->

File: mbzirc2020/mbzirc2020_common/urdf/fixed_link.urdf.xacro (robot description, xacro)
@@ -2,5 +2,5 @@
 <robot
     xmlns:xacro="http://www.ros.org/wiki/xacro" name="hydrusx_fixed_link" >
-  <xacro:macro name="hydrusx_fixed_link" params="self rotor_direction with_battery:=1 tilt_angle:=0">
+  <xacro:macro name="hydrusx_fixed_link" params="self rotor_direction with_battery:=1 with_leg:=1 tilt_angle:=0">
     <!-- link -->
     <link name="link${self}">
@@ -110,7 +110,9 @@
     <xacro:if value="${self == 2}">
       <!-- leg -->
-      <xacro:standard_leg_joint parent = "link${self}" >
-        <origin xyz="0.0 0.0 0" rpy="0 0 0"/>
-      </xacro:standard_leg_joint>
+      <xacro:if value="${with_leg == 1}">
+        <xacro:standard_leg_joint parent = "link${self}" >
+          <origin xyz="0.0 0.0 0" rpy="0 0 0"/>
+        </xacro:standard_leg_joint>
+      </xacro:if>
       <!-- fixed joint  -->
       <joint name="joint${self}" type="fixed">

File: mbzirc2020/mbzirc2020_task2/mbzirc2020_task2_common/robots/hydrus.gazebo.xacro (robot description, xacro)
@@ -16,5 +16,5 @@
           <width>1280</width>
           <height>720</height>
-          <format>RGB</format>
+          <format>B8G8R8</format>
         </image>
         <clip>

File: mbzirc2020/mbzirc2020_task2/mbzirc2020_task2_common/robots/hydrus.urdf.xacro (robot description, xacro)
@@ -4,5 +4,28 @@
   <!-- base kinematics model -->
   <xacro:include filename="$(find mbzirc2020_common)/robots/default.urdf.xacro" />
-  <xacro:robot_model tilt_angle = "10" horizontal_vio = "0" default_battery = "1"  />
+  <xacro:robot_model tilt_angle = "10" horizontal_vio = "0" default_battery = "0"  />
+  <!-- special battery arrangement -->
+  <xacro:extra_module name = "bat1" parent = "link1" visible = "1"
+                      model_url = "package://hydrus/urdf/mesh/battery/Kypom-3000-6s.dae" scale="0.001">
+    <origin xyz="${link_length/2} 0.0 -0.048" rpy="0 0 0"/>
+    <inertial>
+      <origin xyz="0 0 0" rpy="0 0 0"/>
+      <mass value="0.4108"/>
+      <inertia
+          ixx="0.0001" iyy="0.0006" izz="0.0006"
+          ixy="0.0" ixz="0.0"  iyz="0.0"/>
+    </inertial>
+  </xacro:extra_module>
+  <xacro:extra_module name = "bat2" parent = "link4" visible = "1"
+                      model_url = "package://hydrus/urdf/mesh/battery/Kypom-3000-6s.dae" scale="0.001">
+    <origin xyz="${link_length/2} 0.0 -0.048" rpy="0 0 0"/>
+    <inertial>
+      <origin xyz="0 0 0" rpy="0 0 0"/>
+      <mass value="0.4108"/>
+      <inertia
+          ixx="0.0001" iyy="0.0006" izz="0.0006"
+          ixy="0.0" ixz="0.0"  iyz="0.0"/>
+    </inertial>
+  </xacro:extra_module>
   <!-- processor: intel upboard -->
   <!-- TODO: change to brix -->

Commit message: Add flag to disable the downward vio (realsense t265) in default robot urdf file

File: mbzirc2020/mbzirc2020_common/robots/default.urdf.xacro (robot description, xacro)
@@ -6,5 +6,5 @@
   <xacro:include filename="$(find hydrus)/urdf/link.urdf.xacro" />
   <xacro:include filename="$(find mbzirc2020_common)/urdf/fixed_link.urdf.xacro" />
-  <xacro:macro name="robot_model" params="tilt_angle:=0 horizontal_vio:=0 default_battery:=1 with_leg:=1">
+  <xacro:macro name="robot_model" params="tilt_angle:=0 downward_vio:=1 horizontal_vio:=0 default_battery:=1 with_leg:=1">
     <xacro:if value="${tilt_angle == 0}"> <!--no tilt angle-->
       <xacro:hydrusx_link links="4" self="1" rotor_direction="-1" with_battery = "${default_battery}" with_leg = "${with_leg}" tilt_mode="0" />
@@ -88,16 +88,18 @@
     <!-- end: gps -->
     <!-- 2.3 downwards rs-t265 (VIO) -->
-    <xacro:extra_module name = "realsense1_pose_frame" parent = "link2" visible = "1"
-                        model_url = "package://mbzirc2020_common/urdf/mesh/modules/sensor/downward_realsense_unit.STL">
-      <origin xyz="${link_length/2 + 0.127} 0.0 -0.022" rpy="0 ${pi/2} ${pi/2}"/>
-      <inertial>
-        <mass value = "0.065" /> <!-- sensor + usb-cable -->
-        <origin xyz="-0.009 -0.01 0" rpy="0 0 0"/>
-        <inertia
-            ixx="0.0" ixy="0.0" ixz="0.0"
-            iyy="0.0" iyz="0.0"
-            izz="0.0"/>
-      </inertial>
-    </xacro:extra_module>
+    <xacro:if value="${downward_vio == 1}">
+      <xacro:extra_module name = "realsense1_pose_frame" parent = "link2" visible = "1"
+                          model_url = "package://mbzirc2020_common/urdf/mesh/modules/sensor/downward_realsense_unit.STL">
+	<origin xyz="${link_length/2 + 0.127} 0.0 -0.022" rpy="0 ${pi/2} ${pi/2}"/>
+	<inertial>
+          <mass value = "0.065" /> <!-- sensor + usb-cable -->
+          <origin xyz="-0.009 -0.01 0" rpy="0 0 0"/>
+          <inertia
+              ixx="0.0" ixy="0.0" ixz="0.0"
+              iyy="0.0" iyz="0.0"
+              izz="0.0"/>
+	</inertial>
+      </xacro:extra_module>
+    </xacro:if>
     <!-- end: rs-5265 -->
     <!-- 2.4 horizontal rs-t265 (option VIO) -->
@@ -116,4 +118,5 @@
         </xacro:extra_module>
     </xacro:if>
+    <!-- end: rs-5265 -->
   </xacro:macro>
 </robot>
