Commit message: Enable multiple robot bringup in single gazebo world. Please refer to https://github.com/tongtybj/aerial_robot/pull/399

File: mbzirc2020/mbzirc2020_common/robots/default.gazebo.xacro (robot description, xacro)
@@ -1,41 +1,8 @@
 <?xml version="1.0"?>
 <robot
-    xmlns:xacro="http://www.ros.org/wiki/xacro" name="hydrusx" >
-  <!-- gazebo elements: hw interface -->
-  <gazebo>
-    <plugin name="gazebo_ros_control" filename="libgazebo_ros_control.so">
-      <robotNamespace>/hydrusx</robotNamespace>
-      <!-- <robotSimType>gazebo_ros_control/DefaultRobotHWSim</robotSimType> -->
-      <robotSimType>gazebo_ros_control/AerialRobotHWSim</robotSimType>
-    </plugin>
-  </gazebo>
-  <!-- imu plugin -->
-  <gazebo reference="fc">
-    <gravity>true</gravity>
-    <sensor name="imu_sensor" type="imu">
-      <always_on>true</always_on>
-      <update_rate>200</update_rate>
-      <visualize>true</visualize>
-      <topic>__default_topic__</topic>
-      <plugin filename="libgazebo_ros_imu_sensor.so" name="imu_plugin">
-        <topicName>ros_imu</topicName>
-        <bodyName>imu_link</bodyName>
-        <updateRateHZ>200.0</updateRateHZ>
-        <gaussianNoise>0.001</gaussianNoise>
-        <xyzOffset>0 0 0</xyzOffset>
-        <rpyOffset>0 0 0</rpyOffset>
-        <frameName>imu</frameName>
-      </plugin>
-      <pose>0 0 0 0 0 0</pose>
-    </sensor>
-  </gazebo>
-  <!-- gps plugin -->
-  <gazebo>
-    <plugin name="gps_controller" filename="libhector_gazebo_ros_gps.so">
-      <updateRate>5.0</updateRate>
-      <bodyName>gps</bodyName>
-      <topicName>/fix</topicName>
-      <velocityTopicName>/fix_velocity</velocityTopicName>
-    </plugin>
-  </gazebo>
+    xmlns:xacro="http://www.ros.org/wiki/xacro" name="hydrus" >
+  <!--<xacro:arg name="robot_name" default="hydrus" />-->
+  <!-- gazebo plugin for default controller and sensors -->
+  <xacro:include filename="$(find aerial_robot_simulation)/xacro/spinal.gazebo.xacro" />
+  <xacro:gazebo_spinal robot_name="$(arg robot_name)" />
 </robot>

File: mbzirc2020/mbzirc2020_common/robots/default.urdf.xacro (robot description, xacro)
@@ -1,5 +1,5 @@
 <?xml version="1.0"?>
 <robot
-    xmlns:xacro="http://www.ros.org/wiki/xacro" name="hydrusx" >
+    xmlns:xacro="http://www.ros.org/wiki/xacro" name="hydrus" >
   <!-- basic kinematics model -->
   <xacro:include filename="$(find hydrus)/urdf/common.xacro" />
@@ -8,14 +8,14 @@
   <xacro:macro name="robot_model" params="tilt_angle:=0 downward_vio:=1 horizontal_vio:=0 default_battery:=1 with_leg:=1">
     <xacro:if value="${tilt_angle == 0}"> <!--no tilt angle-->
-      <xacro:hydrusx_link links="4" self="1" rotor_direction="-1" with_battery = "${default_battery}" with_leg = "${with_leg}" tilt_mode="0" />
-      <xacro:hydrusx_fixed_link self="2" rotor_direction="1"  with_battery = "${default_battery}" with_leg = "${with_leg}" tilt_angle = "0" />
-      <xacro:hydrusx_fixed_link self="3" rotor_direction="-1" with_battery = "${default_battery}" with_leg = "${with_leg}" tilt_angle = "0" />
-      <xacro:hydrusx_link links="4" self="4" rotor_direction="1"  with_battery = "${default_battery}" with_leg = "${with_leg}" tilt_mode="0" />
+      <xacro:hydrus_link links="4" self="1" rotor_direction="-1" with_battery = "${default_battery}" with_leg = "${with_leg}" tilt_mode="0" />
+      <xacro:hydrus_fixed_link self="2" rotor_direction="1"  with_battery = "${default_battery}" with_leg = "${with_leg}" tilt_angle = "0" />
+      <xacro:hydrus_fixed_link self="3" rotor_direction="-1" with_battery = "${default_battery}" with_leg = "${with_leg}" tilt_angle = "0" />
+      <xacro:hydrus_link links="4" self="4" rotor_direction="1"  with_battery = "${default_battery}" with_leg = "${with_leg}" tilt_mode="0" />
     </xacro:if>
     <xacro:unless value="${tilt_angle == 0}">
-      <xacro:hydrusx_link links="4" self="1" rotor_direction="-1" with_battery = "${default_battery}" with_leg = "${with_leg}" tilt_mode="1" tilt_angle="${tilt_angle}" />
-      <xacro:hydrusx_fixed_link self="2" rotor_direction="1"  with_battery = "${default_battery}" with_leg = "${with_leg}" tilt_angle = "${tilt_angle}" />
-      <xacro:hydrusx_fixed_link self="3" rotor_direction="-1" with_battery = "${default_battery}" with_leg = "${with_leg}" tilt_angle = "${tilt_angle}" />
-      <xacro:hydrusx_link links="4" self="4" rotor_direction="1"  with_battery = "${default_battery}" with_leg = "${with_leg}" tilt_mode="1" tilt_angle="${tilt_angle}"/>
+      <xacro:hydrus_link links="4" self="1" rotor_direction="-1" with_battery = "${default_battery}" with_leg = "${with_leg}" tilt_mode="1" tilt_angle="${tilt_angle}" />
+      <xacro:hydrus_fixed_link self="2" rotor_direction="1"  with_battery = "${default_battery}" with_leg = "${with_leg}" tilt_angle = "${tilt_angle}" />
+      <xacro:hydrus_fixed_link self="3" rotor_direction="-1" with_battery = "${default_battery}" with_leg = "${with_leg}" tilt_angle = "${tilt_angle}" />
+      <xacro:hydrus_link links="4" self="4" rotor_direction="1"  with_battery = "${default_battery}" with_leg = "${with_leg}" tilt_mode="1" tilt_angle="${tilt_angle}"/>
     </xacro:unless>
     <!-- onboard -->

File: mbzirc2020/mbzirc2020_common/urdf/fixed_link.urdf.xacro (robot description, xacro)
@@ -1,6 +1,6 @@
 <?xml version="1.0"?>
 <robot
-    xmlns:xacro="http://www.ros.org/wiki/xacro" name="hydrusx_fixed_link" >
-  <xacro:macro name="hydrusx_fixed_link" params="self rotor_direction with_battery:=1 with_leg:=1 tilt_angle:=0">
+    xmlns:xacro="http://www.ros.org/wiki/xacro" name="hydrus_fixed_link" >
+  <xacro:macro name="hydrus_fixed_link" params="self rotor_direction with_battery:=1 with_leg:=1 tilt_angle:=0">
     <!-- link -->
     <link name="link${self}">

File: mbzirc2020/mbzirc2020_task1/mbzirc2020_task1_common/robots/hydrus.gazebo.xacro (robot description, xacro)
@@ -1,6 +1,7 @@
 <?xml version="1.0"?>
 <robot
-    xmlns:xacro="http://www.ros.org/wiki/xacro" name="hydrusx" >
+    xmlns:xacro="http://www.ros.org/wiki/xacro" name="hydrus" >
   <!-- base robot model -->
+  <xacro:arg name="robot_name" default="hydrus" />
   <xacro:arg name="monocular_camera" default="true" />
   <xacro:include filename="$(find mbzirc2020_task1_common)/robots/hydrus.urdf.xacro" />
@@ -102,4 +103,5 @@
         </camera>
         <plugin name="depth_camera" filename="libgazebo_ros_openni_kinect.so">
+          <robotNamespace>$(arg robot_name)</robotNamespace>
 	  <baseline>0.06</baseline>
 	  <alwaysOn>true</alwaysOn>

File: mbzirc2020/mbzirc2020_task1/mbzirc2020_task1_common/robots/hydrus.urdf.xacro (robot description, xacro)
@@ -1,5 +1,5 @@
 <?xml version="1.0"?>
 <robot
-    xmlns:xacro="http://www.ros.org/wiki/xacro" name="hydrusx" >
+    xmlns:xacro="http://www.ros.org/wiki/xacro" name="hydrus" >
   <!-- base kinematics model -->
   <xacro:arg name="monocular_camera" default="true" />

File: mbzirc2020/mbzirc2020_task2/mbzirc2020_task2_common/robots/default.urdf.xacro (robot description, xacro)
@@ -1,5 +1,5 @@
 <?xml version="1.0"?>
 <robot
-    xmlns:xacro="http://www.ros.org/wiki/xacro" name="hydrusx" >
+    xmlns:xacro="http://www.ros.org/wiki/xacro" name="hydrus" >
   <!-- basic kinematics model -->
   <xacro:include filename="$(find hydrus)/urdf/common.xacro" />
@@ -8,14 +8,14 @@
   <xacro:macro name="robot_model" params="tilt_angle:=0 downward_vio:=1 horizontal_vio:=0 default_battery:=1 with_leg:=1">
     <xacro:if value="${tilt_angle == 0}"> <!--no tilt angle-->
-      <xacro:hydrusx_link links="4" self="1" rotor_direction="-1" with_battery = "${default_battery}" with_leg = "${with_leg}" tilt_mode="0" />
-      <xacro:hydrusx_fixed_link self="2" rotor_direction="1"  with_battery = "${default_battery}" with_leg = "${with_leg}" tilt_angle = "0" />
-      <xacro:hydrusx_fixed_link self="3" rotor_direction="-1" with_battery = "${default_battery}" with_leg = "${with_leg}" tilt_angle = "0" />
-      <xacro:hydrusx_link links="4" self="4" rotor_direction="1"  with_battery = "${default_battery}" with_leg = "${with_leg}" tilt_mode="0" />
+      <xacro:hydrus_link links="4" self="1" rotor_direction="-1" with_battery = "${default_battery}" with_leg = "${with_leg}" tilt_mode="0" />
+      <xacro:hydrus_fixed_link self="2" rotor_direction="1"  with_battery = "${default_battery}" with_leg = "${with_leg}" tilt_angle = "0" />
+      <xacro:hydrus_fixed_link self="3" rotor_direction="-1" with_battery = "${default_battery}" with_leg = "${with_leg}" tilt_angle = "0" />
+      <xacro:hydrus_link links="4" self="4" rotor_direction="1"  with_battery = "${default_battery}" with_leg = "${with_leg}" tilt_mode="0" />
     </xacro:if>
     <xacro:unless value="${tilt_angle == 0}">
-      <xacro:hydrusx_link links="4" self="1" rotor_direction="-1" with_battery = "${default_battery}" with_leg = "${with_leg}" tilt_mode="1" tilt_angle="${tilt_angle}" />
-      <xacro:hydrusx_fixed_link self="2" rotor_direction="1"  with_battery = "${default_battery}" with_leg = "${with_leg}" tilt_angle = "${tilt_angle}" />
-      <xacro:hydrusx_fixed_link self="3" rotor_direction="-1" with_battery = "${default_battery}" with_leg = "${with_leg}" tilt_angle = "${tilt_angle}" />
-      <xacro:hydrusx_link links="4" self="4" rotor_direction="1"  with_battery = "${default_battery}" with_leg = "${with_leg}" tilt_mode="1" tilt_angle="${tilt_angle}"/>
+      <xacro:hydrus_link links="4" self="1" rotor_direction="-1" with_battery = "${default_battery}" with_leg = "${with_leg}" tilt_mode="1" tilt_angle="${tilt_angle}" />
+      <xacro:hydrus_fixed_link self="2" rotor_direction="1"  with_battery = "${default_battery}" with_leg = "${with_leg}" tilt_angle = "${tilt_angle}" />
+      <xacro:hydrus_fixed_link self="3" rotor_direction="-1" with_battery = "${default_battery}" with_leg = "${with_leg}" tilt_angle = "${tilt_angle}" />
+      <xacro:hydrus_link links="4" self="4" rotor_direction="1"  with_battery = "${default_battery}" with_leg = "${with_leg}" tilt_mode="1" tilt_angle="${tilt_angle}"/>
     </xacro:unless>
     <!-- onboard -->

File: mbzirc2020/mbzirc2020_task2/mbzirc2020_task2_common/robots/hydrus.gazebo.xacro (robot description, xacro)
@@ -1,5 +1,5 @@
 <?xml version="1.0"?>
 <robot
-    xmlns:xacro="http://www.ros.org/wiki/xacro" name="hydrusx" >
+    xmlns:xacro="http://www.ros.org/wiki/xacro" name="hydrus" >
   <!-- base robot model -->
   <xacro:include filename="$(find mbzirc2020_task2_common)/robots/hydrus.urdf.xacro" />

File: mbzirc2020/mbzirc2020_task2/mbzirc2020_task2_common/robots/hydrus.urdf.xacro (robot description, xacro)
@@ -1,5 +1,5 @@
 <?xml version="1.0"?>
 <robot
-    xmlns:xacro="http://www.ros.org/wiki/xacro" name="hydrusx" >
+    xmlns:xacro="http://www.ros.org/wiki/xacro" name="hydrus" >
   <!-- base kinematics model -->
   <xacro:arg name="horizontal_vio" default="false" />

File: mbzirc2020/mbzirc2020_task2/mbzirc2020_task2_common/robots/hydrus_ground_mode.gazebo.xacro (robot description, xacro)
@@ -1,5 +1,6 @@
 <?xml version="1.0"?>
 <robot
-    xmlns:xacro="http://www.ros.org/wiki/xacro" name="hydrusx" >
+    xmlns:xacro="http://www.ros.org/wiki/xacro" name="hydrus" >
+  <xacro:arg name="robot_name" default="hydrus" />
   <!-- base robot model -->
   <xacro:include filename="$(find mbzirc2020_task2_common)/robots/hydrus_ground_mode.urdf.xacro" />
@@ -128,4 +129,5 @@
       </camera>
       <plugin name="depth_camera" filename="libgazebo_ros_openni_kinect.so">
+        <robotNamespace>$(arg robot_name)</robotNamespace>
 	<baseline>0.06</baseline>
 	<alwaysOn>true</alwaysOn>

File: mbzirc2020/mbzirc2020_task2/mbzirc2020_task2_common/robots/hydrus_ground_mode.urdf.xacro (robot description, xacro)
@@ -1,13 +1,13 @@
 <?xml version="1.0"?>
 <robot
-    xmlns:xacro="http://www.ros.org/wiki/xacro" name="hydrusx" >
+    xmlns:xacro="http://www.ros.org/wiki/xacro" name="hydrus" >
   <!-- base kinematics model -->
   <xacro:include filename="$(find hydrus)/urdf/common.xacro" />
   <xacro:include filename="$(find hydrus)/urdf/link.urdf.xacro" />
   <xacro:include filename="$(find mbzirc2020_common)/urdf/fixed_link.urdf.xacro" />
-  <xacro:hydrusx_link links="4" self="1" rotor_direction="-1" with_battery = "0" with_leg = "0" tilt_mode="0" />
-  <xacro:hydrusx_fixed_link self="2" rotor_direction="1"  with_battery = "0" with_leg = "0" tilt_angle = "0" />
-  <xacro:hydrusx_fixed_link self="3" rotor_direction="-1" with_battery = "0" with_leg = "0" tilt_angle = "0" />
-  <xacro:hydrusx_link links="4" self="4" rotor_direction="1"  with_battery = "0" with_leg = "0" tilt_mode="0" />
+  <xacro:hydrus_link links="4" self="1" rotor_direction="-1" with_battery = "0" with_leg = "0" tilt_mode="0" />
+  <xacro:hydrus_fixed_link self="2" rotor_direction="1"  with_battery = "0" with_leg = "0" tilt_angle = "0" />
+  <xacro:hydrus_fixed_link self="3" rotor_direction="-1" with_battery = "0" with_leg = "0" tilt_angle = "0" />
+  <xacro:hydrus_link links="4" self="4" rotor_direction="1"  with_battery = "0" with_leg = "0" tilt_mode="0" />
   <!-- onboard -->
   <!-- 1.  processor -->

File: mbzirc2020/mbzirc2020_task2/mbzirc2020_task2_common/robots/hydrus_passive_gripper.gazebo.xacro (robot description, xacro)
@@ -1,5 +1,6 @@
 <?xml version="1.0"?>
 <robot
-    xmlns:xacro="http://www.ros.org/wiki/xacro" name="hydrusx" >
+    xmlns:xacro="http://www.ros.org/wiki/xacro" name="hydrus" >
+  <xacro:arg name="robot_name" default="hydrus" />
   <!-- base robot model -->
   <xacro:include filename="$(find mbzirc2020_task2_common)/robots/hydrus_passive_gripper.urdf.xacro" />
@@ -100,4 +101,5 @@
       </camera>
       <plugin name="depth_camera" filename="libgazebo_ros_openni_kinect.so">
+        <robotNamespace>$(arg robot_name)</robotNamespace>
 	<baseline>0.06</baseline>
 	<alwaysOn>true</alwaysOn>

File: mbzirc2020/mbzirc2020_task2/mbzirc2020_task2_common/robots/hydrus_passive_gripper.urdf.xacro (robot description, xacro)
@@ -1,5 +1,5 @@
 <?xml version="1.0"?>
 <robot
-    xmlns:xacro="http://www.ros.org/wiki/xacro" name="hydrusx" >
+    xmlns:xacro="http://www.ros.org/wiki/xacro" name="hydrus" >
   <!-- base kinematics model -->
   <xacro:include filename="$(find mbzirc2020_common)/robots/default.urdf.xacro" />

File: mbzirc2020/mbzirc2020_task2/mbzirc2020_task2_common/robots/hydrus_ring_gripper.gazebo.xacro (robot description, xacro)
@@ -1,5 +1,6 @@
 <?xml version="1.0"?>
 <robot
-    xmlns:xacro="http://www.ros.org/wiki/xacro" name="hydrusx" >
+    xmlns:xacro="http://www.ros.org/wiki/xacro" name="hydrus" >
+  <xacro:arg name="robot_name" default="hydrus" />
   <!-- base robot model -->
   <xacro:include filename="$(find mbzirc2020_task2_common)/robots/hydrus_ring_gripper.urdf.xacro" />
@@ -100,4 +101,5 @@
       </camera>
       <plugin name="depth_camera" filename="libgazebo_ros_openni_kinect.so">
+        <robotNamespace>$(arg robot_name)</robotNamespace>
 	<baseline>0.06</baseline>
 	<alwaysOn>true</alwaysOn>
@@ -128,5 +130,5 @@
     <plugin name="gazebo_grasp_fix" filename="libgazebo_grasp_fix.so">
       <arm>
-        <arm_name>hydrusx_arm</arm_name>
+        <arm_name>hydrus_arm</arm_name>
         <palm_link>link2</palm_link>
         <gripper_link>root</gripper_link>

File: mbzirc2020/mbzirc2020_task2/mbzirc2020_task2_common/robots/hydrus_ring_gripper.urdf.xacro (robot description, xacro)
@@ -1,5 +1,5 @@
 <?xml version="1.0"?>
 <robot
-    xmlns:xacro="http://www.ros.org/wiki/xacro" name="hydrusx" >
+    xmlns:xacro="http://www.ros.org/wiki/xacro" name="hydrus" >
   <!-- base kinematics model -->
   <xacro:include filename="$(find mbzirc2020_task2_common)/robots/default.urdf.xacro" />

File: mbzirc2020/mbzirc2020_task2/mbzirc2020_task2_simulation/urdf/gzplugin_grasp_fix.urdf.xacro (robot description, xacro)
@@ -15,5 +15,5 @@
         -->
         <arm>
-          <arm_name>hydrusx_arm</arm_name>
+          <arm_name>hydrus_arm</arm_name>
           <palm_link>link2</palm_link>
           <gripper_link>link4</gripper_link>

File: mbzirc2020/mbzirc2020_task3/mbzirc2020_task3_common/robots/hydrus.gazebo.xacro (robot description, xacro)
@@ -1,5 +1,7 @@
 <?xml version="1.0"?>
 <robot
-    xmlns:xacro="http://www.ros.org/wiki/xacro" name="hydrusx" >
+    xmlns:xacro="http://www.ros.org/wiki/xacro" name="hydrus" >
+  <xacro:arg name="robot_name" default="hydrus" />
+  <xacro:arg name="monocular_camera" default="true" />
   <!-- base robot model -->
   <xacro:include filename="$(find mbzirc2020_task3_common)/robots/hydrus.urdf.xacro" />
@@ -29,4 +31,5 @@
       </camera>
       <plugin name="camera_controller" filename="libgazebo_ros_camera.so">
+        <robotNamespace>$(arg robot_name)</robotNamespace>
         <alwaysOn>true</alwaysOn>
         <updateRate>0.0</updateRate>

File: mbzirc2020/mbzirc2020_task3/mbzirc2020_task3_common/robots/hydrus.urdf.xacro (robot description, xacro)
@@ -1,5 +1,5 @@
 <?xml version="1.0"?>
 <robot
-    xmlns:xacro="http://www.ros.org/wiki/xacro" name="hydrusx" >
+    xmlns:xacro="http://www.ros.org/wiki/xacro" name="hydrus" >
   <!-- base kinematics model -->
   <xacro:arg name="horizontal_vio" default="0" />

File: mbzirc2020/mbzirc2020_task3/mbzirc2020_task3_common/robots/hydrus_rsd435.gazebo.xacro (robot description, xacro)
@@ -1,5 +1,6 @@
 <?xml version="1.0"?>
 <robot
-    xmlns:xacro="http://www.ros.org/wiki/xacro" name="hydrusx" >
+    xmlns:xacro="http://www.ros.org/wiki/xacro" name="hydrus" >
+  <xacro:arg name="monocular_camera" default="true" />
   <!-- base robot model -->
   <xacro:include filename="$(find mbzirc2020_task3_common)/robots/hydrus_rsd435.urdf.xacro" />

File: mbzirc2020/mbzirc2020_task3/mbzirc2020_task3_common/robots/hydrus_rsd435.urdf.xacro (robot description, xacro)
@@ -1,5 +1,5 @@
 <?xml version="1.0"?>
 <robot
-    xmlns:xacro="http://www.ros.org/wiki/xacro" name="hydrusx" >
+    xmlns:xacro="http://www.ros.org/wiki/xacro" name="hydrus" >
   <!-- base kinematics model -->
   <xacro:arg name="horizontal_vio" default="0" />
