Commit message: Fix the bug about robot model in task2: 1. the configuration for gazebo grasping plugin 2. the radius of propeller protector

File: mbzirc2020/mbzirc2020_common/urdf/fixed_link.urdf.xacro (robot description, xacro)
@@ -88,5 +88,5 @@
         <origin rpy="0 0 0" xyz="0 0 0"/>
         <geometry>
-          <cylinder length="0.1" radius="${protector_radius -0.1}"/>
+          <cylinder length="0.1" radius="${protector_radius + 0.01}"/>
         </geometry>
       </collision>

File: mbzirc2020/mbzirc2020_task2/mbzirc2020_task2_simulation/urdf/gzplugin_grasp_fix.urdf.xacro (robot description, xacro)
@@ -16,8 +16,11 @@
         <arm>
           <arm_name>hydrusx_arm</arm_name>
-          <palm_link>link3</palm_link>
-          <gripper_link>link2</gripper_link>
+          <palm_link>link2</palm_link>
           <gripper_link>link4</gripper_link>
           <gripper_link>root</gripper_link>
+          <gripper_link>thrust1</gripper_link>
+          <gripper_link>thrust2</gripper_link>
+          <gripper_link>thrust3</gripper_link>
+          <gripper_link>thrust4</gripper_link>
         </arm>
         <forces_angle_tolerance>100</forces_angle_tolerance>

Commit message: [mbzirc2020_common] modify fixed link: collision model changes when with_leg is false

File: mbzirc2020/mbzirc2020_common/urdf/fixed_link.urdf.xacro (robot description, xacro)
@@ -49,8 +49,16 @@
       <!-- for fcl in planning -->
       <collision>
+        <xacro:if value="${with_leg == 1}">
           <origin rpy="0 0 0" xyz="${link_length* 0.5} 0 ${- leg_collision_model_height / 2}"/>
           <geometry>
             <box size="${link_length} 0.05 ${leg_collision_model_height}"/>
           </geometry>
+        </xacro:if>
+        <xacro:unless value="${with_leg == 1}">
+          <origin rpy="0 0 0" xyz="${link_length* 0.5} 0 0"/>
+          <geometry>
+            <box size="${link_length} 0.05 0.1"/>
+          </geometry>
+        </xacro:unless>
       </collision>
       <visual>

Commit message: [mbzirc2020_common] add prop_15inch arg in hydrus_fixed_link

File: mbzirc2020/mbzirc2020_common/urdf/fixed_link.urdf.xacro (robot description, xacro)
@@ -2,5 +2,5 @@
 <robot
     xmlns:xacro="http://www.ros.org/wiki/xacro" name="hydrus_fixed_link" >
-  <xacro:macro name="hydrus_fixed_link" params="self rotor_direction with_battery:=1 with_leg:=1 tilt_angle:=0">
+  <xacro:macro name="hydrus_fixed_link" params="self rotor_direction with_battery:=1 with_leg:=1 tilt_angle:=0 prop_15inch:=0">
     <!-- link -->
     <link name="link${self}">
@@ -80,5 +80,10 @@
       <parent link="link${self}"/>
       <child link="thrust${self}"/>
-      <origin rpy="0 ${-rotor_direction * tilt_angle * pi / 180.0} 0" xyz="${link_length* 0.5} 0 0.045"/>
+      <xacro:if value="${prop_15inch == 1}">
+        <origin rpy="0 ${-rotor_direction * tilt_angle * pi / 180.0} 0" xyz="${link_length* 0.5 + 0.01944 * rotor_direction} 0 0.05395"/>
+      </xacro:if>
+      <xacro:unless value="${prop_15inch == 1}">
+        <origin rpy="0 ${-rotor_direction * tilt_angle * pi / 180.0} 0" xyz="${link_length* 0.5} 0 0.045"/>
+      </xacro:unless>
       <axis xyz="0 0 ${rotor_direction}"/>
     </joint>

Commit message: [mbzirc2020_common] update inertial parameter of prop_15inch model

File: mbzirc2020/mbzirc2020_common/urdf/fixed_link.urdf.xacro (robot description, xacro)
@@ -17,11 +17,22 @@
         </xacro:if>
         <xacro:unless value="${tilt_angle == 0}">
-          <inertial>
-            <origin xyz="${link_length* 0.5 - 0.041294} 0.0 0.02189" rpy="0 0 0"/>
-            <mass value="0.51919"/>
-            <inertia
-                ixx="0.002049" iyy="0.010608" izz="0.011696"
-                ixy="0.00000" ixz="0.000267" iyz="0.00000"/>
-          </inertial>
+          <xacro:if value="${prop_15inch == 1}">
+            <inertial>
+              <origin xyz="${link_length* 0.5 - 0.035768} 0.0 0.024087" rpy="0 0 0"/>
+              <mass value="0.513137"/>
+              <inertia
+                  ixx="0.002135" iyy="0.010964" izz="0.011963"
+                  ixy="-0.000067" ixz="0.000435" iyz="-0.000011"/>
+            </inertial>
+          </xacro:if>
+          <xacro:unless value="${prop_15inch == 1}">
+            <inertial>
+              <origin xyz="${link_length* 0.5 - 0.041294} 0.0 0.02189" rpy="0 0 0"/>
+              <mass value="0.51919"/>
+              <inertia
+                  ixx="0.002049" iyy="0.010608" izz="0.011696"
+                  ixy="0.00000" ixz="0.000267" iyz="0.00000"/>
+            </inertial>
+          </xacro:unless>
         </xacro:unless>
       </xacro:if>
@@ -38,11 +49,22 @@
         </xacro:if>
         <xacro:unless value="${tilt_angle == 0}">
-          <inertial>
-            <origin xyz="${link_length* 0.5 + 0.038503} 0.0 0.0218" rpy="0 0 0"/>
-            <mass value="0.520389"/>
-            <inertia
-                ixx="0.00205" iyy="0.011055" izz="0.012143"
-                ixy="0.00000" ixz="-0.000234" iyz="0.00000"/>
-          </inertial>
+          <xacro:if value="${prop_15inch == 1}">
+            <inertial>
+              <origin xyz="${link_length* 0.5 + 0.035188} 0.0 0.024031" rpy="0 0 0"/>
+              <mass value="0.514337"/>
+              <inertia
+                  ixx="0.002136" iyy="0.011317" izz="0.012316"
+                  ixy="-0.000067" ixz="-0.000428" iyz="0.000011"/>
+            </inertial>
+          </xacro:if>
+          <xacro:unless value="${prop_15inch == 1}">
+            <inertial>
+              <origin xyz="${link_length* 0.5 + 0.038503} 0.0 0.0218" rpy="0 0 0"/>
+              <mass value="0.520389"/>
+              <inertia
+                  ixx="0.00205" iyy="0.011055" izz="0.012143"
+                  ixy="0.00000" ixz="-0.000234" iyz="0.00000"/>
+            </inertial>
+          </xacro:unless>
         </xacro:unless>
       </xacro:if>

Commit message: [mbzirc2020_common] add mesh file for 15inch prop model

File: mbzirc2020/mbzirc2020_common/urdf/fixed_link.urdf.xacro (robot description, xacro)
@@ -91,5 +91,10 @@
           </xacro:if>
           <xacro:unless value="${tilt_angle == 0}">
-            <mesh filename="package://mbzirc2020_common/urdf/mesh/link/tilt_${tilt_angle}deg_fix_joint_link${self}.dae"/>
+            <xacro:if value="${prop_15inch == 1}">
+              <mesh filename="package://mbzirc2020_common/urdf/mesh/link/tilt_${tilt_angle}deg_15inch_fix_joint_link${self}.dae"/>
+            </xacro:if>
+            <xacro:unless value="${prop_15inch == 1}">
+              <mesh filename="package://mbzirc2020_common/urdf/mesh/link/tilt_${tilt_angle}deg_fix_joint_link${self}.dae"/>
+            </xacro:unless>
           </xacro:unless>
         </geometry>
